File: USB-SSB-txcvr.kicad_sch (KiCad schematic)
At the start: 0 parts

Commit message: Hierarchy is mostly done?
Other:
- sheet Tuning DAC 1 renamed Rx Tuning DAC
- sheet Tuning DAC 2 renamed Tx Tuning DAC
- sheet Antenna Tuner, TR Relay ports: added AntTx, TxEnable; removed AntTxEnable
- sheet Receiver signal chain ports: added AntRxIn, RxTRFOut; removed RxFiltered
- sheet Rx Demod ports: added VFO; removed none
- sheet Transmitter signal chain ports: added TxExciterOut, TxI, TxQ, TxVtune1, TxVtune2, TxVtune3, VFO; removed none
- sheet VFO ports: added ControlSCL, ControlSDA, RxVFO, TxVFO; removed none
- sheet microcontroller ports: added TxEnable, TxI, TxQ, TxTuneLDAC-, TxTuneRDY, TxTuneSCL, TxTuneSDA, VFOSCL, VFOSDA; removed none
