File: ant.kicad_sch (KiCad schematic)
At the start: 0 parts

Commit message: Hierarchy is mostly done?
Changed lines of the file:
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@@
 		(comment 2 "WB7NAB")
 	)
-	(hierarchical_label "AntTxEnable"
+	(hierarchical_label "AntTx"
+		(shape input)
+		(at 22.86 69.85 0)
+		(effects
+			(font
+				(size 1.27 1.27)
+			)
+			(justify left)
+		)
+	)
+	(hierarchical_label "TxEnable"
 		(shape input)
 		(at 31.75 54.61 180)
