File: microcontroller.kicad_sch (KiCad schematic)
At the start: 0 parts

Commit message: Hierarchy is mostly done?
Changed lines of the file:
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@@
 		(comment 2 "WB7NAB")
 	)
+	(hierarchical_label "TxTuneSCL"
+		(shape bidirectional)
+		(at 248.92 96.52 0)
+		(effects
+			(font
+				(size 1.27 1.27)
+			)
+			(justify left)
+		)
+	)
+	(hierarchical_label "TxI"
+		(shape output)
+		(at 248.92 86.36 0)
+		(effects
+			(font
+				(size 1.27 1.27)
+			)
+			(justify left)
+		)
+	)
+	(hierarchical_label "TxEnable"
+		(shape output)
+		(at 251.46 72.39 0)
+		(effects
+			(font
+				(size 1.27 1.27)
+			)
+			(justify left)
+		)
+	)
 	(hierarchical_label "RxTuneLDAC-"
-		(shape input)
+		(shape output)
 		(at 248.92 58.42 0)
+		(effects
+			(font
+				(size 1.27 1.27)
+			)
+			(justify left)
+		)
+	)
+	(hierarchical_label "TxTuneSDA"
+		(shape bidirectional)
+		(at 248.92 100.33 0)
 		(effects
 			(font
@@
 		)
 	)
+	(hierarchical_label "TxQ"
+		(shape output)
+		(at 248.92 90.17 0)
+		(effects
+			(font
+				(size 1.27 1.27)
+			)
+			(justify left)
+		)
+	)
+	(hierarchical_label "TxTuneRDY"
+		(shape input)
+		(at 248.92 110.49 0)
+		(effects
+			(font
+				(size 1.27 1.27)
+			)
+			(justify left)
+		)
+	)
 	(hierarchical_label "RxTuneRDY"
 		(shape input)
 		(at 248.92 62.23 0)
+		(effects
+			(font
+				(size 1.27 1.27)
+			)
+			(justify left)
+		)
+	)
+	(hierarchical_label "VFOSCL"
+		(shape bidirectional)
+		(at 245.11 121.92 0)
+		(effects
+			(font
+				(size 1.27 1.27)
+			)
+			(justify left)
+		)
+	)
+	(hierarchical_label "VFOSDA"
+		(shape bidirectional)
+		(at 245.11 127 0)
+		(effects
+			(font
+				(size 1.27 1.27)
+			)
+			(justify left)
+		)
+	)
+	(hierarchical_label "TxTuneLDAC-"
+		(shape output)
+		(at 248.92 106.68 0)
 		(effects
 			(font
@@
 	)
 	(hierarchical_label "RxTuneSDA"
-		(shape input)
+		(shape bidirectional)
 		(at 248.92 53.34 0)
 		(effects
@@
 	)
 	(hierarchical_label "RxTuneSCL"
-		(shape input)
+		(shape bidirectional)
 		(at 248.92 49.53 0)
 		(effects
