File: rx-demod.kicad_sch (KiCad schematic)
At the start: 0 parts

Commit message: Hierarchy is mostly done?
Changed lines of the file:
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@@
+		)
+	)
+	(hierarchical_label "VFO"
+		(shape input)
+		(at 27.94 39.37 0)
+		(effects
+			(font
+				(size 1.27 1.27)
+			)
+			(justify left)
 		)
 	)
 	(hierarchical_label "RxI"
-		(shape input)
+		(shape output)
 		(at 31.75 26.67 180)
 		(effects
@@
 	)
 	(hierarchical_label "RxQ"
-		(shape input)
+		(shape output)
 		(at 31.75 30.48 180)
 		(effects
