File: rx-signal-chain.kicad_sch (KiCad schematic)
At the start: 0 parts

Commit message: Hierarchy is mostly done?
Changed lines of the file:
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@@
 		)
 	)
-	(hierarchical_label "RxFiltered"
+	(hierarchical_label "RxTRFOut"
 		(shape output)
 		(at 40.64 50.8 180)
@@
 		)
 	)
+	(hierarchical_label "AntRxIn"
+		(shape input)
+		(at 246.38 25.4 0)
+		(effects
+			(font
+				(size 1.27 1.27)
+			)
+			(justify left)
+		)
+	)
