File: tx-signal-chain.kicad_sch (KiCad schematic)
At the start: 0 parts

Commit message: Hierarchy is mostly done?
Changed lines of the file:
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@@
+		)
+	)
+	(hierarchical_label "TxVtune1"
+		(shape input)
+		(at 27.94 52.07 0)
+		(effects
+			(font
+				(size 1.27 1.27)
+			)
+			(justify left)
 		)
 	)
@@
 		)
 	)
-	(hierarchical_label "TxVFO"
+	(hierarchical_label "TxVtune3"
+		(shape input)
+		(at 27.94 59.69 0)
+		(effects
+			(font
+				(size 1.27 1.27)
+			)
+			(justify left)
+		)
+	)
+	(hierarchical_label "TxExciterOut"
+		(shape output)
+		(at 242.57 29.21 0)
+		(effects
+			(font
+				(size 1.27 1.27)
+			)
+			(justify left)
+		)
+	)
+	(hierarchical_label "VFO"
 		(shape input)
 		(at 27.94 41.91 0)
 		(effects
 			(font
+				(size 1.27 1.27)
+			)
+			(justify left)
+		)
+	)
+	(hierarchical_label "TxVtune2"
+		(shape input)
+		(at 27.94 55.88 0)
+		(effects
+			(font
