File: hw/front-end-sim.kicad_sch (KiCad schematic)
At the start: 0 parts

Commit message: Starting to build BPFs for 7 bands
Other:
- removed sheet frontend-sim
Changed lines of the file:
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@@
 		(at 95.25 39.37)
 		(size 29.21 30.48)
-		(exclude_from_sim yes)
+		(exclude_from_sim no)
 		(in_bom yes)
 		(on_board yes)
@@
 		(at 22.86 83.185)
 		(size 35.56 17.145)
-		(exclude_from_sim yes)
+		(exclude_from_sim no)
 		(in_bom yes)
 		(on_board yes)
@@
 		(at 95.25 116.84)
 		(size 29.21 21.59)
-		(exclude_from_sim yes)
+		(exclude_from_sim no)
 		(in_bom yes)
 		(on_board yes)
@@
 	)
 	(sheet
-		(at 104.14 27.94)
-		(size 12.7 3.81)
-		(exclude_from_sim no)
-		(in_bom no)
-		(on_board no)
-		(dnp yes)
-		(fields_autoplaced yes)
-		(stroke
-			(width 0.1524)
-			(type solid)
-		)
-		(fill
-			(color 0 0 0 0.0000)
-		)
-		(property "Sheetname" "frontend-sim"
-			(at 104.14 27.2284 0)
-			(effects
-				(font
-					(size 1.27 1.27)
-				)
-				(justify left bottom)
-			)
-		)
-		(property "Sheetfile" "frontend-sim.kicad_sch"
-			(at 104.14 32.3346 0)
-			(effects
-				(font
-					(size 1.27 1.27)
-				)
-				(justify left top)
-			)
-		)
-		(instances
-			(project "USB-SSB-txcvr"
-				(path "/8ae46c04-d01a-4756-8774-512b694bfaff"
-					(page "15")
-				)
-			)
-		)
-	)
-	(sheet
 		(at 245.11 138.43)
 		(size 15.24 12.7)
-		(exclude_from_sim yes)
+		(exclude_from_sim no)
 		(in_bom yes)
 		(on_board yes)
@@
 		(at 208.28 22.86)
 		(size 49.53 95.25)
-		(exclude_from_sim yes)
+		(exclude_from_sim no)
 		(in_bom yes)
 		(on_board yes)
@@
 		(at 148.59 73.66)
 		(size 31.75 24.13)
-		(exclude_from_sim yes)
+		(exclude_from_sim no)
 		(in_bom yes)
 		(on_board yes)
