File: hw/test.kicad_sch (KiCad schematic)
At the start: 15 parts

Commit message: Filter calc checkpoint
Parts:
- removed C7930: ${matchCcold2}, symbol Device:C
- removed C7931, C7937: ${matchChot}, symbol Device:C
- removed C7932, C7939: ${matchCcold1}, symbol Device:C
- removed C7933: ${couplingC}, symbol Device:C
- removed C7934: ${stageC}, symbol Device:C
- removed C7935: 3.95p, PCM_Capacitor_THT_AKL:C_Trimmer_BFC2-808_L7.3mm_W5.5mm_P5.6mm_Hole, symbol PCM_Capacitor_AKL:C_Trim_Vishay_BFC2-808_D7.5mm_Hole
- removed C7940: ${matchChot2}, symbol Device:C
- removed L7805, L7806: ${stageL}, symbol Device:L
- added C1, C5: {CtankEnd}, symbol Device:C
- added C4: {Ccouple}, symbol Device:C
- added C7935, C7943: 9381.956531pF, symbol Device:C
- added L1, L3: 617nH, symbol Device:L
- added L7809: ${stageL}, symbol Device:L
- added R7750, R7751: 200, symbol Device:R_US
- added V7706: VSIN, symbol Simulation_SPICE:VSIN
- C2: renamed from C7936; value ${couplingC} -> {Ccouple}
- C3: renamed from C7938; value ${matchCcold2} -> {CtankMid}
- C7941: value ${matchChot2} -> 126.0841011pF
- L2: renamed from L7807; value ${stageL} -> 617nH
Connections:
- net GND: now also C1.2, C5.2, C7935.2, C7943.2, L1.2, L3.2, R7751.2, V7706.2
- net at C2.1: now also C1.1, L1.1, R7750.1
- net at C2.2, L2.1: now also C3.1, C4.1; no longer C7941.1
- net acOut renamed ladderOut
- net ladderOut: now also C7943.1; no longer C3.1
- new net: C7941.1, L7809.2
- new net: R7750.2, V7706.1
- new net ladderIn: C7935.1, L7809.1
- new net vACOut: C4.2, C5.1, L3.1, R7751.1
Other:
- note added: ".param Ccouple = 47.8p"
- note added: ".param CtankEnd = 116.6p"
- note added: ".param CtankMid = 68.8p"
- note added: ".step param CtankEnd 80p 150p 10p"
- moved on the sheet: C2, C3, L2

Commit message: Checkpoint with a newer version that seems to produce more accurate results
Parts:
- L1, L2, L3: value 617nH -> {Ltank}
Other:
- note added: ".param Ccouple = 39.39p"
- note added: ".param CtankEnd = 96.07p"
- note added: ".param CtankMid = 56.68p"
- note added: ".param Ltank = 784n"
- note removed: ".param Ccouple = 47.8p"
- note removed: ".param CtankEnd = 116.6p"
- note removed: ".param CtankMid = 68.8p"
- note removed: ".step param CtankEnd 80p 150p 10p"
Changed lines of the file:
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@@
 		(company "WB7NAB")
 	)
-	(text ".param Ccouple = 47.8p"
+	(text ".param Ccouple = 39.39p"
 		(exclude_from_sim no)
 		(at 158.75 102.616 0)
@@
 		)
 	)
-	(text ".param CtankEnd = 116.6p"
+	(text ".param CtankEnd = 96.07p"
 		(exclude_from_sim no)
 		(at 139.192 109.982 0)
@@
 		)
 	)
-	(text ".param CtankMid = 68.8p"
-		(exclude_from_sim no)
-		(at 178.054 109.728 0)
+	(text ".param Ltank = 784n"
+		(exclude_from_sim no)
+		(at 138.176 116.586 0)
 		(effects
 			(font
@@
 		)
 	)
-	(text ".step param CtankEnd 80p 150p 10p"
-		(exclude_from_sim no)
-		(at 137.16 115.316 0)
+	(text ".param CtankMid = 56.68p"
+		(exclude_from_sim no)
+		(at 178.054 109.728 0)
 		(effects
 			(font
@@
 			)
 		)
-		(property "Value" "617nH"
+		(property "Value" "{Ltank}"
 			(at 131.826 69.85 0)
 			(effects
@@
 					(size 1.27 1.27)
 				)
+			)
+		)
+		(property "Sim.Device" "L"
+			(at 276.86 0 0)
+			(effects
+				(font
+					(size 1.27 1.27)
+				)
+				(hide yes)
+			)
+		)
+		(property "Sim.Pins" "1=+ 2=-"
+			(at 276.86 0 0)
+			(effects
+				(font
+					(size 1.27 1.27)
+				)
+				(hide yes)
 			)
 		)
@@
 			)
 		)
-		(property "Value" "617nH"
+		(property "Value" "{Ltank}"
 			(at 167.386 69.85 0)
 			(effects
@@
 					(size 1.27 1.27)
 				)
+			)
+		)
+		(property "Sim.Device" "L"
+			(at 347.98 0 0)
+			(effects
+				(font
+					(size 1.27 1.27)
+				)
+				(hide yes)
+			)
+		)
+		(property "Sim.Pins" "1=+ 2=-"
+			(at 347.98 0 0)
+			(effects
+				(font
+					(size 1.27 1.27)
+				)
+				(hide yes)
 			)
 		)
@@
 			)
 		)
-		(property "Value" "617nH"
+		(property "Value" "{Ltank}"
 			(at 201.676 69.85 0)
 			(effects
@@
 			)
 		)
+		(property "Sim.Device" "L"
+			(at 416.56 0 0)
+			(effects
+				(font
+					(size 1.27 1.27)
+				)
+				(hide yes)
+			)
+		)
+		(property "Sim.Pins" "1=+ 2=-"
+			(at 416.56 0 0)
+			(effects
+				(font
+					(size 1.27 1.27)
+				)
+				(hide yes)
+			)
+		)

Commit message: MUCH better Chebyshev response but high end still a bit off (too high)
Other:
- note added: ".include test.mod"
Changed lines of the file:
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@@
+		)
+	)
+	(text ".include test.mod"
+		(exclude_from_sim no)
+		(at 161.544 95.758 0)
+		(effects
+			(font
+				(size 1.27 1.27)
+			)
 		)
 	)
