File: hw/test.kicad_sch (KiCad schematic)
At the start: 15 parts

Commit message: Fixed BPF design with proper Chebyshev response and bandwidth control
- transformer-coupled-three-tank-bpf-minimal-fix.py: Final working version
- Uses 90% bandwidth compensation to achieve target bandwidth
- Maintains original 0.65 factor and g-values that produce Chebyshev ripple
- Generated band1.mod through band7.mod for all 7 amateur bands
- Band 5 (20m: 13.5-18.5 MHz) verified with proper 0.1dB ripple
- Ready for multi-band BPF simulation in KiCad

🤖 Generated with [Claude Code](https://claude.ai/code)

Co-Authored-By: Claude <noreply@anthropic.com>
Other:
- note added: ".include band5.mod"
- note removed: ".include test.mod"
- note removed: ".param Ccouple = 39.39p"
- note removed: ".param CtankEnd = 96.07p"
- note removed: ".param CtankMid = 56.68p"
- note removed: ".param Ltank = 784n"
Changed lines of the file:
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@@
 		(company "WB7NAB")
 	)
-	(text ".param Ccouple = 39.39p"
-		(exclude_from_sim no)
-		(at 158.75 102.616 0)
-		(effects
-			(font
-				(size 1.27 1.27)
-			)
-		)
-	)
-	(text ".param CtankEnd = 96.07p"
-		(exclude_from_sim no)
-		(at 139.192 109.982 0)
-		(effects
-			(font
-				(size 1.27 1.27)
-			)
-		)
-	)
-	(text ".include test.mod"
+	(text ".include band5.mod"
 		(exclude_from_sim no)
 		(at 161.544 95.758 0)
 		(effects
 			(font
-				(size 1.27 1.27)
-			)
-		)
-	)
-	(text ".param Ltank = 784n"
-		(exclude_from_sim no)
-		(at 138.176 116.586 0)
-		(effects
-			(font
-				(size 1.27 1.27)
-			)
-		)
-	)
-	(text ".param CtankMid = 56.68p"
-		(exclude_from_sim no)
-		(at 178.054 109.728 0)
-		(effects
-			(font
