File: hw/DAC.kicad_sch (KiCad schematic)
At the start: 16 parts, among them U1901 TLV320AIC3104RHBR

Commit message: Making some progress on PIN diode bias boost converter. Page number reorg.
Parts:
- renumbered C1901 to C1201, C1902 to C1202, C1903 to C1203, C1904 to C1204, C1905 to C1205, C1906 to C1206, C1907 to C1207, C1908 to C1208, C1909 to C1209, C1910 to C1210, C1911 to C1211, C1912 to C1212, C1913 to C1213, C1914 to C1214, C1915 to C1215, U1901 to U1201
Changed lines of the file:
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@@
 		(dnp no)
 		(fields_autoplaced yes)
-		(property "Reference" "#PWR01905"
+		(property "Reference" "#PWR01205"
 			(at 193.04 152.4 0)
 			(effects
@@
 			(project ""
 				(path "/8ae46c04-d01a-4756-8774-512b694bfaff/b2f84e19-834c-4e66-9c40-3d2adff3404a"
-					(reference "#PWR01905")
+					(reference "#PWR01205")
 					(unit 1)
 				)
@@
 		(on_board yes)
 		(dnp no)
-		(property "Reference" "C1915"
+		(property "Reference" "C1215"
 			(at 252.476 157.48 0)
 			(effects
@@
 			(project "USB-SSB-txcvr"
 				(path "/8ae46c04-d01a-4756-8774-512b694bfaff/b2f84e19-834c-4e66-9c40-3d2adff3404a"
-					(reference "C1915")
+					(reference "C1215")
 					(unit 1)
 				)
@@
 		(dnp no)
 		(fields_autoplaced yes)
-		(property "Reference" "#PWR01910"
+		(property "Reference" "#PWR01210"
 			(at 243.84 168.91 0)
 			(effects
@@
 			(project "USB-SSB-txcvr"
 				(path "/8ae46c04-d01a-4756-8774-512b694bfaff/b2f84e19-834c-4e66-9c40-3d2adff3404a"
-					(reference "#PWR01910")
+					(reference "#PWR01210")
 					(unit 1)
 				)
@@
 		(on_board yes)
 		(dnp no)
-		(property "Reference" "C1909"
+		(property "Reference" "C1209"
 			(at 179.324 157.226 0)
 			(effects
@@
 			(project "USB-SSB-txcvr"
 				(path "/8ae46c04-d01a-4756-8774-512b694bfaff/b2f84e19-834c-4e66-9c40-3d2adff3404a"
-					(reference "C1909")
+					(reference "C1209")
 					(unit 1)
 				)
@@
 		(on_board yes)
 		(dnp no)
-		(property "Reference" "#PWR01902"
+		(property "Reference" "#PWR01202"
 			(at 132.08 152.4 0)
 			(effects
@@
 			(project "USB-SSB-txcvr"
 				(path "/8ae46c04-d01a-4756-8774-512b694bfaff/b2f84e19-834c-4e66-9c40-3d2adff3404a"
-					(reference "#PWR01902")
+					(reference "#PWR01202")
 					(unit 1)
 				)
@@
 		(on_board yes)
 		(dnp no)
-		(property "Reference" "C1907"
+		(property "Reference" "C1207"
 			(at 152.908 157.226 0)
 			(effects
@@
 			(project "USB-SSB-txcvr"
 				(path "/8ae46c04-d01a-4756-8774-512b694bfaff/b2f84e19-834c-4e66-9c40-3d2adff3404a"
-					(reference "C1907")
+					(reference "C1207")
 					(unit 1)
 				)
@@
 		(on_board yes)
 		(dnp no)
-		(property "Reference" "C1914"
+		(property "Reference" "C1214"
 			(at 242.824 157.734 0)
 			(effects
@@
 			(project "USB-SSB-txcvr"
 				(path "/8ae46c04-d01a-4756-8774-512b694bfaff/b2f84e19-834c-4e66-9c40-3d2adff3404a"
-					(reference "C1914")
+					(reference "C1214")
 					(unit 1)
 				)
@@
 		(dnp no)
 		(fields_autoplaced yes)
-		(property "Reference" "#PWR01906"
+		(property "Reference" "#PWR01206"
 			(at 193.04 168.91 0)
 			(effects
@@
 			(project "USB-SSB-txcvr"
 				(path "/8ae46c04-d01a-4756-8774-512b694bfaff/b2f84e19-834c-4e66-9c40-3d2adff3404a"
-					(reference "#PWR01906")
+					(reference "#PWR01206")
 					(unit 1)
 				)
@@
 		(dnp no)
 		(fields_autoplaced yes)
-		(property "Reference" "#PWR01903"
+		(property "Reference" "#PWR01203"
 			(at 132.08 168.91 0)
 			(effects
@@
 			(project "USB-SSB-txcvr"
 				(path "/8ae46c04-d01a-4756-8774-512b694bfaff/b2f84e19-834c-4e66-9c40-3d2adff3404a"
-					(reference "#PWR01903")
+					(reference "#PWR01203")
 					(unit 1)
 				)
@@
 		(dnp no)
 		(fields_autoplaced yes)
-		(property "Reference" "#PWR01907"
+		(property "Reference" "#PWR01207"
 			(at 218.44 151.13 0)
 			(effects
@@
 			(project "USB-SSB-txcvr"
 				(path "/8ae46c04-d01a-4756-8774-512b694bfaff/b2f84e19-834c-4e66-9c40-3d2adff3404a"
-					(reference "#PWR01907")
+					(reference "#PWR01207")
 					(unit 1)
 				)
@@
 		(on_board yes)
 		(dnp no)
-		(property "Reference" "C1910"
+		(property "Reference" "C1210"
 			(at 191.77 157.734 0)
 			(effects
@@
 			(project "USB-SSB-txcvr"
 				(path "/8ae46c04-d01a-4756-8774-512b694bfaff/b2f84e19-834c-4e66-9c40-3d2adff3404a"
-					(reference "C1910")
+					(reference "C1210")
 					(unit 1)
 				)
@@
 		(on_board yes)
 		(dnp no)
-		(property "Reference" "U1901"
+		(property "Reference" "U1201"
 			(at 76.962 39.116 0)
 			(effects
@@
 			(project ""
 				(path "/8ae46c04-d01a-4756-8774-512b694bfaff/b2f84e19-834c-4e66-9c40-3d2adff3404a"
-					(reference "U1901")
+					(reference "U1201")
 					(unit 2)
 				)
@@
 		(on_board yes)
 		(dnp no)
-		(property "Reference" "C1903"
+		(property "Reference" "C1203"
 			(at 143.002 63.5 90)
 			(effects
@@
 			(project "USB-SSB-txcvr"
 				(path "/8ae46c04-d01a-4756-8774-512b694bfaff/b2f84e19-834c-4e66-9c40-3d2adff3404a"
-					(reference "C1903")
+					(reference "C1203")
 					(unit 1)
 				)
@@
 		(on_board yes)
 		(dnp no)
-		(property "Reference" "U1901"
+		(property "Reference" "U1201"
 			(at 197.104 37.846 0)
 			(effects
@@
 			(project ""
 				(path "/8ae46c04-d01a-4756-8774-512b694bfaff/b2f84e19-834c-4e66-9c40-3d2adff3404a"
-					(reference "U1901")
+					(reference "U1201")
 					(unit 1)
 				)
@@
 		(on_board yes)
 		(dnp no)
-		(property "Reference" "C1901"
+		(property "Reference" "C1201"
 			(at 138.684 157.226 0)
 			(effects
@@
 			(project "USB-SSB-txcvr"
 				(path "/8ae46c04-d01a-4756-8774-512b694bfaff/b2f84e19-834c-4e66-9c40-3d2adff3404a"
-					(reference "C1901")
+					(reference "C1201")
 					(unit 1)
 				)
@@
 		(on_board yes)
 		(dnp no)
-		(property "Reference" "C1913"
+		(property "Reference" "C1213"
 			(at 227.076 157.48 0)
 			(effects
@@
 			(project "USB-SSB-txcvr"
 				(path "/8ae46c04-d01a-4756-8774-512b694bfaff/b2f84e19-834c-4e66-9c40-3d2adff3404a"
-					(reference "C1913")
+					(reference "C1213")
 					(unit 1)
 				)
@@
 		(on_board yes)
 		(dnp no)
-		(property "Reference" "C1904"
+		(property "Reference" "C1204"
 			(at 148.844 157.226 0)
 			(effects
@@
 			(project "USB-SSB-txcvr"
 				(path "/8ae46c04-d01a-4756-8774-512b694bfaff/b2f84e19-834c-4e66-9c40-3d2adff3404a"
-					(reference "C1904")
+					(reference "C1204")
 					(unit 1)
 				)
@@
 		(dnp no)
 		(fields_autoplaced yes)
-		(property "Reference" "#PWR01908"
+		(property "Reference" "#PWR01208"
 			(at 218.44 168.91 0)
 			(effects
@@
 			(project "USB-SSB-txcvr"
 				(path "/8ae46c04-d01a-4756-8774-512b694bfaff/b2f84e19-834c-4e66-9c40-3d2adff3404a"
-					(reference "#PWR01908")
+					(reference "#PWR01208")
 					(unit 1)
 				)
@@
 		(on_board yes)
 		(dnp no)
-		(property "Reference" "C1908"
+		(property "Reference" "C1208"
 			(at 163.068 157.226 0)
 			(effects
@@
 			(project "USB-SSB-txcvr"
 				(path "/8ae46c04-d01a-4756-8774-512b694bfaff/b2f84e19-834c-4e66-9c40-3d2adff3404a"
-					(reference "C1908")
+					(reference "C1208")
 					(unit 1)
 				)
@@
 		(on_board yes)
 		(dnp no)
-		(property "Reference" "C1906"
+		(property "Reference" "C1206"
 			(at 154.178 60.96 90)
 			(effects
@@
 			(project "USB-SSB-txcvr"
 				(path "/8ae46c04-d01a-4756-8774-512b694bfaff/b2f84e19-834c-4e66-9c40-3d2adff3404a"
-					(reference "C1906")
+					(reference "C1206")
 					(unit 1)
 				)
@@
 		(dnp no)
 		(fields_autoplaced yes)
-		(property "Reference" "#PWR01904"
+		(property "Reference" "#PWR01204"
 			(at 147.32 101.6 0)
 			(effects
@@
 			(project ""
 				(path "/8ae46c04-d01a-4756-8774-512b694bfaff/b2f84e19-834c-4e66-9c40-3d2adff3404a"
-					(reference "#PWR01904")
+					(reference "#PWR01204")
 					(unit 1)
 				)
@@
 		(dnp no)
 		(fields_autoplaced yes)
-		(property "Reference" "#PWR01909"
+		(property "Reference" "#PWR01209"
 			(at 243.84 151.13 0)
 			(effects
@@
 			(project "USB-SSB-txcvr"
 				(path "/8ae46c04-d01a-4756-8774-512b694bfaff/b2f84e19-834c-4e66-9c40-3d2adff3404a"
-					(reference "#PWR01909")
+					(reference "#PWR01209")
 					(unit 1)
 				)
@@
 		(on_board yes)
 		(dnp no)
-		(property "Reference" "C1911"
+		(property "Reference" "C1211"
 			(at 202.184 157.734 0)
 			(effects
@@
 			(project ""
 				(path "/8ae46c04-d01a-4756-8774-512b694bfaff/b2f84e19-834c-4e66-9c40-3d2adff3404a"
-					(reference "C1911")
+					(reference "C1211")
 					(unit 1)
 				)
@@
 		(on_board yes)
 		(dnp no)
-		(property "Reference" "C1905"
+		(property "Reference" "C1205"
 			(at 154.178 55.88 90)
 			(effects
@@
 			(project ""
 				(path "/8ae46c04-d01a-4756-8774-512b694bfaff/b2f84e19-834c-4e66-9c40-3d2adff3404a"
-					(reference "C1905")
+					(reference "C1205")
 					(unit 1)
 				)
@@
 		(dnp no)
 		(fields_autoplaced yes)
-		(property "Reference" "#PWR01901"
+		(property "Reference" "#PWR01201"
 			(at 66.04 91.44 0)
 			(effects
@@
 			(project "USB-SSB-txcvr"
 				(path "/8ae46c04-d01a-4756-8774-512b694bfaff/b2f84e19-834c-4e66-9c40-3d2adff3404a"
-					(reference "#PWR01901")
+					(reference "#PWR01201")
 					(unit 1)
 				)
@@
 		(on_board yes)
 		(dnp no)
-		(property "Reference" "C1902"
+		(property "Reference" "C1202"
 			(at 143.002 58.42 90)
 			(effects
@@
 			(project "USB-SSB-txcvr"
 				(path "/8ae46c04-d01a-4756-8774-512b694bfaff/b2f84e19-834c-4e66-9c40-3d2adff3404a"
-					(reference "C1902")
+					(reference "C1202")
 					(unit 1)
 				)
@@
 		(on_board yes)
 		(dnp no)
-		(property "Reference" "C1912"
+		(property "Reference" "C1212"
 			(at 217.424 157.734 0)
 			(effects
@@
 			(project "USB-SSB-txcvr"
 				(path "/8ae46c04-d01a-4756-8774-512b694bfaff/b2f84e19-834c-4e66-9c40-3d2adff3404a"
-					(reference "C1912")
-					(unit 1)
-				)
+					(reference "C1212")
+					(unit 1)
+				)

Commit message: Tx LPF and its selection is pretty much done. Fix some OCD. Start to describe the design and construction.
Parts:
- renumbered C1201 to C501, C1202 to C502, C1203 to C503, C1204 to C504, C1205 to C505, C1206 to C506, C1207 to C507, C1208 to C508, C1209 to C509, C1210 to C510, C1211 to C511, C1212 to C512, C1213 to C513, C1214 to C514, C1215 to C515, U1201 to U501
Changed lines of the file:
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@@
 		(dnp no)
 		(fields_autoplaced yes)
-		(property "Reference" "#PWR01205"
+		(property "Reference" "#PWR0505"
 			(at 193.04 152.4 0)
 			(effects
@@
 			(project ""
 				(path "/8ae46c04-d01a-4756-8774-512b694bfaff/b2f84e19-834c-4e66-9c40-3d2adff3404a"
-					(reference "#PWR01205")
+					(reference "#PWR0505")
 					(unit 1)
 				)
@@
 		(on_board yes)
 		(dnp no)
-		(property "Reference" "C1215"
+		(property "Reference" "C515"
 			(at 252.476 157.48 0)
 			(effects
@@
 			(project "USB-SSB-txcvr"
 				(path "/8ae46c04-d01a-4756-8774-512b694bfaff/b2f84e19-834c-4e66-9c40-3d2adff3404a"
-					(reference "C1215")
+					(reference "C515")
 					(unit 1)
 				)
@@
 		(dnp no)
 		(fields_autoplaced yes)
-		(property "Reference" "#PWR01210"
+		(property "Reference" "#PWR0510"
 			(at 243.84 168.91 0)
 			(effects
@@
 			(project "USB-SSB-txcvr"
 				(path "/8ae46c04-d01a-4756-8774-512b694bfaff/b2f84e19-834c-4e66-9c40-3d2adff3404a"
-					(reference "#PWR01210")
+					(reference "#PWR0510")
 					(unit 1)
 				)
@@
 		(on_board yes)
 		(dnp no)
-		(property "Reference" "C1209"
+		(property "Reference" "C509"
 			(at 179.324 157.226 0)
 			(effects
@@
 			(project "USB-SSB-txcvr"
 				(path "/8ae46c04-d01a-4756-8774-512b694bfaff/b2f84e19-834c-4e66-9c40-3d2adff3404a"
-					(reference "C1209")
+					(reference "C509")
 					(unit 1)
 				)
@@
 		(on_board yes)
 		(dnp no)
-		(property "Reference" "#PWR01202"
+		(property "Reference" "#PWR0502"
 			(at 132.08 152.4 0)
 			(effects
@@
 			(project "USB-SSB-txcvr"
 				(path "/8ae46c04-d01a-4756-8774-512b694bfaff/b2f84e19-834c-4e66-9c40-3d2adff3404a"
-					(reference "#PWR01202")
+					(reference "#PWR0502")
 					(unit 1)
 				)
@@
 		(on_board yes)
 		(dnp no)
-		(property "Reference" "C1207"
+		(property "Reference" "C507"
 			(at 152.908 157.226 0)
 			(effects
@@
 			(project "USB-SSB-txcvr"
 				(path "/8ae46c04-d01a-4756-8774-512b694bfaff/b2f84e19-834c-4e66-9c40-3d2adff3404a"
-					(reference "C1207")
+					(reference "C507")
 					(unit 1)
 				)
@@
 		(on_board yes)
 		(dnp no)
-		(property "Reference" "C1214"
+		(property "Reference" "C514"
 			(at 242.824 157.734 0)
 			(effects
@@
 			(project "USB-SSB-txcvr"
 				(path "/8ae46c04-d01a-4756-8774-512b694bfaff/b2f84e19-834c-4e66-9c40-3d2adff3404a"
-					(reference "C1214")
+					(reference "C514")
 					(unit 1)
 				)
@@
 		(dnp no)
 		(fields_autoplaced yes)
-		(property "Reference" "#PWR01206"
+		(property "Reference" "#PWR0506"
 			(at 193.04 168.91 0)
 			(effects
@@
 			(project "USB-SSB-txcvr"
 				(path "/8ae46c04-d01a-4756-8774-512b694bfaff/b2f84e19-834c-4e66-9c40-3d2adff3404a"
-					(reference "#PWR01206")
+					(reference "#PWR0506")
 					(unit 1)
 				)
@@
 		(dnp no)
 		(fields_autoplaced yes)
-		(property "Reference" "#PWR01203"
+		(property "Reference" "#PWR0503"
 			(at 132.08 168.91 0)
 			(effects
@@
 			(project "USB-SSB-txcvr"
 				(path "/8ae46c04-d01a-4756-8774-512b694bfaff/b2f84e19-834c-4e66-9c40-3d2adff3404a"
-					(reference "#PWR01203")
+					(reference "#PWR0503")
 					(unit 1)
 				)
@@
 		(dnp no)
 		(fields_autoplaced yes)
-		(property "Reference" "#PWR01207"
+		(property "Reference" "#PWR0507"
 			(at 218.44 151.13 0)
 			(effects
@@
 			(project "USB-SSB-txcvr"
 				(path "/8ae46c04-d01a-4756-8774-512b694bfaff/b2f84e19-834c-4e66-9c40-3d2adff3404a"
-					(reference "#PWR01207")
+					(reference "#PWR0507")
 					(unit 1)
 				)
@@
 		(on_board yes)
 		(dnp no)
-		(property "Reference" "C1210"
+		(property "Reference" "C510"
 			(at 191.77 157.734 0)
 			(effects
@@
 			(project "USB-SSB-txcvr"
 				(path "/8ae46c04-d01a-4756-8774-512b694bfaff/b2f84e19-834c-4e66-9c40-3d2adff3404a"
-					(reference "C1210")
+					(reference "C510")
 					(unit 1)
 				)
@@
 		(on_board yes)
 		(dnp no)
-		(property "Reference" "U1201"
+		(property "Reference" "U501"
 			(at 76.962 39.116 0)
 			(effects
@@
 			(project ""
 				(path "/8ae46c04-d01a-4756-8774-512b694bfaff/b2f84e19-834c-4e66-9c40-3d2adff3404a"
-					(reference "U1201")
+					(reference "U501")
 					(unit 2)
 				)
@@
 		(on_board yes)
 		(dnp no)
-		(property "Reference" "C1203"
+		(property "Reference" "C503"
 			(at 143.002 63.5 90)
 			(effects
@@
 			(project "USB-SSB-txcvr"
 				(path "/8ae46c04-d01a-4756-8774-512b694bfaff/b2f84e19-834c-4e66-9c40-3d2adff3404a"
-					(reference "C1203")
+					(reference "C503")
 					(unit 1)
 				)
@@
 		(on_board yes)
 		(dnp no)
-		(property "Reference" "U1201"
+		(property "Reference" "U501"
 			(at 197.104 37.846 0)
 			(effects
@@
 			(project ""
 				(path "/8ae46c04-d01a-4756-8774-512b694bfaff/b2f84e19-834c-4e66-9c40-3d2adff3404a"
-					(reference "U1201")
+					(reference "U501")
 					(unit 1)
 				)
@@
 		(on_board yes)
 		(dnp no)
-		(property "Reference" "C1201"
+		(property "Reference" "C501"
 			(at 138.684 157.226 0)
 			(effects
@@
 			(project "USB-SSB-txcvr"
 				(path "/8ae46c04-d01a-4756-8774-512b694bfaff/b2f84e19-834c-4e66-9c40-3d2adff3404a"
-					(reference "C1201")
+					(reference "C501")
 					(unit 1)
 				)
@@
 		(on_board yes)
 		(dnp no)
-		(property "Reference" "C1213"
+		(property "Reference" "C513"
 			(at 227.076 157.48 0)
 			(effects
@@
 			(project "USB-SSB-txcvr"
 				(path "/8ae46c04-d01a-4756-8774-512b694bfaff/b2f84e19-834c-4e66-9c40-3d2adff3404a"
-					(reference "C1213")
+					(reference "C513")
 					(unit 1)
 				)
@@
 		(on_board yes)
 		(dnp no)
-		(property "Reference" "C1204"
+		(property "Reference" "C504"
 			(at 148.844 157.226 0)
 			(effects
@@
 			(project "USB-SSB-txcvr"
 				(path "/8ae46c04-d01a-4756-8774-512b694bfaff/b2f84e19-834c-4e66-9c40-3d2adff3404a"
-					(reference "C1204")
+					(reference "C504")
 					(unit 1)
 				)
@@
 		(dnp no)
 		(fields_autoplaced yes)
-		(property "Reference" "#PWR01208"
+		(property "Reference" "#PWR0508"
 			(at 218.44 168.91 0)
 			(effects
@@
 			(project "USB-SSB-txcvr"
 				(path "/8ae46c04-d01a-4756-8774-512b694bfaff/b2f84e19-834c-4e66-9c40-3d2adff3404a"
-					(reference "#PWR01208")
+					(reference "#PWR0508")
 					(unit 1)
 				)
@@
 		(on_board yes)
 		(dnp no)
-		(property "Reference" "C1208"
+		(property "Reference" "C508"
 			(at 163.068 157.226 0)
 			(effects
@@
 			(project "USB-SSB-txcvr"
 				(path "/8ae46c04-d01a-4756-8774-512b694bfaff/b2f84e19-834c-4e66-9c40-3d2adff3404a"
-					(reference "C1208")
+					(reference "C508")
 					(unit 1)
 				)
@@
 		(on_board yes)
 		(dnp no)
-		(property "Reference" "C1206"
+		(property "Reference" "C506"
 			(at 154.178 60.96 90)
 			(effects
@@
 			(project "USB-SSB-txcvr"
 				(path "/8ae46c04-d01a-4756-8774-512b694bfaff/b2f84e19-834c-4e66-9c40-3d2adff3404a"
-					(reference "C1206")
+					(reference "C506")
 					(unit 1)
 				)
@@
 		(dnp no)
 		(fields_autoplaced yes)
-		(property "Reference" "#PWR01204"
+		(property "Reference" "#PWR0504"
 			(at 147.32 101.6 0)
 			(effects
@@
 			(project ""
 				(path "/8ae46c04-d01a-4756-8774-512b694bfaff/b2f84e19-834c-4e66-9c40-3d2adff3404a"
-					(reference "#PWR01204")
+					(reference "#PWR0504")
 					(unit 1)
 				)
@@
 		(dnp no)
 		(fields_autoplaced yes)
-		(property "Reference" "#PWR01209"
+		(property "Reference" "#PWR0509"
 			(at 243.84 151.13 0)
 			(effects
@@
 			(project "USB-SSB-txcvr"
 				(path "/8ae46c04-d01a-4756-8774-512b694bfaff/b2f84e19-834c-4e66-9c40-3d2adff3404a"
-					(reference "#PWR01209")
+					(reference "#PWR0509")
 					(unit 1)
 				)
@@
 		(on_board yes)
 		(dnp no)
-		(property "Reference" "C1211"
+		(property "Reference" "C511"
 			(at 202.184 157.734 0)
 			(effects
@@
 			(project ""
 				(path "/8ae46c04-d01a-4756-8774-512b694bfaff/b2f84e19-834c-4e66-9c40-3d2adff3404a"
-					(reference "C1211")
+					(reference "C511")
 					(unit 1)
 				)
@@
 		(on_board yes)
 		(dnp no)
-		(property "Reference" "C1205"
+		(property "Reference" "C505"
 			(at 154.178 55.88 90)
 			(effects
@@
 			(project ""
 				(path "/8ae46c04-d01a-4756-8774-512b694bfaff/b2f84e19-834c-4e66-9c40-3d2adff3404a"
-					(reference "C1205")
+					(reference "C505")
 					(unit 1)
 				)
@@
 		(dnp no)
 		(fields_autoplaced yes)
-		(property "Reference" "#PWR01201"
+		(property "Reference" "#PWR0501"
 			(at 66.04 91.44 0)
 			(effects
@@
 			(project "USB-SSB-txcvr"
 				(path "/8ae46c04-d01a-4756-8774-512b694bfaff/b2f84e19-834c-4e66-9c40-3d2adff3404a"
-					(reference "#PWR01201")
+					(reference "#PWR0501")
 					(unit 1)
 				)
@@
 		(on_board yes)
 		(dnp no)
-		(property "Reference" "C1202"
+		(property "Reference" "C502"
 			(at 143.002 58.42 90)
 			(effects
@@
 			(project "USB-SSB-txcvr"
 				(path "/8ae46c04-d01a-4756-8774-512b694bfaff/b2f84e19-834c-4e66-9c40-3d2adff3404a"
-					(reference "C1202")
+					(reference "C502")
 					(unit 1)
 				)
@@
 		(on_board yes)
 		(dnp no)
-		(property "Reference" "C1212"
+		(property "Reference" "C512"
 			(at 217.424 157.734 0)
 			(effects
@@
 			(project "USB-SSB-txcvr"
 				(path "/8ae46c04-d01a-4756-8774-512b694bfaff/b2f84e19-834c-4e66-9c40-3d2adff3404a"
-					(reference "C1212")
-					(unit 1)
-				)
+					(reference "C512")
+					(unit 1)
+				)

Commit message: Embarking on a whole new arch for rx without BPFs and using a single digitally tuned tank plus three QSDs to accomplish image rejection in digital domain
Parts:
- C501, C502, C503, C504, C505, C506, C507, C508, C509, C510, C511, C512, C513, C514, C515: footprint (none) -> Capacitor_SMD:C_0805_2012Metric
- U501: footprint RHB32_3P45X3P45 -> (none)
Connections:
- net RxPCM is gone; now on net AudioDIN: U501.5 (DOUT)
- net AudioDIN: no longer U501.4 (DIN)
- net AudioWCLK: now reaches U501.3 (WCLK)
- no-connect marks 0 -> 1

Commit message: Converting to use busses as global symbols instead of tedium. Using 2n7002 Nexperia dual MOSFET because of its LOW LOW capacitance spec for L, C, and attenuator switching.
Connections:
- net AUDIOnRESET renamed reset
- net AudioBCLK renamed BCLK
- net AudioDIN renamed data
- net AudioMCLK renamed MCLK
- net AudioSCL renamed SCL
- net AudioSDA renamed SDA
- net AudioWCLK renamed WCLK
Other:
- title: DAC and ADC -> ADC

Commit message: LC tank for tx side is now switch C + switch L using reed relays. Rx preselector in flux but coming together
Parts:
- added IC501: AK5578EN, QFN50P900X900X100-65N, symbol AK5578EN:AK5578EN
Other:
- moved on the sheet: C501, C502, C503, C504, C505, C506, C507, C508, C509, C510, C511, C512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
