File: hw/DAC.kicad_sch (KiCad schematic)
At the start: 17 parts, among them IC501 AK5578EN, U501 TLV320AIC3104RHBR

Commit message: "Finished" the rx preselector with GaAs MESFET switches for C and L. Added diode protection clamp for the front end
Parts:
- renumbered C502 to C501, C503 to C502, C505 to C503, C506 to C504, C501 to C505, C504 to C506
Changed lines of the file:
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@@
 		(on_board yes)
 		(dnp no)
-		(property "Reference" "#PWR0502"
+		(property "Reference" "#PWR0503"
 			(at 21.59 184.15 0)
 			(effects
@@
 			(project "USB-SSB-txcvr"
 				(path "/8ae46c04-d01a-4756-8774-512b694bfaff/0ee31834-a2c3-474b-9f7c-c9b4f3cadb3f/6f6125da-73eb-482c-be1e-c27608407434"
-					(reference "#PWR01102")
+					(reference "#PWR01103")
 					(unit 1)
 				)
 				(path "/8ae46c04-d01a-4756-8774-512b694bfaff/0ee31834-a2c3-474b-9f7c-c9b4f3cadb3f/7dc5e910-3f5d-4e38-885c-c6c1fd22d44b"
-					(reference "#PWR01202")
+					(reference "#PWR01203")
 					(unit 1)
 				)
 				(path "/8ae46c04-d01a-4756-8774-512b694bfaff/0ee31834-a2c3-474b-9f7c-c9b4f3cadb3f/ffbf7dd2-d900-47c5-8239-8fcdef3c063e"
-					(reference "#PWR0502")
+					(reference "#PWR0503")
 					(unit 1)
 				)
@@
 		(dnp no)
 		(fields_autoplaced yes)
-		(property "Reference" "#PWR0503"
+		(property "Reference" "#PWR0504"
 			(at 21.59 200.66 0)
 			(effects
@@
 			(project "USB-SSB-txcvr"
 				(path "/8ae46c04-d01a-4756-8774-512b694bfaff/0ee31834-a2c3-474b-9f7c-c9b4f3cadb3f/6f6125da-73eb-482c-be1e-c27608407434"
-					(reference "#PWR01103")
+					(reference "#PWR01104")
 					(unit 1)
 				)
 				(path "/8ae46c04-d01a-4756-8774-512b694bfaff/0ee31834-a2c3-474b-9f7c-c9b4f3cadb3f/7dc5e910-3f5d-4e38-885c-c6c1fd22d44b"
-					(reference "#PWR01203")
+					(reference "#PWR01204")
 					(unit 1)
 				)
 				(path "/8ae46c04-d01a-4756-8774-512b694bfaff/0ee31834-a2c3-474b-9f7c-c9b4f3cadb3f/ffbf7dd2-d900-47c5-8239-8fcdef3c063e"
-					(reference "#PWR0503")
+					(reference "#PWR0504")
 					(unit 1)
 				)
@@
 		(on_board yes)
 		(dnp no)
-		(property "Reference" "C503"
+		(property "Reference" "C502"
 			(at -155.448 68.58 90)
 			(effects
@@
 			(project "USB-SSB-txcvr"
 				(path "/8ae46c04-d01a-4756-8774-512b694bfaff/0ee31834-a2c3-474b-9f7c-c9b4f3cadb3f/6f6125da-73eb-482c-be1e-c27608407434"
-					(reference "C1103")
+					(reference "C1102")
 					(unit 1)
 				)
 				(path "/8ae46c04-d01a-4756-8774-512b694bfaff/0ee31834-a2c3-474b-9f7c-c9b4f3cadb3f/7dc5e910-3f5d-4e38-885c-c6c1fd22d44b"
-					(reference "C1203")
+					(reference "C1202")
 					(unit 1)
 				)
 				(path "/8ae46c04-d01a-4756-8774-512b694bfaff/0ee31834-a2c3-474b-9f7c-c9b4f3cadb3f/ffbf7dd2-d900-47c5-8239-8fcdef3c063e"
-					(reference "C503")
+					(reference "C502")
 					(unit 1)
 				)
@@
 		(on_board yes)
 		(dnp no)
-		(property "Reference" "C501"
+		(property "Reference" "C505"
 			(at 28.194 188.976 0)
 			(effects
@@
 			(project "USB-SSB-txcvr"
 				(path "/8ae46c04-d01a-4756-8774-512b694bfaff/0ee31834-a2c3-474b-9f7c-c9b4f3cadb3f/6f6125da-73eb-482c-be1e-c27608407434"
-					(reference "C1101")
+					(reference "C1105")
 					(unit 1)
 				)
 				(path "/8ae46c04-d01a-4756-8774-512b694bfaff/0ee31834-a2c3-474b-9f7c-c9b4f3cadb3f/7dc5e910-3f5d-4e38-885c-c6c1fd22d44b"
-					(reference "C1201")
+					(reference "C1205")
 					(unit 1)
 				)
 				(path "/8ae46c04-d01a-4756-8774-512b694bfaff/0ee31834-a2c3-474b-9f7c-c9b4f3cadb3f/ffbf7dd2-d900-47c5-8239-8fcdef3c063e"
-					(reference "C501")
+					(reference "C505")
 					(unit 1)
 				)
@@
 		(on_board yes)
 		(dnp no)
-		(property "Reference" "C504"
+		(property "Reference" "C506"
 			(at 38.354 188.976 0)
 			(effects
@@
 			(project "USB-SSB-txcvr"
 				(path "/8ae46c04-d01a-4756-8774-512b694bfaff/0ee31834-a2c3-474b-9f7c-c9b4f3cadb3f/6f6125da-73eb-482c-be1e-c27608407434"
-					(reference "C1104")
+					(reference "C1106")
 					(unit 1)
 				)
 				(path "/8ae46c04-d01a-4756-8774-512b694bfaff/0ee31834-a2c3-474b-9f7c-c9b4f3cadb3f/7dc5e910-3f5d-4e38-885c-c6c1fd22d44b"
-					(reference "C1204")
+					(reference "C1206")
 					(unit 1)
 				)
 				(path "/8ae46c04-d01a-4756-8774-512b694bfaff/0ee31834-a2c3-474b-9f7c-c9b4f3cadb3f/ffbf7dd2-d900-47c5-8239-8fcdef3c063e"
-					(reference "C504")
+					(reference "C506")
 					(unit 1)
 				)
@@
 		(on_board yes)
 		(dnp no)
-		(property "Reference" "C506"
+		(property "Reference" "C504"
 			(at -144.272 66.04 90)
 			(effects
@@
 			(project "USB-SSB-txcvr"
 				(path "/8ae46c04-d01a-4756-8774-512b694bfaff/0ee31834-a2c3-474b-9f7c-c9b4f3cadb3f/6f6125da-73eb-482c-be1e-c27608407434"
-					(reference "C1106")
+					(reference "C1104")
 					(unit 1)
 				)
 				(path "/8ae46c04-d01a-4756-8774-512b694bfaff/0ee31834-a2c3-474b-9f7c-c9b4f3cadb3f/7dc5e910-3f5d-4e38-885c-c6c1fd22d44b"
-					(reference "C1206")
+					(reference "C1204")
 					(unit 1)
 				)
 				(path "/8ae46c04-d01a-4756-8774-512b694bfaff/0ee31834-a2c3-474b-9f7c-c9b4f3cadb3f/ffbf7dd2-d900-47c5-8239-8fcdef3c063e"
-					(reference "C506")
+					(reference "C504")
 					(unit 1)
 				)
@@
 		(dnp no)
 		(fields_autoplaced yes)
-		(property "Reference" "#PWR0504"
+		(property "Reference" "#PWR0502"
 			(at -160.02 93.98 0)
 			(effects
@@
 			(project "USB-SSB-txcvr"
 				(path "/8ae46c04-d01a-4756-8774-512b694bfaff/0ee31834-a2c3-474b-9f7c-c9b4f3cadb3f/6f6125da-73eb-482c-be1e-c27608407434"
-					(reference "#PWR01104")
+					(reference "#PWR01102")
 					(unit 1)
 				)
 				(path "/8ae46c04-d01a-4756-8774-512b694bfaff/0ee31834-a2c3-474b-9f7c-c9b4f3cadb3f/7dc5e910-3f5d-4e38-885c-c6c1fd22d44b"
-					(reference "#PWR01204")
+					(reference "#PWR01202")
 					(unit 1)
 				)
 				(path "/8ae46c04-d01a-4756-8774-512b694bfaff/0ee31834-a2c3-474b-9f7c-c9b4f3cadb3f/ffbf7dd2-d900-47c5-8239-8fcdef3c063e"
-					(reference "#PWR0504")
+					(reference "#PWR0502")
 					(unit 1)
 				)
@@
 		(on_board yes)
 		(dnp no)
-		(property "Reference" "C505"
+		(property "Reference" "C503"
 			(at -144.272 60.96 90)
 			(effects
@@
 			(project "USB-SSB-txcvr"
 				(path "/8ae46c04-d01a-4756-8774-512b694bfaff/0ee31834-a2c3-474b-9f7c-c9b4f3cadb3f/6f6125da-73eb-482c-be1e-c27608407434"
-					(reference "C1105")
+					(reference "C1103")
 					(unit 1)
 				)
 				(path "/8ae46c04-d01a-4756-8774-512b694bfaff/0ee31834-a2c3-474b-9f7c-c9b4f3cadb3f/7dc5e910-3f5d-4e38-885c-c6c1fd22d44b"
-					(reference "C1205")
+					(reference "C1203")
 					(unit 1)
 				)
 				(path "/8ae46c04-d01a-4756-8774-512b694bfaff/0ee31834-a2c3-474b-9f7c-c9b4f3cadb3f/ffbf7dd2-d900-47c5-8239-8fcdef3c063e"
-					(reference "C505")
+					(reference "C503")
 					(unit 1)
 				)
@@
 		(on_board yes)
 		(dnp no)
-		(property "Reference" "C502"
+		(property "Reference" "C501"
 			(at -155.448 63.5 90)
 			(effects
@@
 			(project "USB-SSB-txcvr"
 				(path "/8ae46c04-d01a-4756-8774-512b694bfaff/0ee31834-a2c3-474b-9f7c-c9b4f3cadb3f/6f6125da-73eb-482c-be1e-c27608407434"
-					(reference "C1102")
+					(reference "C1101")
 					(unit 1)
 				)
 				(path "/8ae46c04-d01a-4756-8774-512b694bfaff/0ee31834-a2c3-474b-9f7c-c9b4f3cadb3f/7dc5e910-3f5d-4e38-885c-c6c1fd22d44b"
-					(reference "C1202")
+					(reference "C1201")
 					(unit 1)
 				)
 				(path "/8ae46c04-d01a-4756-8774-512b694bfaff/0ee31834-a2c3-474b-9f7c-c9b4f3cadb3f/ffbf7dd2-d900-47c5-8239-8fcdef3c063e"
-					(reference "C502")
-					(unit 1)
-				)
+					(reference "C501")
+					(unit 1)
+				)

Commit message: More Tx LPF design and a doc. The schematic now reflects 200 ohm domain for the LPFs and the PA LC tanks too.
Parts:
- removed U501: TLV320AIC3104RHBR, symbol TLV320AIC3104:HPA01211RHBR
- added R501: 47, symbol Device:R_US
- C501, C503: value .1uF -> 0.1uF; footprint Capacitor_SMD:C_0805_2012Metric -> (none)
- C502, C504: value .1uF -> 4.7uF; footprint Capacitor_SMD:C_0805_2012Metric -> (none)
- C505, C506: value 1uF -> 10uF
- C507: value 0.1uF -> 10uF
- C509: value 10uF -> 0.1uF
- C514: value 1uF -> 0.1uF
Connections:
- net +1.8V is gone; now on net VREF: C514.1, C515.1
- net RxIn is gone; now on net GND: C503.1
- net RxIp is gone; now on net GND: C501.1
- net RxQn is gone; now on net GND: C504.1
- net RxQp is gone; now on net GND: C502.1
- net +3.3V: now also C503.2, C504.2, IC501.25 (TVDD), IC501.30 (PW1), IC501.31 (PW2), IC501.32 (MSN), IC501.54 (I2C), IC501.57 (LDOE), IC501.58 (ODP)
- net +3.3VA: now also IC501.15 (AVDD2), IC501.2 (AVDD1), R501.1; no longer C507.1, C508.1, C509.1
- net GND: now also IC501.1 (AVSS1), IC501.10 (AIN5N), IC501.12 (VREFL3), IC501.13 (AIN6N), IC501.16 (AVSS2), IC501.20 (VREFL4), IC501.26 (DVSS), IC501.29 (PW0), IC501.4 (AIN3N), IC501.44 (CKS1/CAD0_I2C/CSN), IC501.46 (CKS3/CAD1), IC501.47 (SLOW/DCKB), IC501.48 (SD/PMOD), IC501.49 (DIF0/DSDSEL0), IC501.5 (VREFL2), IC501.50 (DIF1/DSDSEL1), IC501.53 (PSN/CAD0_SP1), IC501.55 (DP), IC501.56 (DCKS/HPFE), IC501.60 (AIN1N), IC501.61 (VREFL1), IC501.63 (AIN2N), IC501.65 (THERMAL_PAD), IC501.7 (AIN4N)
- net VREF: now reaches IC501.11 (VREFH3)
- net VREF: now also C507.1, C508.1, C509.1, IC501.19 (VREFH4), IC501.6 (VREFH2), IC501.62 (VREFH1), R501.2
- net RxQ2p: now reaches IC501.14 (AIN6P)
- net QSD.MCLK: now reaches IC501.24 (MCLK)
- net at IC501.27 (VDD18): now also C501.2, C502.2
- net QSD.reset: now reaches IC501.28 (PDN)
- net RxI1p: now reaches IC501.3 (AIN3P)
- net QSD.BCLK: now reaches IC501.33 (BICK/DCLK)
- net QSD.WCLK: now reaches IC501.34 (LRCK/DSDOL1)
- net QSD.SDA0: now reaches IC501.43 (CKS0/SDA/CDTI)
- net QSD.SCL0: now reaches IC501.45 (CKS2/SCL/CCLK)
- net RxI0p: now reaches IC501.59 (AIN1P)
- net RxQ0p: now reaches IC501.64 (AIN2P)
- net RxQ1p: now reaches IC501.8 (AIN4P)
- net RxI2p: now reaches IC501.9 (AIN5P)
- no-connect marks 1 -> 10
Other:
- note added: "power ch1-6"
