File: hw/ethernet.kicad_sch (KiCad schematic)
At the start: 37 parts, among them J2301 RJ45_Abracon_ARJP11A-MASA-B-A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, U2301 LAN8742A, U2302 USBLC6-4SC6, Y2301 ECS-250-8-37B2-RWN

Commit message: Starting to switch to new rx architecture
Parts:
- renumbered C2301 to C2501, C2302 to C2502, C2303 to C2503, C2304 to C2504, C2305 to C2505, C2306 to C2506, C2307 to C2507, C2308 to C2508, C2309 to C2509, C2310 to C2510, C2311 to C2511, C2312 to C2512, FB2301 to FB2501, J2301 to J2501, R2301 to R2501, R2302 to R2502, R2303 to R2503, R2304 to R2504, R2305 to R2505, R2306 to R2506, R2307 to R2507, R2308 to R2508, R2309 to R2509, R2310 to R2510, R2311 to R2511, R2312 to R2512, R2313 to R2513, R2314 to R2514, R2315 to R2515, R2316 to R2516, R2317 to R2517, R2318 to R2518, R2319 to R2519, R2320 to R2520, U2301 to U2501, U2302 to U2502, Y2301 to Y2501

Commit message: Converting to use busses as global symbols instead of tedium. Using 2n7002 Nexperia dual MOSFET because of its LOW LOW capacitance spec for L, C, and attenuator switching.
Parts:
- renumbered C2501 to C2201, C2502 to C2202, C2503 to C2203, C2504 to C2204, C2505 to C2205, C2506 to C2206, C2507 to C2207, C2508 to C2208, C2509 to C2209, C2510 to C2210, C2511 to C2211, C2512 to C2212, FB2501 to FB2201, J2501 to J2201, R2501 to R2201, R2502 to R2202, R2503 to R2203, R2504 to R2204, R2505 to R2205, R2506 to R2206, R2507 to R2207, R2508 to R2208, R2509 to R2209, R2510 to R2210, R2511 to R2211, R2512 to R2212, R2513 to R2213, R2514 to R2214, R2515 to R2215, R2516 to R2216, R2517 to R2217, R2518 to R2218, R2519 to R2219, R2520 to R2220, U2501 to U2201, U2502 to U2202, Y2501 to Y2201

Commit message: Moved ant page into tx page, added Bruene Direction Coupler to measure VSWR. General cleanup, page renumber, reannote
Parts:
- renumbered C2201 to C1901, C2202 to C1902, C2203 to C1903, C2204 to C1904, C2205 to C1905, C2206 to C1906, C2207 to C1907, C2208 to C1908, C2209 to C1909, C2210 to C1910, C2211 to C1911, C2212 to C1912, FB2201 to FB1901, J2201 to J1901, R2201 to R1901, R2202 to R1902, R2203 to R1903, R2204 to R1904, R2205 to R1905, R2206 to R1906, R2207 to R1907, R2208 to R1908, R2209 to R1909, R2210 to R1910, R2211 to R1911, R2212 to R1912, R2213 to R1913, R2214 to R1914, R2215 to R1915, R2216 to R1916, R2217 to R1917, R2218 to R1918, R2219 to R1919, R2220 to R1920, U2201 to U1901, U2202 to U1902, Y2201 to Y1901

Commit message: Removed USB data, SD card. Added USB-PD (not complete yet). Added SPI display.
Parts:
- renumbered C1901 to C1801, C1902 to C1802, C1903 to C1803, C1904 to C1804, C1905 to C1805, C1906 to C1806, C1907 to C1807, C1908 to C1808, C1909 to C1809, C1910 to C1810, C1911 to C1811, C1912 to C1812, FB1901 to FB1801, J1901 to J1801, R1901 to R1801, R1902 to R1802, R1903 to R1803, R1904 to R1804, R1905 to R1805, R1906 to R1806, R1907 to R1807, R1908 to R1808, R1909 to R1809, R1910 to R1810, R1911 to R1811, R1912 to R1812, R1913 to R1813, R1914 to R1814, R1915 to R1815, R1916 to R1816, R1917 to R1817, R1918 to R1818, R1919 to R1819, R1920 to R1820, U1901 to U1801, U1902 to U1802, Y1901 to Y1801

Commit message: "Final" rx preselector design for good digital tuning in 800 ohm domain and general 1MHz..30MHz coverage
Parts:
- renumbered C1801 to C1901, C1802 to C1902, C1803 to C1903, C1804 to C1904, C1805 to C1905, C1806 to C1906, C1807 to C1907, C1808 to C1908, C1809 to C1909, C1810 to C1910, C1811 to C1911, C1812 to C1912, FB1801 to FB1901, J1801 to J1901, R1801 to R1901, R1802 to R1902, R1803 to R1903, R1804 to R1904, R1805 to R1905, R1806 to R1906, R1807 to R1907, R1808 to R1908, R1809 to R1909, R1810 to R1910, R1811 to R1911, R1812 to R1912, R1813 to R1913, R1814 to R1914, R1815 to R1915, R1816 to R1916, R1817 to R1917, R1818 to R1918, R1819 to R1919, R1820 to R1920, U1801 to U1901, U1802 to U1902, Y1801 to Y1901

Commit message: USB-PD now "done". Veer power cleaned up a bit. Working voltage increased for caps that need it. Power sequencing for FPGA handled. Analog rails now come from separate buck + (quiet) LDO for each. Starting on digital antenna tuner design.
Parts:
- renumbered C1901 to C2001, C1902 to C2002, C1903 to C2003, C1904 to C2004, C1905 to C2005, C1906 to C2006, C1907 to C2007, C1908 to C2008, C1909 to C2009, C1910 to C2010, C1911 to C2011, C1912 to C2012, FB1901 to FB2001, J1901 to J2001, R1901 to R2001, R1902 to R2002, R1903 to R2003, R1904 to R2004, R1905 to R2005, R1906 to R2006, R1907 to R2007, R1908 to R2008, R1909 to R2009, R1910 to R2010, R1911 to R2011, R1912 to R2012, R1913 to R2013, R1914 to R2014, R1915 to R2015, R1916 to R2016, R1917 to R2017, R1918 to R2018, R1919 to R2019, R1920 to R2020, U1901 to U2001, U1902 to U2002, Y1901 to Y2001

Commit message: Ready for first schematic review with Claude.ai
Parts:
- renumbered C2001 to C2201, C2002 to C2202, C2003 to C2203, C2004 to C2204, C2005 to C2205, C2006 to C2206, C2007 to C2207, C2008 to C2208, C2009 to C2209, C2010 to C2210, C2011 to C2211, C2012 to C2212, FB2001 to FB2201, J2001 to J2201, R2001 to R2201, R2002 to R2202, R2003 to R2203, R2004 to R2204, R2005 to R2205, R2006 to R2206, R2007 to R2207, R2008 to R2208, R2009 to R2209, R2010 to R2210, R2011 to R2211, R2012 to R2212, R2013 to R2213, R2014 to R2214, R2015 to R2215, R2016 to R2216, R2017 to R2217, R2018 to R2218, R2019 to R2219, R2020 to R2220, U2001 to U2201, U2002 to U2202, Y2001 to Y2201
Other:
- company: (none) -> WB7NAB
- title: (none) -> Ethernet

Commit message: Revamp the rx preselector to achieve general coverage from 1MHz to 30MHz with overlapping bands
Parts:
- renumbered C2201 to C2401, C2202 to C2402, C2203 to C2403, C2204 to C2404, C2205 to C2405, C2206 to C2406, C2207 to C2407, C2208 to C2408, C2209 to C2409, C2210 to C2410, C2211 to C2411, C2212 to C2412, FB2201 to FB2401, J2201 to J2401, R2201 to R2401, R2202 to R2402, R2203 to R2403, R2204 to R2404, R2205 to R2405, R2206 to R2406, R2207 to R2407, R2208 to R2408, R2209 to R2409, R2210 to R2410, R2211 to R2411, R2212 to R2412, R2213 to R2413, R2214 to R2414, R2215 to R2415, R2216 to R2416, R2217 to R2417, R2218 to R2418, R2219 to R2419, R2220 to R2420, U2201 to U2401, U2202 to U2402, Y2201 to Y2401
