File: hw/USB-SSB-txcvr.kicad_pcb (KiCad board)
At the start: 6 copper layers, 200 x 150 mm, 456 parts, among them IC1001 AS169-73LF, IC1002 MC74HC1G04DFT2G-Q, IC1101 AS169-73LF, IC1102 MC74HC1G04DFT2G-Q, IC1201 AS169-73LF, IC1202 MC74HC1G04DFT2G-Q, IC1301 AS169-73LF, IC1302 MC74HC1G04DFT2G-Q, IC1401 AS169-73LF, IC1402 MC74HC1G04DFT2G-Q, IC1501 AS169-73LF, IC1502 MC74HC1G04DFT2G-Q, IC1601 AS169-73LF, IC1602 MC74HC1G04DFT2G-Q, IC1701 AS169-73LF, IC1702 MC74HC1G04DFT2G-Q, IC2001 TPL7407LADR, IC2101 TPL7407LADR, IC2102 TPL7407LADR, IC801 AS169-73LF, IC802 MC74HC1G04DFT2G-Q, IC901 AS169-73LF, IC902 MC74HC1G04DFT2G-Q, J2301 RJ45_Abracon_ARJP11A-MASA-B-A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, J2401 MSD-1-A, J602 USB4216-03-A, J701 Conn_Coaxial_Power, K2001 G2RL-1A, K2002 G2RL-1A, K2003 G2RL-1A, K2101 G5V-2_Split, K2102 G5V-2_Split, K2103 G5V-2_Split, K2104 G5V-2_Split, K2105 G5V-2_Split, K2106 G5V-2_Split, K2107 G5V-2_Split, K2108 G5V-2_Split, K701 G5Q-1, Q1901 CSD18543Q3A, Q1902 CSD18543Q3A, Q1903 CSD18543Q3A, Q1904 CSD18543Q3A, Q2001 2N7002, Q2002 2N7002, Q2003 2N7002, Q2004 2N7002, Q2005 2N7002, Q2006 2N7002, Q2007 2N7002, Q2008 2N7002, Q2009 2N7002, Q2010 2N7002, Q601 CSD18543Q3A, U1801 TPS7A2012DQN, U1802 TPS22917LDBV, U1803 TPS7A2033DQN, U1804 LMR51430XDDCR, U1805 LMR51430XDDCR, U1901 LM34936RHFR, U1902 TLV9062xD, U201 STM32H753ZIT6, U2201 ICE40UP5K-SG48ITR, U2301 LAN8742A, U2302 USBLC6-4SC6, U2401 CM1624, U401 UCC27511ADBV, Y202 ECS-2033-250-BN, Y2301 ECS-250-8-37B2-RWN

Commit message: All footprints assigned at least on trial basis.
Parts:
- removed C1001, C1002, C1101, C1102, C1906, C1908, C2202, C2303, C2307, C2308, C2309, C2310, C2311, C507, C508, C511, C513, C515, C801, C802, C901, C902: 0.1uF, Capacitor_SMD:C_0805_2012Metric
- removed C1003, C1013, C904, C912: 330pF, Capacitor_SMD:C_0805_2012Metric
- removed C1004, C1006, C1010, C1012: 200pF, Capacitor_SMD:C_0805_2012Metric
- removed C1005, C1008, C1011: 2400pF, Capacitor_SMD:C_0805_2012Metric
- removed C1007, C1103, C1113, C804, C812: 180pF, Capacitor_SMD:C_0805_2012Metric
- removed C1104, C1107, C1112: 82pF, Capacitor_SMD:C_0805_2012Metric
- removed C1105, C1108, C1111: 1300pF, Capacitor_SMD:C_0805_2012Metric
- removed C1106, C1110: 91pF, Capacitor_SMD:C_0805_2012Metric
- removed C1706, C1710: 24pF, Capacitor_SMD:C_0805_2012Metric
- removed C1707, C1712, C1905: 27pF, Capacitor_SMD:C_0805_2012Metric
- removed C1708: 510pF, Capacitor_SMD:C_0805_2012Metric
- removed C1711, C906, C910: 560pF, Capacitor_SMD:C_0805_2012Metric
- removed C1713: 47pF, Capacitor_SMD:C_0805_2012Metric
- removed C1901: 10pF, Capacitor_SMD:C_0805_2012Metric
- removed C1902: 470pF, Capacitor_SMD:C_0805_2012Metric
- removed C1903: 47nF, Capacitor_SMD:C_0805_2012Metric
- removed C1904: 1.2nF, Capacitor_SMD:C_0805_2012Metric
- removed C1907, C807, C903, C913: 820pF, Capacitor_SMD:C_0805_2012Metric
- removed C1909, C2203, C2205, C2206, C2209, C2211: 4.7uF, Capacitor_SMD:C_0805_2012Metric
- removed C1910, C1911: 0.47uF, Capacitor_SMD:C_0805_2012Metric
- removed C1912: 68uF 50V, Library:EEH-ZA1H680P
- removed C1913, C1914: 1uF 50V, Capacitor_SMD:C_1206_3216Metric
- removed C1915: 1nF, Capacitor_SMD:C_0805_2012Metric
- removed C1916, C1917, C1918, C1919, C1920: 10uF 50V, Capacitor_SMD:C_1206_3216Metric
- removed C2118, C2130: 649pF, Capacitor_SMD:C_1206_3216Metric
- removed C2119: 442pF, Capacitor_SMD:C_1206_3216Metric
- removed C2120: 422pF, Capacitor_SMD:C_1206_3216Metric
- removed C2121: 140pF, Capacitor_SMD:C_1206_3216Metric
- removed C2122: 105pF, Capacitor_SMD:C_1206_3216Metric
- removed C2123, C2124: 301pF, Capacitor_SMD:C_1206_3216Metric
- removed C2125, C2136: 56.2pF, Capacitor_SMD:C_0805_2012Metric
- removed C2126: 19.6pF, Capacitor_SMD:C_0805_2012Metric
- removed C2127: 14pF, Capacitor_SMD:C_0805_2012Metric
- removed C2128, C2129, C2137: 40.2pF, Capacitor_SMD:C_0805_2012Metric
- removed C2131: 226pF, Capacitor_SMD:C_1206_3216Metric
- removed C2132, C2135: 162pF, Capacitor_SMD:C_1206_3216Metric
- removed C2133, C2134: 487pF, Capacitor_SMD:C_1206_3216Metric
- removed C2138, C2139, C2141: 115pF, Capacitor_SMD:C_1206_3216Metric
- removed C2140: 332pF, Capacitor_SMD:C_1206_3216Metric
- removed C2142: 82.5pF, Capacitor_SMD:C_1206_3216Metric
- removed C2143, C2144: 237pF, Capacitor_SMD:C_1206_3216Metric
- removed C2201, C2304, C510, C512, C514: 1uF, Capacitor_SMD:C_0805_2012Metric
- removed C2204, C2207, C2208, C2210, C2212: .1uF, Capacitor_SMD:C_0805_2012Metric
- removed C226: 2.2uF, Capacitor_SMD:C_0805_2012Metric
- removed C2301, C2302: 8.2pF, Capacitor_SMD:C_0603_1608Metric
- removed C2305: 470pF, Capacitor_SMD:C_1206_3216Metric
- removed C2306, C509: 10uF, Capacitor_SMD:C_0805_2012Metric
- removed C2312, C806, C810: 1000pF, Capacitor_SMD:C_0805_2012Metric
- removed C803, C813: 1500pF, Capacitor_SMD:C_0805_2012Metric
- removed C805, C808, C811: 11nF, Capacitor_SMD:C_0805_2012Metric
- removed C905, C908, C911: 4700pF, Capacitor_SMD:C_0805_2012Metric
- removed C907: 68pF, Capacitor_SMD:C_0805_2012Metric
- removed D1801: PMEG45T15EPD, Package_TO_SOT_SMD:Nexperia_CFP15_SOT-1289
- removed D2002, D2003, D2004, D2005, D2006, D2007, D2008, D2009, D2010: SMP1302-079LF, Library:SC-79
- removed FB2301: BLM21AG102SN1D, Inductor_SMD:L_0805_2012Metric
- removed IC1001, IC1101, IC1201, IC1301, IC1401, IC1501, IC1601, IC1701, IC801, IC901: AS169-73LF, Library:SOT-6
- removed IC1002, IC1102, IC1202, IC1302, IC1402, IC1502, IC1602, IC1702, IC802, IC902: MC74HC1G04DFT2G-Q, Package_TO_SOT_SMD:SOT-353_SC-70-5
- removed IC2001, IC2101, IC2102: TPL7407LADR, Package_SO:JEITA_SOIC-16_3.9x9.9mm_P1.27mm
- removed J2301: RJ45_Abracon_ARJP11A-MASA-B-A-EMU2, Connector_RJ:RJ45_Abracon_ARJP11A-MA_Horizontal
- removed J602: USB4216-03-A, Library:USB421603A
- removed J701: Conn_Coaxial_Power, Connector_Coaxial:SMA_Amphenol_132289_EdgeMount
- removed K2001, K2002, K2003: G2RL-1A, Relay_THT:Relay_SPST_Omron_G2RL-1A
- removed L1901: 6.8uH, Library:Bourns PQ2614BLA-6R8K
- removed L2002, L2003, L2004, L2005, L2007, L2009, L2011, L2012, L2013, L2014, L2015: 2.2uH, Inductor_SMD:L_0805_2012Metric
- removed L2006: 500nH, Inductor_SMD:L_0805_2012Metric
- removed L2008: 300nH, Inductor_SMD:L_0805_2012Metric
- removed L2010: 82nH, Inductor_SMD:L_0805_2012Metric
- removed Q1901, Q1902, Q1903, Q1904, Q601: CSD18543Q3A, Package_SON:VSON-8_3.3x3.3mm_P0.65mm_NexFET
- removed Q2006, Q2007, Q2008, Q2009, Q2010: 2N7002, Package_TO_SOT_SMD:SOT-23
- removed R1901, R1902: 15K, Resistor_SMD:R_0603_1608Metric
- removed R1903, R1905, R1907, R1908, R1909, R1910, R1912, R1913: 10k, Resistor_SMD:R_0603_1608Metric
- removed R1904: 93.1k, Resistor_SMD:R_0603_1608Metric
- removed R1906, R1911: 66.5k, Resistor_SMD:R_0603_1608Metric
- removed R1914: 100, Resistor_SMD:R_0603_1608Metric
- removed R1915: 0.008, Library:KRL3216T4AMR008FT1
- removed R402: 500k, Resistor_SMD:R_0603_1608Metric
- removed U1901: LM34936RHFR, symbols:RHF0028A
- removed U1902: TLV9062xD, Package_SO:SOIC-8_3.9x4.9mm_P1.27mm
- removed U2201: ICE40UP5K-SG48ITR, Package_DFN_QFN:QFN-48-1EP_7x7mm_P0.5mm_EP5.6x5.6mm
- removed U2301: LAN8742A, Package_DFN_QFN:VQFN-24-1EP_4x4mm_P0.5mm_EP2.5x2.5mm_ThermalVias
- removed U2302: USBLC6-4SC6, Package_TO_SOT_SMD:SOT-23-6
- removed Y202: ECS-2033-250-BN, symbols:ECS2033250BN
- removed Y2301: ECS-250-8-37B2-RWN, symbols:ECS2033250BN
- added C1209: 1uF, Capacitor_SMD:C_0805_2012Metric, F.Cu at (-56.9, 140.6)
- added C1214: 0.1uF, Capacitor_SMD:C_0805_2012Metric, F.Cu at (-56.9, 143.6)
- added C1215: 0.1uF, Capacitor_SMD:C_0805_2012Metric, F.Cu at (-56.9, 146.6)
- added C1216: 2.2uF, Capacitor_SMD:C_1206_3216Metric, F.Cu at (-69.5, 130.7)
- added C1217: 3.3nF, Capacitor_SMD:C_1206_3216Metric, F.Cu at (-69.5, 134.0)
- added C1218: 3.3nF, Capacitor_SMD:C_1206_3216Metric, F.Cu at (-69.5, 137.4)
- added C1219: 3.3nF, Capacitor_SMD:C_1206_3216Metric, F.Cu at (-69.5, 140.7)
- added C1220: 3.3nF, Capacitor_SMD:C_1206_3216Metric, F.Cu at (-69.5, 144.1)
- added C1309: 1uF, Capacitor_SMD:C_0805_2012Metric, F.Cu at (-56.9, 117.4)
- added C1314: 0.1uF, Capacitor_SMD:C_0805_2012Metric, F.Cu at (-56.9, 120.4)
- added C1315: 0.1uF, Capacitor_SMD:C_0805_2012Metric, F.Cu at (-56.9, 123.4)
- added C1316: 2.2uF, Capacitor_SMD:C_1206_3216Metric, F.Cu at (-69.5, 107.5)
- added C1317: 3.3nF, Capacitor_SMD:C_1206_3216Metric, F.Cu at (-69.5, 110.8)
- added C1318: 3.3nF, Capacitor_SMD:C_1206_3216Metric, F.Cu at (-69.5, 114.2)
- added C1319: 3.3nF, Capacitor_SMD:C_1206_3216Metric, F.Cu at (-69.5, 117.5)
- added C1320: 3.3nF, Capacitor_SMD:C_1206_3216Metric, F.Cu at (-69.5, 120.9)
- added C1409: 1uF, Capacitor_SMD:C_0805_2012Metric, F.Cu at (-70.2, 179.5)
- added C1414: 0.1uF, Capacitor_SMD:C_0805_2012Metric, F.Cu at (-70.2, 182.5)
- added C1415: 0.1uF, Capacitor_SMD:C_0805_2012Metric, F.Cu at (-70.2, 185.5)
- added C1416: 2.2uF, Capacitor_SMD:C_1206_3216Metric, F.Cu at (-82.9, 169.7)
- added C1417: 3.3nF, Capacitor_SMD:C_1206_3216Metric, F.Cu at (-82.9, 173.0)
- added C1418: 3.3nF, Capacitor_SMD:C_1206_3216Metric, F.Cu at (-82.9, 176.3)
- added C1419: 3.3nF, Capacitor_SMD:C_1206_3216Metric, F.Cu at (-82.9, 179.7)
- added C1420: 3.3nF, Capacitor_SMD:C_1206_3216Metric, F.Cu at (-82.9, 183.1)
- added C1509: 1nF, Capacitor_SMD:C_1206_3216Metric, F.Cu at (-129.2, 78.7)
- added C1514: 910pF, Capacitor_SMD:C_1206_3216Metric, F.Cu at (-129.2, 82.0)
- added C1515: 910pF, Capacitor_SMD:C_1206_3216Metric, F.Cu at (-129.2, 85.4)
- added C1516: 330pF, Capacitor_SMD:C_1206_3216Metric, F.Cu at (-129.2, 88.7)
- added C1517: 330pF, Capacitor_SMD:C_1206_3216Metric, F.Cu at (-129.2, 92.1)
- added C1518: 220pF, Capacitor_SMD:C_1206_3216Metric, F.Cu at (-129.2, 95.4)
- added C1519: 22pF, Capacitor_SMD:C_1206_3216Metric, F.Cu at (-129.2, 98.8)
- added C1520: 270pF, Capacitor_SMD:C_1206_3216Metric, F.Cu at (-129.2, 102.1)
- added C1521: 220pF, Capacitor_SMD:C_1206_3216Metric, F.Cu at (-123.5, 78.7)
- added C1522: 47pF, Capacitor_SMD:C_1206_3216Metric, F.Cu at (-123.5, 82.0)
- added C1523: 47pF, Capacitor_SMD:C_1206_3216Metric, F.Cu at (-123.5, 85.4)
- added C1524: 47pF, Capacitor_SMD:C_1206_3216Metric, F.Cu at (-123.5, 88.7)
- added C1525: 47pF, Capacitor_SMD:C_1206_3216Metric, F.Cu at (-123.5, 92.1)
- added C1526: 33pF, Capacitor_SMD:C_1206_3216Metric, F.Cu at (-123.5, 95.4)
- added C1527: 33pF, Capacitor_SMD:C_1206_3216Metric, F.Cu at (-123.5, 98.8)
- added C1528: 33pF, Capacitor_SMD:C_1206_3216Metric, F.Cu at (-123.5, 102.1)
- added C1529: 27pF, Capacitor_SMD:C_1206_3216Metric, F.Cu at (-117.8, 78.7)
- added C1530: 22pF, Capacitor_SMD:C_1206_3216Metric, F.Cu at (-117.8, 82.0)
- added C1531: 22pF, Capacitor_SMD:C_1206_3216Metric, F.Cu at (-117.8, 85.4)
- added C1532: 22pF, Capacitor_SMD:C_1206_3216Metric, F.Cu at (-117.8, 88.7)
- added C1533: 22pF, Capacitor_SMD:C_1206_3216Metric, F.Cu at (-117.8, 92.1)
- added C1534: 33pF, Capacitor_SMD:C_1206_3216Metric, F.Cu at (-117.8, 95.4)
- added C1535: 33pF, Capacitor_SMD:C_1206_3216Metric, F.Cu at (-117.8, 98.8)
- added C1536: 16pF, Capacitor_SMD:C_1206_3216Metric, F.Cu at (-117.8, 102.1)
- added C1537: 16pF, Capacitor_SMD:C_1206_3216Metric, F.Cu at (-112.2, 78.7)
- added C1538: 16pF, Capacitor_SMD:C_1206_3216Metric, F.Cu at (-112.2, 82.0)
- added C1539: 8pF, Capacitor_SMD:C_1206_3216Metric, F.Cu at (-112.2, 85.4)
- added C1540: 4pF, Capacitor_SMD:C_1206_3216Metric, F.Cu at (-112.2, 88.7)
- added C1609: 330pF, Capacitor_SMD:C_1206_3216Metric, F.Cu at (-157.2, 160.4)
- added C1614: 240pF, Capacitor_SMD:C_1206_3216Metric, F.Cu at (-157.2, 163.7)
- added C1615: 390pF, Capacitor_SMD:C_1206_3216Metric, F.Cu at (-157.2, 167.1)
- added C1616: 180pF, Capacitor_SMD:C_1206_3216Metric, F.Cu at (-157.2, 170.4)
- added C1617: 150pF, Capacitor_SMD:C_1206_3216Metric, F.Cu at (-157.2, 173.8)
- added C1618: 100pF, Capacitor_SMD:C_1206_3216Metric, F.Cu at (-157.2, 177.1)
- added C1619: 82pF, Capacitor_SMD:C_1206_3216Metric, F.Cu at (-157.2, 180.5)
- added C1620: 56pF, Capacitor_SMD:C_1206_3216Metric, F.Cu at (-157.2, 183.8)
- added C1621: 39pF, Capacitor_SMD:C_1206_3216Metric, F.Cu at (-151.5, 160.4)
- added C1622: 27pF, Capacitor_SMD:C_1206_3216Metric, F.Cu at (-151.5, 163.7)
- added C1623: 100pF, Capacitor_SMD:C_1206_3216Metric, F.Cu at (-151.5, 167.1)
- added C1624: 68pF, Capacitor_SMD:C_1206_3216Metric, F.Cu at (-151.5, 170.4)
- added C1625: 47pF, Capacitor_SMD:C_1206_3216Metric, F.Cu at (-151.5, 173.8)
- added C1626: 33pF, Capacitor_SMD:C_1206_3216Metric, F.Cu at (-151.5, 177.1)
- added C1627: 24pF, Capacitor_SMD:C_0805_2012Metric, F.Cu at (-186.8, 175.3)
- added C1628: 100pF, Capacitor_SMD:C_1206_3216Metric, F.Cu at (-151.5, 180.5)
- added C1629: 68pF, Capacitor_SMD:C_1206_3216Metric, F.Cu at (-151.5, 183.8)
- added C1630: 47pF, Capacitor_SMD:C_1206_3216Metric, F.Cu at (-145.9, 160.4)
- added C1631: 33pF, Capacitor_SMD:C_1206_3216Metric, F.Cu at (-145.9, 163.7)
- added C1632: 24pF, Capacitor_SMD:C_0805_2012Metric, F.Cu at (-186.8, 178.3)
- added C1633: 100pF, Capacitor_SMD:C_1206_3216Metric, F.Cu at (-145.9, 167.1)
- added C1634: 82pF, Capacitor_SMD:C_1206_3216Metric, F.Cu at (-145.9, 170.4)
- added C1635: 56pF, Capacitor_SMD:C_1206_3216Metric, F.Cu at (-145.9, 173.8)
- added C1636: 39pF, Capacitor_SMD:C_1206_3216Metric, F.Cu at (-145.9, 177.1)
- added C1637: 27pF, Capacitor_SMD:C_1206_3216Metric, F.Cu at (-145.9, 180.5)
- added C1814: 0.1uF, Capacitor_SMD:C_0805_2012Metric, F.Cu at (-59.4, 190.5)
- added C1815: 0.1uF, Capacitor_SMD:C_0805_2012Metric, F.Cu at (-59.4, 193.5)
- added C1816: 10uF, Capacitor_SMD:C_0805_2012Metric, F.Cu at (-59.4, 196.5)
- added C1817: 10uF, Capacitor_SMD:C_0805_2012Metric, F.Cu at (-54.9, 190.5)
- added C1818: 1uF, Capacitor_SMD:C_0805_2012Metric, F.Cu at (-54.9, 193.5)
- added C1819: 1uF, Capacitor_SMD:C_0805_2012Metric, F.Cu at (-54.9, 196.5)
- added C1820: 10uF, Capacitor_SMD:C_0805_2012Metric, F.Cu at (-50.5, 190.5)
- added C1821: 10uF, Capacitor_SMD:C_0805_2012Metric, F.Cu at (-50.5, 193.5)
- added C2026: 10uF 100V, Capacitor_SMD:C_1206_3216Metric, F.Cu at (-154.5, 195.8)
- added C2027: 0.1uF, Capacitor_SMD:C_0805_2012Metric, F.Cu at (-146.6, 189.0)
- added C2028: 10uF, Capacitor_SMD:C_0805_2012Metric, F.Cu at (-146.6, 192.0)
- added C2403: 0.1uF, Capacitor_SMD:C_0805_2012Metric, F.Cu at (-103.7, 169.5)
- added C2404: 1uF, Capacitor_SMD:C_0805_2012Metric, F.Cu at (-103.7, 172.5)
- added C2405: 470pF, Capacitor_SMD:C_1206_3216Metric, F.Cu at (-91.1, 184.0)
- added C2406: 10uF, Capacitor_SMD:C_0805_2012Metric, F.Cu at (-103.7, 175.5)
- added C2407: 0.1uF, Capacitor_SMD:C_0805_2012Metric, F.Cu at (-99.2, 169.5)
- added C2408: 0.1uF, Capacitor_SMD:C_0805_2012Metric, F.Cu at (-99.2, 172.5)
- added C2409: 0.1uF, Capacitor_SMD:C_0805_2012Metric, F.Cu at (-99.2, 175.5)
- added C2410: 0.1uF, Capacitor_SMD:C_0805_2012Metric, F.Cu at (-94.8, 169.5)
- added C2411: 0.1uF, Capacitor_SMD:C_0805_2012Metric, F.Cu at (-94.8, 172.5)
- added C2412: 1000pF, Capacitor_SMD:C_0805_2012Metric, F.Cu at (-94.8, 175.5)
- added C315: 0.1uF, Capacitor_SMD:C_0805_2012Metric, F.Cu at (-129.8, 169.5)
- added C316: 4.7uF, Capacitor_SMD:C_0805_2012Metric, F.Cu at (-129.8, 172.5)
- added C317: 0.1uF, Capacitor_SMD:C_0805_2012Metric, F.Cu at (-129.8, 175.5)
- added C318: 4.7uF, Capacitor_SMD:C_0805_2012Metric, F.Cu at (-129.8, 178.5)
- added C319: 1uF, Capacitor_SMD:C_0805_2012Metric, F.Cu at (-129.8, 181.5)
- added C320: 0.1uF, Capacitor_SMD:C_0805_2012Metric, F.Cu at (-129.8, 184.5)
- added C404: 8pF, Capacitor_SMD:C_1206_3216Metric, F.Cu at (-59.2, 44.1)
- added C405: 16pF, Capacitor_SMD:C_1206_3216Metric, F.Cu at (-59.2, 47.4)
- added C406: 32pF, Capacitor_SMD:C_1206_3216Metric, F.Cu at (-59.2, 50.8)
- added C407: 64pF, Capacitor_SMD:C_1206_3216Metric, F.Cu at (-59.2, 54.1)
- added C408: 1uF, Capacitor_SMD:C_0805_2012Metric, F.Cu at (-54.9, 57.3)
- added C409: 128pF, Capacitor_SMD:C_1206_3216Metric, F.Cu at (-53.5, 44.1)
- added C410: 1uF, Capacitor_SMD:C_0805_2012Metric, F.Cu at (-54.9, 60.3)
- added C411: 256pF, Capacitor_SMD:C_1206_3216Metric, F.Cu at (-53.5, 47.4)
- added C412: 1uF, Capacitor_SMD:C_0805_2012Metric, F.Cu at (-54.9, 63.3)
- added C413: 1uF, Capacitor_SMD:C_0805_2012Metric, F.Cu at (-54.9, 66.3)
- added C414: 512pF, Capacitor_SMD:C_1206_3216Metric, F.Cu at (-53.5, 50.8)
- added C415: 1uF, Capacitor_SMD:C_0805_2012Metric, F.Cu at (-54.9, 69.4)
- added C416: 1024pF, Capacitor_SMD:C_1206_3216Metric, F.Cu at (-53.5, 54.1)
- added C417: 1uF, Capacitor_SMD:C_0805_2012Metric, F.Cu at (-54.9, 72.4)
- added C418: 2048pF, Capacitor_SMD:C_1206_3216Metric, F.Cu at (-47.9, 44.1)
- added C419: 1uF, Capacitor_SMD:C_1206_3216Metric, F.Cu at (-47.9, 47.4)
- added C420: 1uF, Capacitor_SMD:C_1206_3216Metric, F.Cu at (-47.9, 50.8)
- added C421: 2.2nF, Capacitor_SMD:C_1206_3216Metric, F.Cu at (-47.9, 54.1)
- added C606: .1uF, Capacitor_SMD:C_0805_2012Metric, F.Cu at (-218.0, 189.0)
- added C607: 4.7uF, Capacitor_SMD:C_0805_2012Metric, F.Cu at (-218.0, 192.0)
- added C608: 0.1uF, Capacitor_SMD:C_0805_2012Metric, F.Cu at (-218.0, 195.0)
- added C609: 0.1uF, Capacitor_SMD:C_0805_2012Metric, F.Cu at (-218.0, 198.0)
- added C610: 10nF, Capacitor_SMD:C_0805_2012Metric, F.Cu at (-218.0, 201.1)
- added C611: 1nF, Capacitor_SMD:C_0805_2012Metric, F.Cu at (-213.5, 189.0)
- added C612: 4.7uF, Capacitor_SMD:C_0805_2012Metric, F.Cu at (-213.5, 192.0)
- added C613: 0.1uF, Capacitor_SMD:C_0805_2012Metric, F.Cu at (-213.5, 195.0)
- added C614: 4.7uF, Capacitor_SMD:C_0805_2012Metric, F.Cu at (-213.5, 198.0)
- added C615: 0.1uF, Capacitor_SMD:C_0805_2012Metric, F.Cu at (-213.5, 201.1)
- added C701: 10uF, Capacitor_SMD:C_1206_3216Metric, F.Cu at (-58.8, 185.3)
- added CF1801: 1uF, Capacitor_SMD:C_0805_2012Metric, F.Cu at (-50.5, 196.5)
- added D301: STS321150B100AH, Diode_SMD:D_SOD-323, F.Cu at (-129.8, 187.5)
- added FB2401: BLM21AG102SN1D, Inductor_SMD:L_0805_2012Metric, F.Cu at (-91.6, 191.7)
- added J2001: Amphenol 10167129, Library:1016712900011LF, F.Cu at (-193.8, 196.6)
- added J201: 68710814022, Library:68710814022, F.Cu at (-58.6, 78.6)
- added J202: FTSH-105-01-L-DV-K, Library:FTSH10501LDVK, F.Cu at (-71.4, 97.4)
- added J501: SO239, Connector_Coaxial:SMA_Amphenol_132289_EdgeMount, F.Cu at (-89.3, 153.7)
- added K1501: TQ2-5V, symbols:RELAY_TQ2_PAN, F.Cu at (-130.4, 32.8)
- added K1502: TQ2-5V, symbols:RELAY_TQ2_PAN, F.Cu at (-119.6, 32.8)
- added K1503: TQ2-5V, symbols:RELAY_TQ2_PAN, F.Cu at (-108.8, 32.8)
- added K1504: TQ2-5V, symbols:RELAY_TQ2_PAN, F.Cu at (-98.1, 32.8)
- added K1505: TQ2-5V, symbols:RELAY_TQ2_PAN, F.Cu at (-87.3, 32.8)
- added K1506: TQ2-5V, symbols:RELAY_TQ2_PAN, F.Cu at (-130.4, 48.5)
- added K1507: TQ2-5V, symbols:RELAY_TQ2_PAN, F.Cu at (-119.6, 48.5)
- added K1508: TQ2-5V, symbols:RELAY_TQ2_PAN, F.Cu at (-108.8, 48.5)
- added K1509: TQ2-5V, symbols:RELAY_TQ2_PAN, F.Cu at (-98.1, 48.5)
- added K1510: TQ2-5V, symbols:RELAY_TQ2_PAN, F.Cu at (-87.3, 48.5)
- added K1511: TQ2-5V, symbols:RELAY_TQ2_PAN, F.Cu at (-130.4, 64.1)
- added K1512: TQ2-5V, symbols:RELAY_TQ2_PAN, F.Cu at (-119.6, 64.1)
- added K1513: TQ2-5V, symbols:RELAY_TQ2_PAN, F.Cu at (-108.8, 64.1)
- added K1601: TQ2-5V, symbols:RELAY_TQ2_PAN, F.Cu at (-218.6, 119.6)
- added K1602: TQ2-5V, symbols:RELAY_TQ2_PAN, F.Cu at (-207.8, 119.6)
- added K1603: TQ2-5V, symbols:RELAY_TQ2_PAN, F.Cu at (-197.1, 119.6)
- added K1604: TQ2-5V, symbols:RELAY_TQ2_PAN, F.Cu at (-186.3, 119.6)
- added K1605: TQ2-5V, symbols:RELAY_TQ2_PAN, F.Cu at (-175.5, 119.6)
- added K1606: TQ2-5V, symbols:RELAY_TQ2_PAN, F.Cu at (-164.7, 119.6)
- added K1607: TQ2-5V, symbols:RELAY_TQ2_PAN, F.Cu at (-154.0, 119.6)
- added K1608: TQ2-5V, symbols:RELAY_TQ2_PAN, F.Cu at (-143.2, 119.6)
- added K1701: TQ2-5V, symbols:RELAY_TQ2_PAN, F.Cu at (-218.6, 32.8)
- added K1702: TQ2-5V, symbols:RELAY_TQ2_PAN, F.Cu at (-207.8, 32.8)
- added K1703: TQ2-5V, symbols:RELAY_TQ2_PAN, F.Cu at (-197.1, 32.8)
- added K1704: TQ2-5V, symbols:RELAY_TQ2_PAN, F.Cu at (-186.3, 32.8)
- added K1705: TQ2-5V, symbols:RELAY_TQ2_PAN, F.Cu at (-175.5, 32.8)
- added K1706: TQ2-5V, symbols:RELAY_TQ2_PAN, F.Cu at (-164.7, 32.8)
- added K1707: TQ2-5V, symbols:RELAY_TQ2_PAN, F.Cu at (-154.0, 32.8)
- added K1708: TQ2-5V, symbols:RELAY_TQ2_PAN, F.Cu at (-143.2, 32.8)
- added K2109: TQ2-5V, symbols:RELAY_TQ2_PAN, F.Cu at (-177.6, 190.3)
- added K501: TQ2-5V, symbols:RELAY_TQ2_PAN, F.Cu at (-86.4, 130.5)
- added K702: TQ2-5V, symbols:RELAY_TQ2_PAN, F.Cu at (-60.0, 170.7)
- added K703: TQ2-5V, symbols:RELAY_TQ2_PAN, F.Cu at (-49.2, 170.7)
- added L1201: 2.2uH, Library:INDC2012X105N, F.Cu at (-52.4, 130.5)
- added L1301: 2.2uH, Library:INDC2012X105N, F.Cu at (-52.4, 107.3)
- added L1401: 2.2uH, Library:INDC2012X105N, F.Cu at (-65.8, 169.5)
- added L1501: 500nH, Inductor_SMD:L_Coilcraft_2929SQ-501, F.Cu at (-100.8, 82.0)
- added L1502: 300nH, Inductor_SMD:L_Coilcraft_2222SQ-301, F.Cu at (-101.9, 91.1)
- added L1503: 82nH, Inductor_SMD:L_Coilcraft_1515SQ-82N, F.Cu at (-105.0, 98.3)
- added L1601: 18uH, Library:L_Wurth_10.6mm_sq_SMT, F.Cu at (-213.7, 139.1)
- added L1602: 10uH, Library:L_Wurth_10.6mm_sq_SMT, F.Cu at (-200.6, 139.1)
- added L1603: 6.8uH, Library:L_Wurth_12.2mm_sq_SMT, F.Cu at (-212.7, 166.3)
- added L1604: 18uH, Library:L_Wurth_10.6mm_sq_SMT, F.Cu at (-187.6, 139.1)
- added L1605: 10uH, Library:L_Wurth_10.6mm_sq_SMT, F.Cu at (-174.5, 139.1)
- added L1606: 6.8uH, Library:L_Wurth_12.2mm_sq_SMT, F.Cu at (-197.6, 166.3)
- added L1607: 4.7uH, Library:L_Wurth_12.2mm_sq_SMT, F.Cu at (-182.6, 166.3)
- added L1608: 3.3uH, Library:L_Wurth_10.6mm_sq_SMT, F.Cu at (-161.5, 139.1)
- added L1609: 2.2uH, Library:L_Wurth_8.1mm_sq_SMT, F.Cu at (-214.7, 179.4)
- added L1610: 1.8uH, Library:L_Wurth_10.6mm_sq_SMT, F.Cu at (-213.7, 152.2)
- added L1611: 1.5uH, Library:L_Wurth_10.6mm_sq_SMT, F.Cu at (-200.6, 152.2)
- added L1612: 4.7uH, Library:L_Wurth_12.2mm_sq_SMT, F.Cu at (-167.5, 166.3)
- added L1613: 3.3uH, Library:L_Wurth_10.6mm_sq_SMT, F.Cu at (-187.6, 152.2)
- added L1614: 2.2uH, Library:L_Wurth_8.1mm_sq_SMT, F.Cu at (-203.6, 179.4)
- added L1615: 1.8uH, Library:L_Wurth_10.6mm_sq_SMT, F.Cu at (-174.5, 152.2)
- added L1616: 1.5uH, Library:L_Wurth_10.6mm_sq_SMT, F.Cu at (-161.5, 152.2)
- added L1701: 64uH, Inductor_THT:L_Toroid_Vertical_L35.1mm_W21.1mm_P18.50mm_Vishay_TJ6, F.Cu at (-201.9, 48.0)
- added L1702: 32uH, Inductor_THT:L_Toroid_Vertical_L35.1mm_W21.1mm_P18.50mm_Vishay_TJ6, F.Cu at (-201.9, 71.0)
- added L1703: 16uH, Inductor_THT:L_Toroid_Vertical_L35.1mm_W21.1mm_P18.50mm_Vishay_TJ6, F.Cu at (-201.9, 94.1)
- added L1704: 8uH, Inductor_THT:L_Toroid_Vertical_L26.7mm_W14.0mm_P10.16mm_Pulse_D, F.Cu at (-169.4, 48.4)
- added L1705: 4uH, Inductor_THT:L_Toroid_Vertical_L26.7mm_W14.0mm_P10.16mm_Pulse_D, F.Cu at (-169.4, 63.9)
- added L1706: 2uH, Inductor_THT:L_Toroid_Vertical_L26.7mm_W14.0mm_P10.16mm_Pulse_D, F.Cu at (-169.4, 79.5)
- added L1707: 1uH, Library:Coilcraft-uni10, F.Cu at (-149.3, 51.8)
- added L1708: 0.5uH, Library:Coilcraft-uni10, F.Cu at (-149.3, 63.9)
- added L1803: 3.3uH, Inductor_SMD:L_0805_2012Metric, F.Cu at (-59.3, 199.4)
- added L301: 1.2uH, Inductor_SMD:L_0805_2012Metric, F.Cu at (-113.1, 190.2)
- added L401: 8t bifilar, Inductor_THT:L_CommonMode_Toroid_Vertical_L19.3mm_W10.8mm_Px6.35mm_Py15.24mm_Bourns_8100, F.Cu at (-59.2, 33.1)
- added L402: 8.2uH, Inductor_SMD:L_Coilcraft_1008HQ_2520Metric, F.Cu at (-59.5, 58.2)
- added L403: 2.7uH, Inductor_SMD:L_Coilcraft_1008HQ_2520Metric, F.Cu at (-59.5, 62.8)
- added L404: 820nH, Inductor_SMD:L_Coilcraft_1008HQ_2520Metric, F.Cu at (-59.5, 67.4)
- added L405: 270nH, Inductor_SMD:L_Coilcraft_1008HQ_2520Metric, F.Cu at (-59.5, 72.0)
- added L501: 16t:8t bifilar #18AWG FT140-43, Inductor_THT:L_CommonMode_Toroid_Vertical_L36.8mm_W20.3mm_Px15.24mm_Py22.86mm_Bourns_8100, F.Cu at (-124.2, 131.0)
- added Q1001: 2N7002K, Package_TO_SOT_SMD:SOT-23, F.Cu at (-123.9, 205.2)
- added Q1101: 2N7002K, Package_TO_SOT_SMD:SOT-23, F.Cu at (-51.7, 161.9)
- added Q501: IRFP250NPBF, Library:TO545P530X1560X2460-3P, F.Cu at (-89.0, 109.6)
- added Q801: 2N7002K, Package_TO_SOT_SMD:SOT-23, F.Cu at (-64.3, 161.9)
- added Q901: 2N7002K, Package_TO_SOT_SMD:SOT-23, F.Cu at (-111.4, 205.2)
- added R1001: 10k, Resistor_SMD:R_0603_1608Metric, F.Cu at (-130.0, 206.7)
- added R1002: 34, Resistor_SMD:R_1206_3216Metric, F.Cu at (-129.2, 197.1)
- added R1003: 562, Resistor_SMD:R_1206_3216Metric, F.Cu at (-129.2, 200.4)
- added R1004: 34, Resistor_SMD:R_1206_3216Metric, F.Cu at (-129.2, 203.8)
- added R1101: 10k, Resistor_SMD:R_0603_1608Metric, F.Cu at (-57.8, 163.4)
- added R1102: 34, Resistor_SMD:R_1206_3216Metric, F.Cu at (-57.0, 153.9)
- added R1103: 562, Resistor_SMD:R_1206_3216Metric, F.Cu at (-57.0, 157.2)
- added R1104: 34, Resistor_SMD:R_1206_3216Metric, F.Cu at (-57.0, 160.5)
- added R1201: 10k, Resistor_SMD:R_0603_1608Metric, F.Cu at (-64.7, 130.3)
- added R1202: 10k, Resistor_SMD:R_0603_1608Metric, F.Cu at (-64.7, 132.8)
- added R1203: 10k, Resistor_SMD:R_0603_1608Metric, F.Cu at (-64.7, 135.3)
- added R1204: 10k, Resistor_SMD:R_0603_1608Metric, F.Cu at (-64.7, 137.8)
- added R1205: 10k, Resistor_SMD:R_0603_1608Metric, F.Cu at (-60.7, 130.3)
- added R1206: 10k, Resistor_SMD:R_0603_1608Metric, F.Cu at (-60.7, 132.8)
- added R1207: 10k, Resistor_SMD:R_0603_1608Metric, F.Cu at (-60.7, 135.3)
- added R1208: 10k, Resistor_SMD:R_0603_1608Metric, F.Cu at (-60.7, 137.8)
- added R1209: 330, Resistor_SMD:R_0603_1608Metric, F.Cu at (-56.6, 130.3)
- added R1210: 330, Resistor_SMD:R_0603_1608Metric, F.Cu at (-56.6, 132.8)
- added R1211: 330, Resistor_SMD:R_0603_1608Metric, F.Cu at (-56.6, 135.3)
- added R1212: 330, Resistor_SMD:R_0603_1608Metric, F.Cu at (-56.6, 137.8)
- added R1301: 10k, Resistor_SMD:R_0603_1608Metric, F.Cu at (-64.7, 107.1)
- added R1302: 10k, Resistor_SMD:R_0603_1608Metric, F.Cu at (-64.7, 109.6)
- added R1303: 10k, Resistor_SMD:R_0603_1608Metric, F.Cu at (-64.7, 112.1)
- added R1304: 10k, Resistor_SMD:R_0603_1608Metric, F.Cu at (-64.7, 114.6)
- added R1305: 10k, Resistor_SMD:R_0603_1608Metric, F.Cu at (-60.7, 107.1)
- added R1306: 10k, Resistor_SMD:R_0603_1608Metric, F.Cu at (-60.7, 109.6)
- added R1307: 10k, Resistor_SMD:R_0603_1608Metric, F.Cu at (-60.7, 112.1)
- added R1308: 10k, Resistor_SMD:R_0603_1608Metric, F.Cu at (-60.7, 114.6)
- added R1309: 330, Resistor_SMD:R_0603_1608Metric, F.Cu at (-56.6, 107.1)
- added R1310: 330, Resistor_SMD:R_0603_1608Metric, F.Cu at (-56.6, 109.6)
- added R1311: 330, Resistor_SMD:R_0603_1608Metric, F.Cu at (-56.6, 112.1)
- added R1312: 330, Resistor_SMD:R_0603_1608Metric, F.Cu at (-56.6, 114.6)
- added R1401: 10k, Resistor_SMD:R_0603_1608Metric, F.Cu at (-78.1, 169.2)
- added R1402: 10k, Resistor_SMD:R_0603_1608Metric, F.Cu at (-78.1, 171.7)
- added R1403: 10k, Resistor_SMD:R_0603_1608Metric, F.Cu at (-78.1, 174.2)
- added R1404: 10k, Resistor_SMD:R_0603_1608Metric, F.Cu at (-78.1, 176.8)
- added R1405: 10k, Resistor_SMD:R_0603_1608Metric, F.Cu at (-74.0, 169.2)
- added R1406: 10k, Resistor_SMD:R_0603_1608Metric, F.Cu at (-74.0, 171.7)
- added R1407: 10k, Resistor_SMD:R_0603_1608Metric, F.Cu at (-74.0, 174.2)
- added R1408: 10k, Resistor_SMD:R_0603_1608Metric, F.Cu at (-74.0, 176.8)
- added R1409: 330, Resistor_SMD:R_0603_1608Metric, F.Cu at (-70.0, 169.2)
- added R1410: 330, Resistor_SMD:R_0603_1608Metric, F.Cu at (-70.0, 171.7)
- added R1411: 330, Resistor_SMD:R_0603_1608Metric, F.Cu at (-70.0, 174.2)
- added R1412: 330, Resistor_SMD:R_0603_1608Metric, F.Cu at (-70.0, 176.8)
- added R201: 10k, Resistor_SMD:R_0603_1608Metric, F.Cu at (-63.4, 85.3)
- added R202: 10k, Resistor_SMD:R_0603_1608Metric, F.Cu at (-63.4, 87.8)
- added R2021: 10k, Resistor_SMD:R_0603_1608Metric, F.Cu at (-185.9, 195.1)
- added R203: 10k, Resistor_SMD:R_0603_1608Metric, F.Cu at (-63.4, 90.3)
- added R204: 10k, Resistor_SMD:R_0603_1608Metric, F.Cu at (-63.4, 92.9)
- added R205: 10k, Resistor_SMD:R_0603_1608Metric, F.Cu at (-63.4, 95.4)
- added R206: 10k, Resistor_SMD:R_0603_1608Metric, F.Cu at (-59.4, 85.3)
- added R207: 10k, Resistor_SMD:R_0603_1608Metric, F.Cu at (-59.4, 87.8)
- added R208: 10k, Resistor_SMD:R_0603_1608Metric, F.Cu at (-59.4, 90.3)
- added R209: 100, Resistor_SMD:R_0603_1608Metric, F.Cu at (-59.4, 92.9)
- added R210: 10k, Resistor_SMD:R_0603_1608Metric, F.Cu at (-59.4, 95.4)
- added R2401: 10k, Resistor_SMD:R_0603_1608Metric, F.Cu at (-103.9, 178.3)
- added R2402: 33, Resistor_SMD:R_0603_1608Metric, F.Cu at (-103.9, 180.8)
- added R2403: 33, Resistor_SMD:R_0603_1608Metric, F.Cu at (-103.9, 183.3)
- added R2404: 33, Resistor_SMD:R_0603_1608Metric, F.Cu at (-103.9, 185.8)
- added R2405: 33, Resistor_SMD:R_0603_1608Metric, F.Cu at (-103.9, 188.3)
- added R2406: 10k, Resistor_SMD:R_0603_1608Metric, F.Cu at (-103.9, 190.8)
- added R2407: 100k, Resistor_SMD:R_0603_1608Metric, F.Cu at (-103.9, 193.3)
- added R2408: 10k, Resistor_SMD:R_0603_1608Metric, F.Cu at (-99.9, 178.3)
- added R2409: 10k, Resistor_SMD:R_0603_1608Metric, F.Cu at (-99.9, 180.8)
- added R2410: 10k, Resistor_SMD:R_0603_1608Metric, F.Cu at (-99.9, 183.3)
- added R2411: 0, Resistor_SMD:R_0603_1608Metric, F.Cu at (-99.9, 185.8)
- added R2412: 0, Resistor_SMD:R_0603_1608Metric, F.Cu at (-99.9, 188.3)
- added R2413: 49.9, Resistor_SMD:R_0603_1608Metric, F.Cu at (-99.9, 190.8)
- added R2414: 49.9, Resistor_SMD:R_0603_1608Metric, F.Cu at (-99.9, 193.3)
- added R2415: 12.1k, Resistor_SMD:R_0603_1608Metric, F.Cu at (-95.9, 178.3)
- added R2416: 49.9, Resistor_SMD:R_0603_1608Metric, F.Cu at (-95.9, 180.8)
- added R2417: 49.9, Resistor_SMD:R_0603_1608Metric, F.Cu at (-95.9, 183.3)
- added R2418: 270, Resistor_SMD:R_0805_2012Metric, F.Cu at (-90.4, 169.4)
- added R2419: 270, Resistor_SMD:R_0805_2012Metric, F.Cu at (-90.4, 172.4)
- added R2420: 10k, Resistor_SMD:R_0603_1608Metric, F.Cu at (-95.9, 185.8)
- added R301: 1k, Resistor_SMD:R_0603_1608Metric, F.Cu at (-109.9, 169.2)
- added R302: 1k, Resistor_SMD:R_0603_1608Metric, F.Cu at (-109.9, 171.7)
- added R303: 10k, Resistor_SMD:R_0603_1608Metric, F.Cu at (-109.9, 174.2)
- added R501: 6.8, Resistor_SMD:R_1206_3216Metric, F.Cu at (-90.8, 129.3)
- added R502: 49.9, Resistor_SMD:R_1206_3216Metric, F.Cu at (-90.8, 132.7)
- added R503: 47k, Resistor_SMD:R_1206_3216Metric, F.Cu at (-90.8, 136.0)
- added R504: 220, Resistor_SMD:R_1206_3216Metric, F.Cu at (-90.8, 139.3)
- added R505: 47k, Resistor_SMD:R_1206_3216Metric, F.Cu at (-90.8, 142.6)
- added R506: 220, Resistor_SMD:R_1206_3216Metric, F.Cu at (-90.8, 145.9)
- added R601: 0, Resistor_SMD:R_0603_1608Metric, F.Cu at (-204.2, 198.1)
- added R602: 100, Resistor_SMD:R_0603_1608Metric, F.Cu at (-204.2, 200.6)
- added R801: 10k, Resistor_SMD:R_0603_1608Metric, F.Cu at (-70.3, 163.4)
- added R802: 34, Resistor_SMD:R_1206_3216Metric, F.Cu at (-69.5, 153.9)
- added R803: 562, Resistor_SMD:R_1206_3216Metric, F.Cu at (-69.5, 157.2)
- added R804: 34, Resistor_SMD:R_1206_3216Metric, F.Cu at (-69.5, 160.5)
- added R901: 10k, Resistor_SMD:R_0603_1608Metric, F.Cu at (-117.5, 206.7)
- added R902: 34, Resistor_SMD:R_1206_3216Metric, F.Cu at (-116.7, 197.1)
- added R903: 562, Resistor_SMD:R_1206_3216Metric, F.Cu at (-116.7, 200.4)
- added R904: 34, Resistor_SMD:R_1206_3216Metric, F.Cu at (-116.7, 203.8)
- added T301: 12t primary : 6T #26 trifilar secondary FT37-43, Library:Toroid-1pri-3sec-ft50, F.Cu at (-120.0, 172.5)
- added T501: 3t:3t Fair-Rite 2843000202 bifilar litz 5/52/38, Library:Fair-Rite 2843000202 bifilar #14AWG, F.Cu at (-121.9, 153.6)
- added T502: ~, Inductor_THT:L_CommonMode_Toroid_Vertical_L38.1mm_W20.3mm_Px15.24mm_Py22.86mm_Bourns_8100, F.Cu at (-123.6, 109.1)
- added T503: Bruene sampler, Library:toroid-pri-sec-ct-ft50, F.Cu at (-84.8, 117.2)
- added TP201: PG0, TestPoint:TestPoint_Pad_1.5x1.5mm, F.Cu at (-74.3, 78.0)
- added TP202: PG1, TestPoint:TestPoint_Pad_1.5x1.5mm, F.Cu at (-74.3, 81.5)
- added TP203: PG2, TestPoint:TestPoint_Pad_1.5x1.5mm, F.Cu at (-74.3, 85.1)
- added TP204: PG3, TestPoint:TestPoint_Pad_1.5x1.5mm, F.Cu at (-74.3, 88.6)
- added TP205: PG4, TestPoint:TestPoint_Pad_1.5x1.5mm, F.Cu at (-70.8, 78.0)
- added TP206: PG5, TestPoint:TestPoint_Pad_1.5x1.5mm, F.Cu at (-70.8, 81.5)
- added TP207: PG6, TestPoint:TestPoint_Pad_1.5x1.5mm, F.Cu at (-70.8, 85.1)
- added TP208: PG7, TestPoint:TestPoint_Pad_1.5x1.5mm, F.Cu at (-70.8, 88.6)
- added TP209: PG8, TestPoint:TestPoint_Pad_1.5x1.5mm, F.Cu at (-67.2, 78.0)
- added TP210: PG14, TestPoint:TestPoint_Pad_1.5x1.5mm, F.Cu at (-67.2, 81.5)
- added TP211: PG15, TestPoint:TestPoint_Pad_1.5x1.5mm, F.Cu at (-67.2, 85.1)
- added U1001: AS183-92LF, Library:SOT65P220X110-6N, F.Cu at (-124.0, 197.3)
- added U1002: AS183-92LF, Library:SOT65P220X110-6N, F.Cu at (-124.0, 201.1)
- added U1101: AS183-92LF, Library:SOT65P220X110-6N, F.Cu at (-51.8, 154.1)
- added U1102: AS183-92LF, Library:SOT65P220X110-6N, F.Cu at (-51.8, 157.8)
- added U1201: SZNUP1105LT1G, Package_TO_SOT_SMD:SOT-23, F.Cu at (-69.9, 148.0)
- added U1202: TS3A4751RUCR, Library:TS3A4751-RUC14, F.Cu at (-52.6, 134.1)
- added U1203: MAX9939AUB+T, symbols:21-0061L_MXM, F.Cu at (-63.0, 141.4)
- added U1204: MAX9939AUB+T, symbols:21-0061L_MXM, F.Cu at (-63.0, 146.1)
- added U1301: SZNUP1105LT1G, Package_TO_SOT_SMD:SOT-23, F.Cu at (-69.9, 124.8)
- added U1302: TS3A4751RUCR, Library:TS3A4751-RUC14, F.Cu at (-52.6, 110.9)
- added U1303: MAX9939AUB+T, symbols:21-0061L_MXM, F.Cu at (-63.0, 118.2)
- added U1304: MAX9939AUB+T, symbols:21-0061L_MXM, F.Cu at (-63.0, 122.9)
- added U1401: SZNUP1105LT1G, Package_TO_SOT_SMD:SOT-23, F.Cu at (-83.3, 186.9)
- added U1402: TS3A4751RUCR, Library:TS3A4751-RUC14, F.Cu at (-66.0, 173.0)
- added U1403: MAX9939AUB+T, symbols:21-0061L_MXM, F.Cu at (-76.4, 180.4)
- added U1404: MAX9939AUB+T, symbols:21-0061L_MXM, F.Cu at (-76.4, 185.1)
- added U1501: TLC6C598PW, Package_SO:TSSOP-16_4.4x5mm_P0.65mm, F.Cu at (-89.7, 90.2)
- added U1502: TLC6C598PW, Package_SO:TSSOP-16_4.4x5mm_P0.65mm, F.Cu at (-89.7, 96.8)
- added U1601: TLC6C598PW, Package_SO:TSSOP-16_4.4x5mm_P0.65mm, F.Cu at (-193.4, 177.1)
- added U1701: TLC6C598PW, Package_SO:TSSOP-16_4.4x5mm_P0.65mm, F.Cu at (-138.5, 49.0)
- added U1806: TPS7A92050DBVR, Package_SON:Texas_X2SON-4_1x1mm_P0.65mm, F.Cu at (-55.4, 199.3)
- added U2001: TLV9062xD, Package_SO:SOIC-8_3.9x4.9mm_P1.27mm, F.Cu at (-153.1, 190.9)
- added U2002: LM34936RHFR, symbols:RHF0028A, F.Cu at (-148.9, 197.4)
- added U2003: STUSB4500QTR, Package_DFN_QFN:QFN-24-1EP_4x4mm_P0.5mm_EP2.7x2.7mm, F.Cu at (-184.4, 190.7)
- added U2101: TLC6C598PW, Package_SO:TSSOP-16_4.4x5mm_P0.65mm, F.Cu at (-163.7, 190.8)
- added U2102: TLC6C598PW, Package_SO:TSSOP-16_4.4x5mm_P0.65mm, F.Cu at (-163.7, 197.4)
- added U2402: USBLC6-4SC6, Package_TO_SOT_SMD:SOT-23-6, F.Cu at (-91.3, 188.1)
- added U301: OPA1692xDGK, Package_SO:VSSOP-8_3x3mm_P0.65mm, F.Cu at (-119.1, 191.2)
- added U302: AS183-92LF, Library:SOT65P220X110-6N, F.Cu at (-125.2, 179.3)
- added U303: AS183-92LF, Library:SOT65P220X110-6N, F.Cu at (-125.2, 183.1)
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Connections:
- net /DACACD/AudioBCLK renamed /microcontroller/Ctrl.qsdBCLK
- net /DACACD/AudioDIN renamed /microcontroller/Ctrl.qsdData
- net /DACACD/AudioMCLK renamed /microcontroller/Ctrl.qsdSCK
- net /DACACD/AudioSCL renamed /microcontroller/Ctrl.usbnALERT
- net /DACACD/AudioWCLK renamed /microcontroller/Ctrl.qsdWCLK
- net /microcontroller/AntFwdV renamed /microcontroller/Ctrl.txMCLK
- net /microcontroller/AntRevV renamed /microcontroller/Ctrl.usbPOK3
- net /microcontroller/PAtankSel.C0 renamed /microcontroller/Ctrl.atten12dB
- net /microcontroller/PAtankSel.C1 renamed /microcontroller/Ctrl.atten6dB
- net /microcontroller/PAtankSel.C2 renamed /microcontroller/Ctrl.atten3dB
- net /microcontroller/PAtankSel.C3 renamed /microcontroller/Ctrl.qsdNSS
- net /microcontroller/PAtankSel.C6 renamed /microcontroller/Ctrl.qsdMOSI
- net /microcontroller/PAtankSel.C7 renamed /microcontroller/FPGA.RESET
- net /microcontroller/PAtankSel.L1 renamed /microcontroller/Ctrl.txBCLK
- net /microcontroller/PAtankSel.L2 renamed /microcontroller/Ctrl.txWCLK
- net /microcontroller/PAtankSel.L3 renamed /microcontroller/Ctrl.usbPOK2
- net /microcontroller/SDpresent renamed /microcontroller/Ctrl.enable6V
- net /microcontroller/USBD3 renamed /microcontroller/Ctrl.switchSCK
- net /microcontroller/USBNXT renamed /microcontroller/Ctrl.switchMOSI
- net /microcontroller/USBSTP renamed /microcontroller/Ctrl.enable5V
- net Net-(U201-2-PF0) renamed /microcontroller/Ctrl.switchRCK
- net Net-(U201-2-PF5) renamed /microcontroller/Ctrl.enFPGAVpp
- net Net-(U201-2-PF6) renamed /microcontroller/Ctrl.enFPGAIOVdd
- C1201 pad 1: /Antenna Tuner, TR Relay/AntRx -> +3.3VA
- C1201 pad 2: Net-(IC1201-J3) -> GND
- C1202 pad 1: +3.3V -> +3.3VA
- C1203 pad 1: Net-(IC1201-J1) -> /Rx Front End/Ctrl.breune
- C1203 pad 2: Net-(C1203-Pad2) -> Net-(U1202-IN1)
- C1204 pad 1: Net-(C1203-Pad2) -> +1.65VBIAS
- C1205 pad 1: Net-(C1203-Pad2) -> Net-(U1202-COM4)
- C1206 pad 1: Net-(C1203-Pad2) -> Net-(U1202-COM3)
- C1206 pad 2: Net-(C1206-Pad2) -> Net-(U1203-INA-)
- C1207 pad 1: Net-(C1206-Pad2) -> Net-(U1202-COM4)
- C1207 pad 2: GND -> Net-(U1204-INA-)
- C1208 pad 1: Net-(C1206-Pad2) -> Net-(U1202-COM3)
- C1210 pad 1: Net-(C1206-Pad2) -> Net-(U1202-COM2)
- C1210 pad 2: Net-(C1210-Pad2) -> Net-(U1204-INA+)
- C1211 pad 1: Net-(C1210-Pad2) -> +5VA
- C1212 pad 1: Net-(C1210-Pad2) -> +5VA
- C1213 pad 1: Net-(C1210-Pad2) -> Net-(U1202-COM2)
- C1213 pad 2: /Rx Front End/BPF5/BPFout -> GND
- C1301 pad 1: /Antenna Tuner, TR Relay/AntRx -> +3.3VA
- C1301 pad 2: Net-(IC1301-J3) -> GND
- C1302 pad 1: +3.3V -> +3.3VA
- C1303 pad 1: Net-(IC1301-J1) -> /Rx Front End/QSD2/rfIn
- C1303 pad 2: Net-(C1303-Pad2) -> Net-(U1302-IN1)
- C1304 pad 1: Net-(C1303-Pad2) -> +1.65VBIAS
- C1305 pad 1: Net-(C1303-Pad2) -> Net-(U1302-COM4)
- C1306 pad 1: Net-(C1303-Pad2) -> Net-(U1302-COM3)
- C1306 pad 2: Net-(C1306-Pad2) -> Net-(U1303-INA-)
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Routing:
- added copper zone on F.Cu, net (none)
- added copper zone on F.Cu, net VBUS
- removed copper zone on F.Cu, net +12V
- removed copper zone on F.Cu, net /Power/Tx EER Envelope Buck-Boost/PA_SENSE

Commit message: Now using H bridge for differential QSE based I/Q tx
Parts:
- removed C504, C506: 10uF 250V, Capacitor_SMD:C_0805_2012Metric
- removed C505: 10uF, Capacitor_SMD:C_0805_2012Metric
- removed Q501: IRFP250NPBF, Library:TO545P530X1560X2460-3P
- removed R506: 220, Resistor_SMD:R_1206_3216Metric
- removed T502: ~, Inductor_THT:L_CommonMode_Toroid_Vertical_L38.1mm_W20.3mm_Px15.24mm_Py22.86mm_Bourns_8100
- removed T503: Bruene sampler, Library:toroid-pri-sec-ct-ft50
- removed U502: TMP110D, Package_SON:Texas_X2SON-5_0.8x0.8mm_P0.48mm
- added Q2301: EPC2037, Package_BGA:EPC_BGA-4_0.9x0.9mm_Layout2x2_P0.45mm, F.Cu at (81.7, 44.8)
- added Q2302: EPC2037, Package_BGA:EPC_BGA-4_0.9x0.9mm_Layout2x2_P0.45mm, F.Cu at (81.7, 47.3)
- added Q2303: IGB110S101XTMA1, Library:IGB110S101XTMA1, F.Cu at (71.6, 24.5)
- added Q2304: IGB110S101XTMA1, Library:IGB110S101XTMA1, F.Cu at (71.6, 30.6)
- added Q2305: IGB110S101XTMA1, Library:IGB110S101XTMA1, F.Cu at (71.6, 36.7)
- added Q2306: IGB110S101XTMA1, Library:IGB110S101XTMA1, F.Cu at (71.6, 42.8)
- added T2301: ~, Inductor_THT:L_CommonMode_Toroid_Vertical_L38.1mm_W20.3mm_Px15.24mm_Py22.86mm_Bourns_8100, F.Cu at (83.1, 24.8)
- added U2301: LMG1210RVRR, Library:RVR0019A, F.Cu at (77.5, 45.6)
- added U2302: LMG1210RVRR, Library:RVR0019A, F.Cu at (77.5, 50.1)
- C502: value 1uF -> 10uF
- C503: value 0.1uF 250V -> 10uF 250V
- R501: value 6.8 -> 49.9
- R502: value 49.9 -> 47k
- R503, R505: value 47k -> 220
- R504: value 220 -> 47k
- T501: value 3t:3t Fair-Rite 2843000202 bifilar litz 5/52/38 -> Bruene sampler; footprint Library:Fair-Rite 2843000202 bifilar #14AWG -> Library:toroid-pri-sec-ct-ft50
- U501: value UCC27511ADBV -> TMP110D; footprint Package_TO_SOT_SMD:SOT-23-6 -> Package_SON:Texas_X2SON-5_0.8x0.8mm_P0.48mm
Connections:
- net /Tx Chain/PA Tank/PA200tx renamed /Tx Chain/H-bridge-PA/PA200
- net /Tx Chain/lpfSerIn renamed /Tx Chain/tunerSerOut
- net /Tx Chain/tankSerIn renamed /Tx Chain/lpfSerOut
- C501 pad 1: 12V -> +3.3V
- C502 pad 1: +3.3V -> +5V
- C503 pad 1: Veer -> Net-(C503-Pad1)
- C503 pad 2: GND -> Net-(J501-In)
- L501 pad 3: Net-(C506-Pad1) -> Net-(C503-Pad1)
- R501 pad 1: Net-(R501-Pad1) -> Net-(K501-1-NC1)
- R501 pad 2: Net-(Q501-G) -> GND
- R502 pad 1: Net-(K501-1-NC1) -> Net-(R502-Pad1)
- R502 pad 2: GND -> /Rx Front End/txFwd
- R503 pad 1: Net-(R503-Pad1) -> /Rx Front End/txFwd
- R503 pad 2: /Rx Front End/txFwd -> GND
- R504 pad 1: /Rx Front End/txFwd -> Net-(R504-Pad1)
- R504 pad 2: GND -> /Rx Front End/txRev
- R505 pad 1: Net-(R505-Pad1) -> /Rx Front End/txRev
- R505 pad 2: /Rx Front End/txRev -> GND
- T501 pad 1: Net-(U501-OUTH) -> /Tx Chain/Tx LPFs/TxOut
- T501 pad 2: Net-(U501-OUTL) -> /Tx Chain/Antenna Tuner/rig
- T501 pad 3: Net-(R501-Pad1) -> GND
- T501 pad 4: GND -> Net-(R504-Pad1)
- U501 pad 1: 12V -> GND
- U501 pad 2: Net-(U501-OUTH) -> /Tx Chain/Ctrl.tmpSCL
- U501 pad 3: Net-(U501-OUTL) -> GND
- U501 pad 4: GND -> /Tx Chain/Ctrl.tmpSDA
- U501 pad 5: GND -> +3.3V
- U602 pad 23: unconnected-(U602-1-IOT_37a-Pad23) -> /FPGA/PAI-
- U602 pad 25: /FPGA/PAgate -> /FPGA/PAI+
- U602 pad 26: unconnected-(U602-1-IOT_39a-Pad26) -> /FPGA/PAQ-
- U602 pad 27: unconnected-(U602-1-IOT_38b-Pad27) -> /FPGA/PAQ+
