File: hw/_autosave-NexRig.kicad_pcb (KiCad board)
At the start: 6 copper layers, 300 x 200 mm, 623 parts, among them IC2001 LTC3779IFE#PBF, J201 68710814022, J202 FTSH-105-01-L-DV-K, J2101 USB C power only, J2401 RJ45_Abracon_ARJP11A-MASA-B-A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, J501 SMA, K1601 G2RL-2, K1602 G2RL-2, K1603 G2RL-2, K1604 G2RL-2, K1605 G2RL-2, K1701 G2RL-2, K1702 G2RL-2, K1703 G2RL-2, K1704 G2RL-2, K1705 G2RL-2, K1706 G2RL-2, K1707 G2RL-2, K2101 G2RL-2, K2102 G2RL-2, K2103 G2RL-2, K2104 G2RL-2, K2105 G2RL-2, K2106 G2RL-2, K2107 G2RL-2, K2108 G2RL-2, K2109 G2RL-2, K501 G2RL-2, K701 G2RL-2, K702 G2RL-2, K703 G2RL-2, Q2001 BSC360N15NS3 G, Q2002 BSC360N15NS3 G, Q2003 BSC360N15NS3 G, Q2004 BSC360N15NS3 G, Q2101 SQJ433EP, Q2303 EPC2207, Q2304 EPC2207, Q2305 EPC2207, Q2306 EPC2207, Q2307 EPC2207, Q2308 EPC2207, T301 12t primary : 6T #26 trifilar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, T502 16t:8t bifilar #18AWG FT140-43, U1201 SZNUP1105LT1G, U1203 MAX9939AUB+T, U1204 MAX9939AUB+T, U1301 SZNUP1105LT1G, U1303 MAX9939AUB+T, U1304 MAX9939AUB+T, U1401 SZNUP1105LT1G, U1403 MAX9939AUB+T, U1404 MAX9939AUB+T, U1501 SN74LVC04APW, U1502 SN74LVC04APW, U1503 AS183-92LF, U1504 MCP23S17, U1505 AS183-92LF, U1506 AS183-92LF, U1507 AS183-92LF, U1508 AS183-92LF, U1509 AS183-92LF, U1510 AS183-92LF, U1511 AS183-92LF, U1512 AS183-92LF, U1513 AS183-92LF, U1514 AS183-92LF, U1515 AS183-92LF, U1601 TLC6C598PW, U1701 TLC6C598PW, U1801 LMR43610R3RPER, U1802 LMR51430, U1803 TPS7A2012DQN, U1805 LMR51430, U1806 TPS7A92050DBVR, U1807 TPS7A2033DQN, U1901 AS183-92LF, U1902 AS183-92LF, U2001 TLV9062xD, U2002 NVTFS6H888NLTAG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

Commit message: Fixed GPIO assignments. Fixed symbol for GRL2-2 relays.
Parts:
- moved U2003 554.4 mm to (127.3, -220.7)
- moved C2015 547.0 mm to (112.4, -208.1)
- moved C2016 547.0 mm to (112.4, -199.9)
- moved R2101 538.0 mm to (112.3, -229.3)
- moved R2102 538.0 mm to (112.3, -226.8)
- moved R2103 538.0 mm to (112.3, -224.3)
- moved U2103 537.6 mm to (121.2, -189.4)
- moved R2104 537.5 mm to (116.3, -244.4)
- moved R2105 537.5 mm to (116.3, -241.9)
- moved R2107 537.5 mm to (116.3, -239.4)
- moved R2108 537.5 mm to (116.3, -236.9)
- moved Q2101 536.9 mm to (122.7, -241.7)
- moved C1819 535.6 mm to (127.8, -203.1)
- moved R2008 534.2 mm to (108.3, -244.4)
- moved R2009 534.2 mm to (108.3, -241.9)
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