File: hw/NexRig.kicad_pcb (KiCad board)
At the start: 6 copper layers, 300 x 200 mm, 690 parts, among them J7701 68710814022, J7702 FTSH-105-01-L-DV-K, J7703 SMA, J7706 USB C power only, J7707 RJ45_Abracon_ARJP11A-MASA-B-A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, K7701 G5Q-14-05, K7702 TQ2-5V-functional, K7703 G5Q-14-05, K7704 G5Q-14-05, K7705 G5Q-14-05, K7706 G5Q-14-05, K7707 G5Q-14-05, K7708 G5Q-14-05, K7709 G5Q-14-05, K7710 G5Q-14-05, K7711 G5Q-14-05, K7712 G5Q-14-05, K7713 G5Q-14-05, K7714 G5Q-14-05, K7715 G5Q-14-05, K7716 G5Q-14-05, K7717 G5Q-14-05, K7718 G5Q-14-05, K7719 G5Q-14-05, K7720 G5Q-14-05, K7721 G5Q-14-05, K7722 G5Q-14-05, K7723 G5Q-14-05, K7724 G5Q-14-05, K7725 G5Q-14-05, K7726 G5Q-14-05, K7727 G5Q-14-05, K7728 G5Q-14-05, K7729 G5Q-14-05, K7730 G5Q-14-05, K7731 G5Q-14-05, K7732 G5Q-14-05, K7733 G5Q-14-05, K7734 G5Q-14-05, K7735 G5Q-14-05, K7736 G5Q-14-05, K7737 G5Q-14-05, Q7701 EPC2207, Q7702 EPC2207, Q7703 EPC2207, Q7704 EPC2207, Q7705 EPC2207, Q7706 EPC2207, Q7707 EPC2207, Q7708 EPC2207, Q7709 BSC360N15NS3 G, Q7710 BSC360N15NS3 G, Q7711 BSC360N15NS3 G, Q7712 BSC360N15NS3 G, Q7713 SQJ433EP, Q7717 IPB026N06NATMA1, T7701 12t primary : 6T #26 trifilar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, T7702 GUANELLA-2P-1S, T7704 GUANELLA-2P-1S, U7701 STM32H753ZIT6, U7702 MC74HCT125ADTR2G-Q, U7703 OPA1692xDGK, U7704 SN74LVC04APW, U7706 AS183-92LF, U7707 AS183-92LF, U7708 AS183-92LF, U7709 AK5578EN, U7710 LMG1210RVRR, U7711 PCT2075DP, U7712 ECP5-LFE5U-12, U7713 TPIC6C595PWR, U7714 LMG1210RVRR, U7715 LMG1210RVRR, U7716 LMG1210RVRR, U7717 SZNUP1105LT1G, U7718 TS3A4751RUCR, U7719 MAX9939AUB+T, U7720 MAX9939AUB+T, U7721 SZNUP1105LT1G, U7722 TS3A4751RUCR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

Commit message: Checkpoint for yet another merge
Parts:
- removed C7730: 100nF, Capacitor_SMD:C_0603_1608Metric
- removed FID101, FID102, FID103: Fiducial, Fiducial:Fiducial_0.5mm_Mask2mm
- removed MH101, MH102, MH103, MH104: MountingHole, MountingHole:MountingHole_3.2mm_M3_ISO7380_Pad
- removed U7705: ~, Library:SOT65P220X110-6N
- J7703: value SMA -> ANT
- moved MH7702 450.3 mm to (160.0, -168.7)
- moved MH7703 444.1 mm to (160.0, -360.7)
- moved FID7702 442.9 mm to (155.7, -166.7)
- moved FID7703 433.2 mm to (155.7, -362.7)
- moved GD7701 360.6 mm to (158.2, -340.2), turned to 180 degrees
- moved J7703 348.7 mm to (159.2, -349.2), turned to 180 degrees
- moved R7723 314.8 mm to (153.2, -350.5), turned to 90 degrees
- moved C7764 293.9 mm to (162.0, -334.0), turned to 90 degrees
- moved C7763 289.9 mm to (159.6, -334.0), turned to 90 degrees
- moved C7762 285.9 mm to (157.3, -334.0), turned to 90 degrees
- moved C7761 281.9 mm to (155.0, -334.0), turned to 90 degrees
- moved FID7701 189.7 mm to (-127.3, -166.7)
- moved MH7701 187.7 mm to (-132.0, -168.7)
- moved MH7704 171.2 mm to (-132.0, -360.7)
