File: hw/eer-buckboost.kicad_sch (KiCad schematic)
At the start: 60 parts, among them Q7709 BSC360N15NS3 G, Q7710 BSC360N15NS3 G, Q7711 BSC360N15NS3 G, Q7712 BSC360N15NS3 G, U7756 TLV9062xD, U7757 NVTFS6H888NLTAG, U7758 LTC3779IFE#PBF, U7759 PCT2075DP

Commit message: All symbols and footprints seem right now, and schematic again imports into PCB without error
Parts:
- renumbered C7921 to C7920, C7922 to C7921, C7923 to C7922, C7924 to C7923, C7925 to C7924, C7926 to C7925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
