File: hw/tx-bridge.kicad_sch (KiCad schematic)
At the start: 9 parts, among them Q7701 EPC2207, Q7702 EPC2207, U7709 LMG1210RVRR

Commit message: Checkpoint. FPGA is mostly done (need a check!). Working on new LPFs. Need inductor footprints and to fix a bunch of broken/missing footprints.
Parts:
- C7754: footprint Capacitor_SMD:C_0805_2012Metric -> Capacitor_SMD:C_0603_1608Metric
- C7755: footprint Capacitor_SMD:C_0201_0603Metric -> Capacitor_SMD:C_0603_1608Metric
Changed lines of the file:
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@@
 			)
 		)
-		(property "Footprint" "Capacitor_SMD:C_0805_2012Metric"
+		(property "Footprint" "Capacitor_SMD:C_0603_1608Metric"
 			(at 63.8048 95.25 0)
 			(effects
@@
 			)
 		)
-		(property "Footprint" "Capacitor_SMD:C_0201_0603Metric"
+		(property "Footprint" "Capacitor_SMD:C_0603_1608Metric"
 			(at 129.8448 99.06 0)
 			(effects

Commit message: OK I have part numbers for consolidated caps, resistors, inductors and all ICs are now Uxxx refdes.
Parts:
- C7754: Manufacturer_Name (none) -> Kemet; Manufacturer_Part_Number (none) -> C0805F104K1RACAUTO; Mouser Part Number (none) -> 80-C0805F104K1RAUTO
- C7755: Manufacturer_Name (none) -> Murata; Manufacturer_Part_Number (none) -> GXT155R71E223KE01D; Mouser Part Number (none) -> 81-GXT155R71E223KE1D
- C7756, C7757: footprint Capacitor_SMD:C_0805_2012Metric -> Capacitor_SMD:C_0603_1608Metric; Manufacturer_Name (none) -> Taoup Uidem; Manufacturer_Part_Number (none) -> 81-GXT155R71E223KE1D; Mouser Part Number (none) -> 963-MLAST168BB5106MT
- C7758: Manufacturer_Name (none) -> Murata; Manufacturer_Part_Number (none) -> GRM155R61E105KE11D; Mouser Part Number (none) -> 81-GRM155R61E105KE1D
- renumbered U7709 to U7710

Commit message: All symbols and footprints seem right now, and schematic again imports into PCB without error
Parts:
- renumbered C7754 to C7753, C7755 to C7754, C7756 to C7755, C7757 to C7756, C7758 to C7757, U7710 to U7709
