File: hw/rx-presel.kicad_sch (KiCad schematic)
At the start: 55 parts, among them U1501 SN74LVC04APW, U1502 SN74LVC04APW, U1503 AS183-92LF, U1504 MCP23S17, U1505 AS183-92LF, U1506 AS183-92LF, U1507 AS183-92LF, U1508 AS183-92LF, U1509 AS183-92LF, U1510 AS183-92LF, U1511 AS183-92LF, U1512 AS183-92LF, U1513 AS183-92LF, U1514 AS183-92LF, U1515 AS183-92LF

Commit message: I think I have finished the relay conversion and 5V SPI I/O expander crap
Parts:
- renumbered C1501 to C7834, C1502 to C7835, C1503 to C7836, C1504 to C7837, C1505 to C7838, C1506 to C7839, C1507 to C7840, C1508 to C7841, C1509 to C7842, C1510 to C7843, C1511 to C7844, C1512 to C7845, C1513 to C7846, C1514 to C7847, L1501 to L7703, L1502 to L7704, R1501 to R7763, R1502 to R7764, R1503 to R7765, R1504 to R7766, R1505 to R7767, R1506 to R7768, R1507 to R7769, R1508 to R7770, R1509 to R7771, R1510 to R7772, R1511 to R7773, R1512 to R7774, R1513 to R7775, R1514 to R7776, R1515 to R7777, R1516 to R7778, R1517 to R7779, R1518 to R7780, R1519 to R7781, R1520 to R7782, R1521 to R7783, R1522 to R7784, R1523 to R7785, R1524 to R7786, U1501 to U7724, U1502 to U7725, U1503 to U7726, U1504 to U7727, U1505 to U7728, U1506 to U7729, U1507 to U7730, U1508 to U7731, U1509 to U7732, U1510 to U7733, U1511 to U7734, U1512 to U7735, U1513 to U7736, U1514 to U7737, U1515 to U7738

Commit message: Starting to build guanella transformers. Mostly converted to 1-2-1 tx, but FPGA still to do.
Parts:
- renumbered C7834 to C7857, C7835 to C7858, C7836 to C7859, C7837 to C7860, C7838 to C7861, C7839 to C7862, C7840 to C7863, C7841 to C7864, C7842 to C7865, C7843 to C7866, C7844 to C7867, C7845 to C7868, C7846 to C7869, C7847 to C7870, U7724 to U7730, U7725 to U7731, U7726 to U7732, U7727 to U7733, U7728 to U7734, U7729 to U7735, U7730 to U7736, U7731 to U7737, U7732 to U7738, U7733 to U7739, U7734 to U7740, U7735 to U7741, U7736 to U7742, U7737 to U7743, U7738 to U7744

Commit message: Checkpoint. FPGA is mostly done (need a check!). Working on new LPFs. Need inductor footprints and to fix a bunch of broken/missing footprints.
Parts:
- C7859, C7860, C7862, C7863, C7864, C7865, C7866, C7867, C7868, C7869, C7870: footprint Capacitor_SMD:C_0201_0603Metric -> Capacitor_SMD:C_0603_1608Metric
Changed lines of the file:
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@@
 			)
 		)
-		(property "Footprint" "Capacitor_SMD:C_0201_0603Metric"
+		(property "Footprint" "Capacitor_SMD:C_0603_1608Metric"
 			(at 103.8352 148.59 0)
 			(effects
@@
 			)
 		)
-		(property "Footprint" "Capacitor_SMD:C_0201_0603Metric"
+		(property "Footprint" "Capacitor_SMD:C_0603_1608Metric"
 			(at 70.8152 148.59 0)
 			(effects
@@
 			)
 		)
-		(property "Footprint" "Capacitor_SMD:C_0201_0603Metric"
+		(property "Footprint" "Capacitor_SMD:C_0603_1608Metric"
 			(at 153.3652 148.59 0)
 			(effects
@@
 			)
 		)
-		(property "Footprint" "Capacitor_SMD:C_0201_0603Metric"
+		(property "Footprint" "Capacitor_SMD:C_0603_1608Metric"
 			(at 186.3852 148.59 0)
 			(effects
@@
 			)
 		)
-		(property "Footprint" "Capacitor_SMD:C_0201_0603Metric"
+		(property "Footprint" "Capacitor_SMD:C_0603_1608Metric"
 			(at 87.3252 148.59 0)
 			(effects
@@
 			)
 		)
-		(property "Footprint" "Capacitor_SMD:C_0201_0603Metric"
+		(property "Footprint" "Capacitor_SMD:C_0603_1608Metric"
 			(at 219.4052 148.59 0)
 			(effects
@@
 			)
 		)
-		(property "Footprint" "Capacitor_SMD:C_0201_0603Metric"
+		(property "Footprint" "Capacitor_SMD:C_0603_1608Metric"
 			(at 136.8552 148.59 0)
 			(effects
@@
 			)
 		)
-		(property "Footprint" "Capacitor_SMD:C_0201_0603Metric"
+		(property "Footprint" "Capacitor_SMD:C_0603_1608Metric"
 			(at 235.9152 148.59 0)
 			(effects
@@
 			)
 		)
-		(property "Footprint" "Capacitor_SMD:C_0201_0603Metric"
+		(property "Footprint" "Capacitor_SMD:C_0603_1608Metric"
 			(at 202.8952 148.59 0)
 			(effects
@@
 			)
 		)
-		(property "Footprint" "Capacitor_SMD:C_0201_0603Metric"
+		(property "Footprint" "Capacitor_SMD:C_0603_1608Metric"
 			(at 169.8752 148.59 0)
 			(effects
@@
 			)
 		)
-		(property "Footprint" "Capacitor_SMD:C_0201_0603Metric"
+		(property "Footprint" "Capacitor_SMD:C_0603_1608Metric"
 			(at 120.3452 148.59 0)
 			(effects

Commit message: OK I have part numbers for consolidated caps, resistors, inductors and all ICs are now Uxxx refdes.
Parts:
- C7868: renamed from C7857; footprint Capacitor_SMD:C_0805_2012Metric -> Capacitor_SMD:C_0402_1005Metric; Manufacturer_Name (none) -> Murata; Manufacturer_Part_Number (none) -> GRM155R61E105KE11D; Mouser Part Number (none) -> 81-GRM155R61E105KE1D; cap-type X7R -> X5R; working-voltage 50V -> 25V
- C7869: renamed from C7858; footprint Capacitor_SMD:C_0805_2012Metric -> Capacitor_SMD:C_0402_1005Metric; Manufacturer_Name (none) -> Murata; Manufacturer_Part_Number (none) -> GRM155R61E105KE11D; Mouser Part Number (none) -> 81-GRM155R61E105KE1D; cap-type X7R -> X5R; working-voltage 50V -> 25V
- C7870: renamed from C7859; Manufacturer_Name (none) -> TDK; Manufacturer_Part_Number (none) -> CGA3E2C0G1H080D080AA; Mouser Part Number (none) -> 810-CGA3E2C0G1H080D; working-voltage 250 -> 50V
- C7871: renamed from C7860; value 16pF -> 15pF; Manufacturer_Name (none) -> TDK; Manufacturer_Part_Number (none) -> CGA3E2C0G1H150J080AA; Mouser Part Number (none) -> 810-CGA3E2C0G1H150J; working-voltage 250V -> 50V
- C7872: renamed from C7861; footprint Capacitor_SMD:C_0805_2012Metric -> Capacitor_SMD:C_0402_1005Metric; Manufacturer_Name (none) -> Murata; Manufacturer_Part_Number (none) -> GRM155R61E105KE11D; Mouser Part Number (none) -> 81-GRM155R61E105KE1D; cap-type X7R -> X5R; working-voltage 50V -> 25V
- C7873: renamed from C7862; value 32pF -> 33pF; Manufacturer_Name (none) -> TDK; Manufacturer_Part_Number (none) -> CGA3E2C0G1H330J080AA; Mouser Part Number (none) -> 810-CGA3E2C0G1H330J; working-voltage 250V -> 50V
- C7874: renamed from C7863; value 64pF -> 68pF; Manufacturer_Name (none) -> TDK; Manufacturer_Part_Number (none) -> CGA3E2C0G1H680J080AA; Mouser Part Number (none) -> 810-CGA3E2C0G1H680J; working-voltage 250V -> 50V
- C7875: renamed from C7864; value 128pF -> 120pF; Manufacturer_Name (none) -> TDK; Manufacturer_Part_Number (none) -> CGA3E2C0G1H121J080AA; Mouser Part Number (none) -> 810-CGA3E2C0G1H121J; working-voltage 250V -> 50V
- C7876: renamed from C7865; value 256pF -> 250pF; Manufacturer_Name (none) -> Kyocera AVX; Manufacturer_Part_Number (none) -> 06035A251JAT2A; Mouser Part Number (none) -> 581-06035A251J; working-voltage 250V -> 50V
- C7877: renamed from C7866; value 512pF -> 560pF; Manufacturer_Name (none) -> TDK; Manufacturer_Part_Number (none) -> CGA3E2C0G1H561J080AA; Mouser Part Number (none) -> 810-CGA3E2C0G1H561J
- C7878: renamed from C7867; value 1024pF -> 1nF; Manufacturer_Name (none) -> TDK; Manufacturer_Part_Number (none) -> C1608C0G1H102J080AA; Mouser Part Number (none) -> 810-C1608C0G1H102J; working-voltage 250V -> 50V
- C7879: renamed from C7868; value 2048pF -> 2.2nF; Manufacturer_Name (none) -> TDK; Manufacturer_Part_Number (none) -> CGA3E2C0G1H222J080AE; Mouser Part Number (none) -> 810-CGA3E2C0G1H222J8; working-voltage 250 -> 50V
- C7880: renamed from C7869; value 4096pF -> 3.9nF; Manufacturer_Name (none) -> TDK; Manufacturer_Part_Number (none) -> CGA3E2C0G1H392J080AA; Mouser Part Number (none) -> 810-CGA3E2C0G1H392J; working-voltage 250V -> 50V
- C7881: renamed from C7870; value 8192pF -> 8.2nF; Manufacturer_Name (none) -> TDK; Manufacturer_Part_Number (none) -> CGA3E2C0G1H822J080AE; Mouser Part Number (none) -> 810-CGA3E2C0G1H822J8; working-voltage 250V -> 50V
- renumbered R7763 to R7767, R7764 to R7768, R7765 to R7769, R7766 to R7770, R7767 to R7771, R7768 to R7772, R7769 to R7773, R7770 to R7774, R7771 to R7775, R7772 to R7776, R7773 to R7777, R7774 to R7778, R7775 to R7779, R7776 to R7780, R7777 to R7781, R7778 to R7782, R7779 to R7783, R7780 to R7784, R7781 to R7785, R7782 to R7786, R7783 to R7787, R7784 to R7788, R7785 to R7789, R7786 to R7790, U7730 to U7729, U7731 to U7730, U7732 to U7731, U7733 to U7732, U7734 to U7733, U7735 to U7734, U7736 to U7735, U7737 to U7736, U7738 to U7737, U7739 to U7738, U7740 to U7739, U7741 to U7740, U7742 to U7741, U7743 to U7742, U7744 to U7743

Commit message: All symbols and footprints seem right now, and schematic again imports into PCB without error
Parts:
- renumbered C7868 to C7867, C7869 to C7868, C7870 to C7869, C7871 to C7870, C7872 to C7871, C7873 to C7872, C7874 to C7873, C7875 to C7874, C7876 to C7875, C7877 to C7876, C7878 to C7877, C7879 to C7878, C7880 to C7879, C7881 to C7880, U7729 to U7728, U7730 to U7729, U7731 to U7730, U7732 to U7731, U7733 to U7732, U7734 to U7733, U7735 to U7734, U7736 to U7735, U7737 to U7736, U7738 to U7737, U7739 to U7738, U7740 to U7739, U7741 to U7740, U7742 to U7741, U7743 to U7742

Commit message: I'm thinking I might make a NexRx with just the rx portion of this design first to test my skills and capabilities.
Parts:
- renumbered C7867 to C7866, C7868 to C7867, C7869 to C7868, C7870 to C7869, C7871 to C7870, C7872 to C7871, C7873 to C7872, C7874 to C7873, C7875 to C7874, C7876 to C7875, C7877 to C7876, C7878 to C7877, C7879 to C7878, C7880 to C7879

Commit message: Off to a great start building just the NexRx
Parts:
- renumbered C7866 to C1501, C7867 to C1502, C7868 to C1503, C7869 to C1504, C7870 to C1505, C7871 to C1506, C7872 to C1507, C7873 to C1508, C7874 to C1509, C7875 to C1510, C7876 to C1511, C7877 to C1512, C7878 to C1513, C7879 to C1514, L7703 to L1501, L7704 to L1502, R7767 to R1501, R7768 to R1502, R7769 to R1503, R7770 to R1504, R7771 to R1505, R7772 to R1506, R7773 to R1507, R7774 to R1508, R7775 to R1509, R7776 to R1510, R7777 to R1511, R7778 to R1512, R7779 to R1513, R7780 to R1514, R7781 to R1515, R7782 to R1516, R7783 to R1517, R7784 to R1518, R7785 to R1519, R7786 to R1520, R7787 to R1521, R7788 to R1522, R7789 to R1523, R7790 to R1524, U7728 to U1501, U7729 to U1502, U7730 to U1503, U7731 to U1504, U7732 to U1505, U7733 to U1506, U7734 to U1507, U7735 to U1508, U7736 to U1509, U7737 to U1510, U7738 to U1511, U7739 to U1512, U7740 to U1513, U7741 to U1514, U7742 to U1515

Commit message: All ERC pass. Import to PCB works with no footprints missing.
Parts:
- U1501, U1502: footprint PW14 -> Library:PW14
- U1503, U1505, U1506, U1507, U1508, U1509, U1510, U1511, U1512, U1513, U1514, U1515: footprint SOT65P220X110-6N -> Library:SOT65P220X110-6N
- U1504: footprint QFN65P600X600X100-29N-D -> Library:QFN65P600X600X100-29N-D
Changed lines of the file:
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@@
 			)
 		)
-		(property "Footprint" "SOT65P220X110-6N"
+		(property "Footprint" "Library:SOT65P220X110-6N"
 			(at 346.38 148.59 0)
 			(effects
@@
 			)
 		)
-		(property "Footprint" "PW14"
+		(property "Footprint" "Library:PW14"
 			(at 33.02 44.45 0)
 			(effects
@@
 			)
 		)
-		(property "Footprint" "SOT65P220X110-6N"
+		(property "Footprint" "Library:SOT65P220X110-6N"
 			(at 123.52 148.59 0)
 			(effects
@@
 			)
 		)
-		(property "Footprint" "SOT65P220X110-6N"
+		(property "Footprint" "Library:SOT65P220X110-6N"
 			(at 57.48 148.59 0)
 			(effects
@@
 			)
 		)
-		(property "Footprint" "SOT65P220X110-6N"
+		(property "Footprint" "Library:SOT65P220X110-6N"
 			(at 73.99 148.59 0)
 			(effects
@@
 			)
 		)
-		(property "Footprint" "SOT65P220X110-6N"
+		(property "Footprint" "Library:SOT65P220X110-6N"
 			(at 40.97 148.59 0)
 			(effects
@@
 			)
 		)
-		(property "Footprint" "SOT65P220X110-6N"
+		(property "Footprint" "Library:SOT65P220X110-6N"
 			(at -25.07 148.59 0)
 			(effects
@@
 			)
 		)
-		(property "Footprint" "SOT65P220X110-6N"
+		(property "Footprint" "Library:SOT65P220X110-6N"
 			(at 107.01 148.59 0)
 			(effects
@@
 			)
 		)
-		(property "Footprint" "PW14"
+		(property "Footprint" "Library:PW14"
 			(at 33.02 81.28 0)
 			(effects
@@
 			)
 		)
-		(property "Footprint" "SOT65P220X110-6N"
+		(property "Footprint" "Library:SOT65P220X110-6N"
 			(at 90.5 148.59 0)
 			(effects
@@
 			)
 		)
-		(property "Footprint" "QFN65P600X600X100-29N-D"
+		(property "Footprint" "Library:QFN65P600X600X100-29N-D"
 			(at 107.95 145.796 0)
 			(effects
@@
 			)
 		)
-		(property "Footprint" "SOT65P220X110-6N"
+		(property "Footprint" "Library:SOT65P220X110-6N"
 			(at 140.03 148.59 0)
 			(effects
@@
 			)
 		)
-		(property "Footprint" "SOT65P220X110-6N"
+		(property "Footprint" "Library:SOT65P220X110-6N"
 			(at 7.95 148.59 0)
 			(effects
@@
 			)
 		)
-		(property "Footprint" "SOT65P220X110-6N"
+		(property "Footprint" "Library:SOT65P220X110-6N"
 			(at 24.46 148.59 0)
 			(effects
@@
 			)
 		)
-		(property "Footprint" "SOT65P220X110-6N"
+		(property "Footprint" "Library:SOT65P220X110-6N"
 			(at -8.56 148.59 0)
 			(effects
