File: hw/NexRx.kicad_pcb (KiCad board)
At the start: 6 copper layers, 99 x 99 mm, 359 parts, among them J101 SMA, J1201 pwr+data, J201 68710814022, J202 FTSH-105-01-L-DV-K, T101 INPUT, T301 BN-43-202, 200 : 3-way 50 ohm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, U1001 AS183-92LF, U1002 AS183-92LF, U1101 AS183-92LF, U1102 AS183-92LF, U1201 LMR51430, U1202 TPS6123, U1203 TPS7A92050DBVR, U1204 TPS22918DBVT, U1205 TPS7A2033DQN, U1206 TPS22918DBVR, U1207 TPS74612PQWDRBRQ1, U1301 ICE40UP5K-SG48I, U1401 MAX9939AUB+T, U1501 MAX9939AUB+T, U1601 MAX9939AUB+T, U1701 MAX9939AUB+T, U1801 MAX9939AUB+T, U1901 MAX9939AUB+T, U2001 MCP23S17, U2002 SN74LVC2G14DBV, U2003 SN74LVC2G14DBV, U2004 SN74LVC2G14DBV, U2005 SN74LVC2G14DBV, U2006 SN74LVC2G14DBV, U2007 SN74LVC2G14DBV, U2008 SN74LVC2G14DBV, U2009 SN74LVC2G14DBV, U201 STM32H753VITx, U202 USB3343, U301 OPA1692xDGK, U302 AK5578EN, U401 TS3A4751RUCR, U501 TS3A4751RUCR, U601 TS3A4751RUCR, U701 AS183-92LF, U702 AS183-92LF, U703 AS183-92LF, U704 AS183-92LF, U705 AS183-92LF, U706 AS183-92LF, U707 AS183-92LF, U708 AS183-92LF, U709 AS183-92LF, U710 AS183-92LF, U711 AS183-92LF, U712 AS183-92LF, U801 AS183-92LF, U802 AS183-92LF, U901 AS183-92LF, U902 AS183-92LF, Y1301 40MHz, Y201 25MHz, Y202 26MHz

Commit message: Checkpoint to prep for full scale Gemini review and cleanup
Routing:
- net GND: track 311.5 -> 311.4 mm, vias 264 -> 269

Commit message: hw: remove ethernet page (page 24) and sync BOM metadata
Parts:
- D101: value STS321150B100AH -> TPD1E0B04DPY; footprint Diode_SMD:Infineon_SG-WLL-2-3_0.58x0.28_P0.36mm -> Diode_SMD:D_SOD-882
- D301: value CDSOD323-TxxC -> 19V
- J101: footprint Library:RFPCSMA27F -> Library:733910083
- J1201: footprint Library:UJ20CHGMSMT4P16TR -> Connector_USB:USB_C_Receptacle_HRO_TYPE-C-31-M-12
- T301: value BN-43-202, 200 : 3-way 50 ohm, pentafilar 2 turns #30 AWG -> BN-43-202, 200 : 3-way 22 ohm, hexafilar 2 turns #30 AWG
- U1204: value TPS22918DBVT -> TPS22918DBVR
- U1206: footprint Library:SOT95P280X145-6N -> Package_TO_SOT_SMD:SOT-23-6
- U301: value OPA1692xDGK -> OPA1692IDGK
- Y201: value 25MHz -> 26MHz
- moved J101 4.04 mm to (29.5, -331.9)
Connections:
- C101 pad 2: Net-(J101-In) -> Net-(C101-Pad2)
- GD101 pad 1: Net-(J101-In) -> Net-(C101-Pad2)
- GD101 pad 3: Net-(J101-In) -> Net-(C101-Pad2)
- J101 pad 1: Net-(J101-In) -> GND
- J101 pad 5: GND -> Net-(C101-Pad2)
- R101 pad 1: Net-(J101-In) -> Net-(C101-Pad2)
Routing:
- net Net-(C101-Pad2): track 0.00 -> 26.1 mm
- net Net-(J101-In): track 25.7 -> 0.00 mm
