File: hw/gpio-expander.kicad_sch (KiCad schematic)
At the start: 8 parts, among them U2001 STM32C011F_4-6_Ux, U2002 STM32C011F_4-6_Ux, U2003 STM32C011F_4-6_Ux, U2004 STM32C011F_4-6_Ux

Commit message: Preparing to take another swing at layout for rf200. I THINK the previous gaffes have been repaired elsewhere - cause by BOM machinations and my clumsiness.
Parts:
- U2001, U2002, U2003, U2004: value STM32C011F_4-6_Ux -> STM32C011F4U6TR; JLCPCBpn (none) -> C5456188; Manufacturer_Name (none) -> STMicro; Manufacturer_Part_Number (none) -> ST STM32C011F4U6TR
Changed lines of the file:
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@@
 	)
 	(image
-		(at 220.98 97.79)
+		(at 220.98 80.01)
+		(scale 1.79089)
 		(data "iVBORw0KGgoAAAANSUhEUgAAAXEAAAILCAIAAACRtDvJAAAAA3NCSVQICAjb4U/gAAAgAElEQVR4"
 			"nO3dd0BTV/8/8JNBCEskCTOpA0VUcLQuWqlQtxTcFRG1KloVB2jdq1gVqziqonWgddQKpVq1LirW"
@@
 			)
 		)
-		(property "Value" "STM32C011F_4-6_Ux"
+		(property "Value" "STM32C011F4U6TR"
 			(at 92.3133 41.91 0)
 			(effects
@@
 		)
 		(property "Description" "STMicroelectronics Arm Cortex-M0+ MCU, 16-32KB flash, 6KB RAM, 48 MHz, 2.0-3.6V, 18 GPIO, UFQFPN20"
+			(at 90.17 64.77 0)
+			(effects
+				(font
+					(size 1.27 1.27)
+				)
+				(hide yes)
+			)
+		)
+		(property "cap-type" ""
+			(at 90.17 64.77 0)
+			(effects
+				(font
+					(size 1.27 1.27)
+				)
+			)
+		)
+		(property "r-power" ""
+			(at 90.17 64.77 0)
+			(effects
+				(font
+					(size 1.27 1.27)
+				)
+			)
+		)
+		(property "label" ""
+			(at 90.17 64.77 0)
+			(effects
+				(font
+					(size 1.27 1.27)
+				)
+			)
+		)
+		(property "JLCPCBpn" "C5456188"
+			(at 90.17 64.77 0)
+			(effects
+				(font
+					(size 1.27 1.27)
+				)
+				(hide yes)
+			)
+		)
+		(property "Manufacturer_Name" "STMicro"
+			(at 90.17 64.77 0)
+			(effects
+				(font
+					(size 1.27 1.27)
+				)
+				(hide yes)
+			)
+		)
+		(property "Manufacturer_Part_Number" "ST STM32C011F4U6TR"
 			(at 90.17 64.77 0)
 			(effects
@@
 			)
 		)
-		(property "Value" "STM32C011F_4-6_Ux"
+		(property "Value" "STM32C011F4U6TR"
 			(at 155.8133 118.11 0)
 			(effects
@@
 		)
 		(property "Description" "STMicroelectronics Arm Cortex-M0+ MCU, 16-32KB flash, 6KB RAM, 48 MHz, 2.0-3.6V, 18 GPIO, UFQFPN20"
+			(at 153.67 140.97 0)
+			(effects
+				(font
+					(size 1.27 1.27)
+				)
+				(hide yes)
+			)
+		)
+		(property "cap-type" ""
+			(at 153.67 140.97 0)
+			(effects
+				(font
+					(size 1.27 1.27)
+				)
+			)
+		)
+		(property "r-power" ""
+			(at 153.67 140.97 0)
+			(effects
+				(font
+					(size 1.27 1.27)
+				)
+			)
+		)
+		(property "label" ""
+			(at 153.67 140.97 0)
+			(effects
+				(font
+					(size 1.27 1.27)
+				)
+			)
+		)
+		(property "JLCPCBpn" "C5456188"
+			(at 153.67 140.97 0)
+			(effects
+				(font
+					(size 1.27 1.27)
+				)
+				(hide yes)
+			)
+		)
+		(property "Manufacturer_Name" "STMicro"
+			(at 153.67 140.97 0)
+			(effects
+				(font
+					(size 1.27 1.27)
+				)
+				(hide yes)
+			)
+		)
+		(property "Manufacturer_Part_Number" "ST STM32C011F4U6TR"
 			(at 153.67 140.97 0)
 			(effects
@@
 			)
 		)
-		(property "Value" "STM32C011F_4-6_Ux"
+		(property "Value" "STM32C011F4U6TR"
 			(at 93.5833 119.38 0)
 			(effects
@@
 		)
 		(property "Description" "STMicroelectronics Arm Cortex-M0+ MCU, 16-32KB flash, 6KB RAM, 48 MHz, 2.0-3.6V, 18 GPIO, UFQFPN20"
+			(at 91.44 142.24 0)
+			(effects
+				(font
+					(size 1.27 1.27)
+				)
+				(hide yes)
+			)
+		)
+		(property "cap-type" ""
+			(at 91.44 142.24 0)
+			(effects
+				(font
+					(size 1.27 1.27)
+				)
+			)
+		)
+		(property "r-power" ""
+			(at 91.44 142.24 0)
+			(effects
+				(font
+					(size 1.27 1.27)
+				)
+			)
+		)
+		(property "label" ""
+			(at 91.44 142.24 0)
+			(effects
+				(font
+					(size 1.27 1.27)
+				)
+			)
+		)
+		(property "JLCPCBpn" "C5456188"
+			(at 91.44 142.24 0)
+			(effects
+				(font
+					(size 1.27 1.27)
+				)
+				(hide yes)
+			)
+		)
+		(property "Manufacturer_Name" "STMicro"
+			(at 91.44 142.24 0)
+			(effects
+				(font
+					(size 1.27 1.27)
+				)
+				(hide yes)
+			)
+		)
+		(property "Manufacturer_Part_Number" "ST STM32C011F4U6TR"
 			(at 91.44 142.24 0)
 			(effects
@@
 			)
 		)
-		(property "Value" "STM32C011F_4-6_Ux"
+		(property "Value" "STM32C011F4U6TR"
 			(at 157.0833 41.91 0)
 			(effects
@@
 			(at 154.94 64.77 0)
 			(effects
+				(font
+					(size 1.27 1.27)
+				)
+				(hide yes)
+			)
+		)
+		(property "cap-type" ""
+			(at 154.94 64.77 0)
+			(effects
+				(font
+					(size 1.27 1.27)
+				)
+			)
+		)
+		(property "r-power" ""
+			(at 154.94 64.77 0)
+			(effects
+				(font
+					(size 1.27 1.27)
+				)
+			)
+		)
+		(property "label" ""
+			(at 154.94 64.77 0)
+			(effects
+				(font
+					(size 1.27 1.27)
+				)
+			)
+		)
+		(property "JLCPCBpn" "C5456188"
+			(at 154.94 64.77 0)
+			(effects
+				(font
+					(size 1.27 1.27)
+				)
+				(hide yes)
+			)
+		)
+		(property "Manufacturer_Name" "STMicro"
+			(at 154.94 64.77 0)
+			(effects
+				(font
+					(size 1.27 1.27)
+				)
+				(hide yes)
+			)
+		)
+		(property "Manufacturer_Part_Number" "ST STM32C011F4U6TR"
+			(at 154.94 64.77 0)
+			(effects

Commit message: Added support for four audio serial links from AK5578 codec to STM32H753, each with 22 ohm series R and I put series R in the clock outputs from STM32 toward AK5578 as well. Reannotated.
Parts:
- renumbered C2033 to C2001, C2034 to C2002, C2036 to C2003, C2035 to C2004, U2004 to U2003, U2003 to U2004
Changed lines of the file:
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@@
 		(dnp no)
 		(fields_autoplaced yes)
-		(property "Reference" "#PWR02042"
+		(property "Reference" "#PWR02003"
 			(at 80.01 45.72 0)
 			(effects
@@
 			(project "NexRx"
 				(path "/8ae46c04-d01a-4756-8774-512b694bfaff/0ee31834-a2c3-474b-9f7c-c9b4f3cadb3f/f2486bc2-eba8-4fb8-890d-ac8b4843b7f5"
-					(reference "#PWR02042")
+					(reference "#PWR02003")
 					(unit 1)
 				)
@@
 		(dnp no)
 		(fields_autoplaced yes)
-		(property "Reference" "#PWR02050"
+		(property "Reference" "#PWR02013"
 			(at 144.78 45.72 0)
 			(effects
@@
 			(project "NexRx"
 				(path "/8ae46c04-d01a-4756-8774-512b694bfaff/0ee31834-a2c3-474b-9f7c-c9b4f3cadb3f/f2486bc2-eba8-4fb8-890d-ac8b4843b7f5"
-					(reference "#PWR02050")
+					(reference "#PWR02013")
 					(unit 1)
 				)
@@
 		(dnp no)
 		(fields_autoplaced yes)
-		(property "Reference" "U2004"
+		(property "Reference" "U2003"
 			(at 155.8133 115.57 0)
 			(effects
@@
 			(project "NexRx"
 				(path "/8ae46c04-d01a-4756-8774-512b694bfaff/0ee31834-a2c3-474b-9f7c-c9b4f3cadb3f/f2486bc2-eba8-4fb8-890d-ac8b4843b7f5"
-					(reference "U2004")
+					(reference "U2003")
 					(unit 1)
 				)
@@
 		(dnp no)
 		(fields_autoplaced yes)
-		(property "Reference" "#PWR02055"
+		(property "Reference" "#PWR02010"
 			(at 133.35 148.59 0)
 			(effects
@@
 			(project "NexRx"
 				(path "/8ae46c04-d01a-4756-8774-512b694bfaff/0ee31834-a2c3-474b-9f7c-c9b4f3cadb3f/f2486bc2-eba8-4fb8-890d-ac8b4843b7f5"
-					(reference "#PWR02055")
+					(reference "#PWR02010")
 					(unit 1)
 				)
@@
 		(dnp no)
 		(fields_autoplaced yes)
-		(property "Reference" "#PWR02053"
+		(property "Reference" "#PWR02009"
 			(at 130.81 63.5 0)
 			(effects
@@
 			(project "NexRx"
 				(path "/8ae46c04-d01a-4756-8774-512b694bfaff/0ee31834-a2c3-474b-9f7c-c9b4f3cadb3f/f2486bc2-eba8-4fb8-890d-ac8b4843b7f5"
-					(reference "#PWR02053")
+					(reference "#PWR02009")
 					(unit 1)
 				)
@@
 		(dnp no)
 		(fields_autoplaced yes)
-		(property "Reference" "U2003"
+		(property "Reference" "U2004"
 			(at 157.0833 39.37 0)
 			(effects
@@
 			(project "NexRx"
 				(path "/8ae46c04-d01a-4756-8774-512b694bfaff/0ee31834-a2c3-474b-9f7c-c9b4f3cadb3f/f2486bc2-eba8-4fb8-890d-ac8b4843b7f5"
-					(reference "U2003")
+					(reference "U2004")
 					(unit 1)
 				)
@@
 		(dnp no)
 		(fields_autoplaced yes)
-		(property "Reference" "#PWR02049"
+		(property "Reference" "#PWR02011"
 			(at 134.62 72.39 0)
 			(effects
@@
 			(project "NexRx"
 				(path "/8ae46c04-d01a-4756-8774-512b694bfaff/0ee31834-a2c3-474b-9f7c-c9b4f3cadb3f/f2486bc2-eba8-4fb8-890d-ac8b4843b7f5"
-					(reference "#PWR02049")
+					(reference "#PWR02011")
 					(unit 1)
 				)
@@
 		(dnp no)
 		(fields_autoplaced yes)
-		(property "Reference" "C2033"
+		(property "Reference" "C2001"
 			(at 82.6769 35.56 0)
 			(effects
@@
 			(project "NexRx"
 				(path "/8ae46c04-d01a-4756-8774-512b694bfaff/0ee31834-a2c3-474b-9f7c-c9b4f3cadb3f/f2486bc2-eba8-4fb8-890d-ac8b4843b7f5"
-					(reference "C2033")
+					(reference "C2001")
 					(unit 1)
 				)
@@
 		(dnp no)
 		(fields_autoplaced yes)
-		(property "Reference" "#PWR02047"
+		(property "Reference" "#PWR02007"
 			(at 91.44 118.11 0)
 			(effects
@@
 			(project "NexRx"
 				(path "/8ae46c04-d01a-4756-8774-512b694bfaff/0ee31834-a2c3-474b-9f7c-c9b4f3cadb3f/f2486bc2-eba8-4fb8-890d-ac8b4843b7f5"
-					(reference "#PWR02047")
+					(reference "#PWR02007")
 					(unit 1)
 				)
@@
 		(dnp no)
 		(fields_autoplaced yes)
-		(property "Reference" "#PWR02048"
+		(property "Reference" "#PWR02008"
 			(at 91.44 172.72 0)
 			(effects
@@
 			(project "NexRx"
 				(path "/8ae46c04-d01a-4756-8774-512b694bfaff/0ee31834-a2c3-474b-9f7c-c9b4f3cadb3f/f2486bc2-eba8-4fb8-890d-ac8b4843b7f5"
-					(reference "#PWR02048")
+					(reference "#PWR02008")
 					(unit 1)
 				)
@@
 		(dnp no)
 		(fields_autoplaced yes)
-		(property "Reference" "C2036"
+		(property "Reference" "C2003"
 			(at 146.1769 111.76 0)
 			(effects
@@
 			(project "NexRx"
 				(path "/8ae46c04-d01a-4756-8774-512b694bfaff/0ee31834-a2c3-474b-9f7c-c9b4f3cadb3f/f2486bc2-eba8-4fb8-890d-ac8b4843b7f5"
-					(reference "C2036")
+					(reference "C2003")
 					(unit 1)
 				)
@@
 		(dnp no)
 		(fields_autoplaced yes)
-		(property "Reference" "C2035"
+		(property "Reference" "C2004"
 			(at 147.4469 35.56 0)
 			(effects
@@
 			(project "NexRx"
 				(path "/8ae46c04-d01a-4756-8774-512b694bfaff/0ee31834-a2c3-474b-9f7c-c9b4f3cadb3f/f2486bc2-eba8-4fb8-890d-ac8b4843b7f5"
-					(reference "C2035")
+					(reference "C2004")
 					(unit 1)
 				)
@@
 		(dnp no)
 		(fields_autoplaced yes)
-		(property "Reference" "#PWR02056"
+		(property "Reference" "#PWR02012"
 			(at 143.51 121.92 0)
 			(effects
@@
 			(project "NexRx"
 				(path "/8ae46c04-d01a-4756-8774-512b694bfaff/0ee31834-a2c3-474b-9f7c-c9b4f3cadb3f/f2486bc2-eba8-4fb8-890d-ac8b4843b7f5"
-					(reference "#PWR02056")
+					(reference "#PWR02012")
 					(unit 1)
 				)
@@
 		(dnp no)
 		(fields_autoplaced yes)
-		(property "Reference" "#PWR02051"
+		(property "Reference" "#PWR02016"
 			(at 154.94 40.64 0)
 			(effects
@@
 			(project "NexRx"
 				(path "/8ae46c04-d01a-4756-8774-512b694bfaff/0ee31834-a2c3-474b-9f7c-c9b4f3cadb3f/f2486bc2-eba8-4fb8-890d-ac8b4843b7f5"
-					(reference "#PWR02051")
+					(reference "#PWR02016")
 					(unit 1)
 				)
@@
 		(dnp no)
 		(fields_autoplaced yes)
-		(property "Reference" "#PWR02043"
+		(property "Reference" "#PWR02005"
 			(at 90.17 40.64 0)
 			(effects
@@
 			(project "NexRx"
 				(path "/8ae46c04-d01a-4756-8774-512b694bfaff/0ee31834-a2c3-474b-9f7c-c9b4f3cadb3f/f2486bc2-eba8-4fb8-890d-ac8b4843b7f5"
-					(reference "#PWR02043")
+					(reference "#PWR02005")
 					(unit 1)
 				)
@@
 		(dnp no)
 		(fields_autoplaced yes)
-		(property "Reference" "#PWR02058"
+		(property "Reference" "#PWR02015"
 			(at 153.67 171.45 0)
 			(effects
@@
 			(project "NexRx"
 				(path "/8ae46c04-d01a-4756-8774-512b694bfaff/0ee31834-a2c3-474b-9f7c-c9b4f3cadb3f/f2486bc2-eba8-4fb8-890d-ac8b4843b7f5"
-					(reference "#PWR02058")
+					(reference "#PWR02015")
 					(unit 1)
 				)
@@
 		(dnp no)
 		(fields_autoplaced yes)
-		(property "Reference" "C2034"
+		(property "Reference" "C2002"
 			(at 83.9469 113.03 0)
 			(effects
@@
 			(project "NexRx"
 				(path "/8ae46c04-d01a-4756-8774-512b694bfaff/0ee31834-a2c3-474b-9f7c-c9b4f3cadb3f/f2486bc2-eba8-4fb8-890d-ac8b4843b7f5"
-					(reference "C2034")
+					(reference "C2002")
 					(unit 1)
 				)
@@
 		(dnp no)
 		(fields_autoplaced yes)
-		(property "Reference" "#PWR02046"
+		(property "Reference" "#PWR02004"
 			(at 81.28 123.19 0)
 			(effects
@@
 			(project "NexRx"
 				(path "/8ae46c04-d01a-4756-8774-512b694bfaff/0ee31834-a2c3-474b-9f7c-c9b4f3cadb3f/f2486bc2-eba8-4fb8-890d-ac8b4843b7f5"
-					(reference "#PWR02046")
+					(reference "#PWR02004")
 					(unit 1)
 				)
@@
 		(dnp no)
 		(fields_autoplaced yes)
-		(property "Reference" "#PWR02052"
+		(property "Reference" "#PWR02017"
 			(at 154.94 95.25 0)
 			(effects
@@
 			(project "NexRx"
 				(path "/8ae46c04-d01a-4756-8774-512b694bfaff/0ee31834-a2c3-474b-9f7c-c9b4f3cadb3f/f2486bc2-eba8-4fb8-890d-ac8b4843b7f5"
-					(reference "#PWR02052")
+					(reference "#PWR02017")
 					(unit 1)
 				)
@@
 		(dnp no)
 		(fields_autoplaced yes)
-		(property "Reference" "#PWR02057"
+		(property "Reference" "#PWR02014"
 			(at 153.67 116.84 0)
 			(effects
@@
 			(project "NexRx"
 				(path "/8ae46c04-d01a-4756-8774-512b694bfaff/0ee31834-a2c3-474b-9f7c-c9b4f3cadb3f/f2486bc2-eba8-4fb8-890d-ac8b4843b7f5"
-					(reference "#PWR02057")
+					(reference "#PWR02014")
 					(unit 1)
 				)
@@
 		(dnp no)
 		(fields_autoplaced yes)
-		(property "Reference" "#PWR02044"
+		(property "Reference" "#PWR02006"
 			(at 90.17 95.25 0)
 			(effects
@@
 			(project "NexRx"
 				(path "/8ae46c04-d01a-4756-8774-512b694bfaff/0ee31834-a2c3-474b-9f7c-c9b4f3cadb3f/f2486bc2-eba8-4fb8-890d-ac8b4843b7f5"
-					(reference "#PWR02044")
+					(reference "#PWR02006")
 					(unit 1)
 				)
@@
 		(dnp no)
 		(fields_autoplaced yes)
-		(property "Reference" "#PWR02041"
+		(property "Reference" "#PWR02001"
 			(at 69.85 72.39 0)
 			(effects
@@
 			(project "NexRx"
 				(path "/8ae46c04-d01a-4756-8774-512b694bfaff/0ee31834-a2c3-474b-9f7c-c9b4f3cadb3f/f2486bc2-eba8-4fb8-890d-ac8b4843b7f5"
-					(reference "#PWR02041")
+					(reference "#PWR02001")
 					(unit 1)
 				)
@@
 		(dnp no)
 		(fields_autoplaced yes)
-		(property "Reference" "#PWR02045"
+		(property "Reference" "#PWR02002"
 			(at 71.12 149.86 0)
 			(effects
@@
 			(project "NexRx"
 				(path "/8ae46c04-d01a-4756-8774-512b694bfaff/0ee31834-a2c3-474b-9f7c-c9b4f3cadb3f/f2486bc2-eba8-4fb8-890d-ac8b4843b7f5"
-					(reference "#PWR02045")
-					(unit 1)
-				)
+					(reference "#PWR02002")
+					(unit 1)
+				)
