File: hw/cpld.kicad_sch (KiCad schematic)
At the start: 13 parts, among them U1001 ICE40LP384-SG32

Commit message: Updates for actual DVT2 BOM order part numbers and fixes
Parts:
- R1001: MFG (none) -> YAGEO; MPN (none) -> RT0402BRD0722K1L; Mouser Part Number (none) -> 603-RT0402BRD0722K1L
- R1002: MFG (none) -> YAGEO; MPN (none) -> RT0402BRD0710KL; Mouser Part Number (none) -> 603-RT0402BRD0710KL
- R1003: MFG (none) -> Wurth Electronik; MPN (none) -> 560112110216; Mouser Part Number (none) -> 710-560112110216
- U1001: MFG (none) -> Lattice Semi; MPN (none) -> ICE40LP384-SG32; Mouser Part Number (none) -> 842-ICE40LP384SG32
Changed lines of the file:
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@@
 			)
 		)
-		(property "Description" "Resistor, Thin Film, 0.1%, 22.1k, 0402"
+		(property "Description" "Resistor, Thin Film, 1%, 22.1k, 0402"
 			(at 26.67 45.72 0)
 			(effects
@@
 			)
 		)
-		(property "MPN" ""
+		(property "MPN" "RT0402BRD0722K1L"
 			(at -111.76 -59.69 0)
 			(effects
@@
 			)
 		)
+		(property "MFG" "YAGEO"
+			(at 26.67 45.72 0)
+			(effects
+				(font
+					(size 1.27 1.27)
+				)
+				(hide yes)
+			)
+		)
+		(property "Mouser Part Number" "603-RT0402BRD0722K1L "
+			(at 26.67 45.72 0)
+			(effects
+				(font
+					(size 1.27 1.27)
+				)
+				(hide yes)
+			)
+		)
 		(pin "1"
 		)
@@
 			)
 		)
-		(property "Description" ""
+		(property "Description" "FPGA - Field Programmable Gate Array iCE40LP Ultra LowPwr 384 LUTs 1.2V"
 			(at 54.61 134.62 0)
 			(effects
@@
 			)
 		)
+		(property "MPN" "ICE40LP384-SG32 "
+			(at 107.95 147.32 0)
+			(effects
+				(font
+					(size 1.27 1.27)
+				)
+				(hide yes)
+			)
+		)
+		(property "Mouser Part Number" "842-ICE40LP384SG32 "
+			(at 107.95 147.32 0)
+			(effects
+				(font
+					(size 1.27 1.27)
+				)
+				(hide yes)
+			)
+		)
+		(property "MFG" "Lattice Semi"
+			(at 107.95 147.32 0)
+			(effects
+				(font
+					(size 1.27 1.27)
+				)
+				(hide yes)
+			)
+		)
 		(pin "33"
 		)
@@
 			)
 		)
-		(property "Description" "Capacitor, MLCC, X7R, 50V, 5%, 100nF, 0603"
+		(property "Description" "Capacitor, MLCC, X7R, 50V, 5%, 100nF, 0402"
 			(at 92.71 99.06 0)
 			(effects
@@
 			)
 		)
-		(property "Description" "Capacitor, MLCC, X7R, 50V, 5%, 100nF, 0603"
+		(property "Description" "Capacitor, MLCC, X7R, 50V, 5%, 100nF, 0402"
 			(at 64.77 104.14 0)
 			(effects
@@
 			)
 		)
-		(property "Description" "Capacitor, MLCC, X7R, 50V, 5%, 100nF, 0603"
+		(property "Description" "Capacitor, MLCC, X7R, 50V, 5%, 100nF, 0402"
 			(at 26.67 76.2 0)
 			(effects
@@
 			)
 		)
-		(property "Description" "Resistor, US symbol"
+		(property "Description" "Resistor, Thin Film, 0.1%, 10k, 0402"
 			(at 20.32 53.34 0)
 			(effects
@@
 			)
 		)
+		(property "MFG" "YAGEO"
+			(at 20.32 53.34 90)
+			(effects
+				(font
+					(size 1.27 1.27)
+				)
+				(hide yes)
+			)
+		)
+		(property "MPN" "RT0402BRD0710KL"
+			(at 20.32 53.34 90)
+			(effects
+				(font
+					(size 1.27 1.27)
+				)
+				(hide yes)
+			)
+		)
+		(property "Mouser Part Number" "603-RT0402BRD0710KL"
+			(at 20.32 53.34 90)
+			(effects
+				(font
+					(size 1.27 1.27)
+				)
+				(hide yes)
+			)
+		)
 		(pin "2"
 		)
@@
 			)
 		)
-		(property "Description" "Capacitor, MLCC, X7R, 50V, 5%, 100nF, 0603"
+		(property "Description" "Capacitor, MLCC, X7R, 50V, 5%, 100nF, 0402"
 			(at 64.77 83.82 0)
 			(effects
@@
 			)
 		)
-		(property "Description" "Resistor, small US symbol"
+		(property "Description" "Resistor, Thick Film, 1%, 22, 0402"
 			(at 101.6 175.26 0)
 			(effects
@@
 			)
 		)
+		(property "MFG" "Wurth Electronik"
+			(at 101.6 175.26 90)
+			(effects
+				(font
+					(size 1.27 1.27)
+				)
+				(hide yes)
+			)
+		)
+		(property "MPN" "560112110216"
+			(at 101.6 175.26 90)
+			(effects
+				(font
+					(size 1.27 1.27)
+				)
+				(hide yes)
+			)
+		)
+		(property "Mouser Part Number" "710-560112110216"
+			(at 101.6 175.26 90)
+			(effects
+				(font
+					(size 1.27 1.27)
+				)
+				(hide yes)
+			)
+		)
 		(pin "1"
 		)
@@
 			)
 		)
-		(property "Description" "Capacitor, Tantalum, 10V, 10%, 4.7uF, 0805"
+		(property "Description" "Capacitor, MLCC, X5R, 10V, 20%, 2.7uF, 0402"
 			(at 46.99 50.8 0)
 			(effects
@@
 			)
 		)
-		(property "Description" "Capacitor, MLCC, X7R, 50V, 5%, 100nF, 0603"
+		(property "Description" "Capacitor, MLCC, X7R, 50V, 5%, 100nF, 0402"
 			(at 113.03 99.06 0)
 			(effects
@@
 			)
 		)
-		(property "Description" "Capacitor, MLCC, X7R, 50V, 5%, 100nF, 0603"
+		(property "Description" "Capacitor, MLCC, X7R, 50V, 5%, 100nF, 0402"
 			(at 92.71 78.74 0)
 			(effects
@@
 			)
 		)
-		(property "Description" "Capacitor, Tantalum, 10V, 10%, 4.7uF, 0805"
+		(property "Description" "Capacitor, MLCC, X5R, 10V, 20%, 2.7uF, 0402"
 			(at 60.96 50.8 0)
 			(effects
@@
 			)
 		)
-		(property "Description" "Capacitor, MLCC, X7R, 50V, 5%, 100nF, 0603"
+		(property "Description" "Capacitor, MLCC, X7R, 50V, 5%, 100nF, 0402"
 			(at 113.03 78.74 0)
 			(effects
