File: hw/filters.kicad_sch (KiCad schematic)
At the start: 37 parts, among them U301 AS183-92LF, U302 AS183-92LF, U303 AS183-92LF, U304 AS183-92LF, U305 AS183-92LF, U306 AS183-92LF, U307 AS183-92LF, U308 AS183-92LF, U309 SN74LVC2G14DCK3

Commit message: Updates for actual DVT2 BOM order part numbers and fixes
Parts:
- C311, C313: MFG Kyocera -> KEMET; MPN 04023A151JAT2A -> C0402C151J3GACTU; Mouser Part Number 581-04023A151J -> C0402C151J3GACTU
- C315: Mouser Part Number 80-C0402C151J3G -> C0402C151J3GACTU
- L301, L302, L303, L304, L305, L306, L307, L308, L309, L310, L311: now left out of the parts list
- U301, U302, U303, U304, U305, U306, U307, U308: MFG (none) -> SKYWORKS; Mouser Part Number (none) -> 873-AS183-92LF
- U309: value SN74LVC2G14DCK3 -> SN74LVC2G14DCKRE4; MFG (none) -> TI; MPN (none) -> SN74LVC2G14DCKRE4; Mouser Part Number (none) -> 595-SN74LVC2G14DCKRE4
Changed lines of the file:
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@@
 			)
 		)
-		(property "Mouser Part Number" ""
+		(property "Mouser Part Number" "873-AS183-92LF"
+			(at 157.48 120.65 0)
+			(effects
+				(font
+					(size 1.27 1.27)
+				)
+				(hide yes)
+			)
+		)
+		(property "MFG" "SKYWORKS"
 			(at 157.48 120.65 0)
 			(effects
@@
 			)
 		)
-		(property "Mouser Part Number" ""
+		(property "Mouser Part Number" "873-AS183-92LF"
+			(at 240.03 96.52 0)
+			(effects
+				(font
+					(size 1.27 1.27)
+				)
+				(hide yes)
+			)
+		)
+		(property "MFG" "SKYWORKS"
 			(at 240.03 96.52 0)
 			(effects
@@
 		(unit 1)
 		(exclude_from_sim no)
-		(in_bom yes)
+		(in_bom no)
 		(on_board yes)
 		(dnp yes)
@@
 			)
 		)
-		(property "Description" "capacitor, US symbol"
+		(property "Description" "Capacitor, MLCC, NP0, 25V, 5%, 1uF, 0402"
 			(at 64.77 97.79 0)
 			(effects
@@
 			)
 		)
-		(property "Description" "capacitor, US symbol"
+		(property "Description" "Capacitor, MLCC, NP0, 25V, 5%, 150pF, 0402"
 			(at 189.23 142.24 0)
 			(effects
@@
 			)
 		)
-		(property "Mouser Part Number" "80-C0402C151J3G"
+		(property "Mouser Part Number" "C0402C151J3GACTU"
 			(at 189.23 142.24 0)
 			(effects
@@
 			)
 		)
-		(property "Mouser Part Number" ""
+		(property "Mouser Part Number" "873-AS183-92LF"
+			(at 34.29 95.25 0)
+			(effects
+				(font
+					(size 1.27 1.27)
+				)
+				(hide yes)
+			)
+		)
+		(property "MFG" "SKYWORKS"
 			(at 34.29 95.25 0)
 			(effects
@@
 			)
 		)
-		(property "Description" "capacitor, US symbol"
+		(property "Description" "Capacitor, MLCC, NP0, 25V, 5%, 300pF, 0402"
 			(at 176.53 85.09 0)
 			(effects
@@
 			)
 		)
-		(property "Description" "capacitor, US symbol"
+		(property "Description" "Capacitor, MLCC, NP0, 25V, 5%, 680pF, 0402"
 			(at 189.23 85.09 0)
 			(effects
@@
 			)
 		)
-		(property "Mouser Part Number" ""
+		(property "Mouser Part Number" "873-AS183-92LF"
+			(at 142.24 95.25 0)
+			(effects
+				(font
+					(size 1.27 1.27)
+				)
+				(hide yes)
+			)
+		)
+		(property "MFG" "SKYWORKS"
 			(at 142.24 95.25 0)
 			(effects
@@
 		(unit 1)
 		(exclude_from_sim no)
-		(in_bom yes)
+		(in_bom no)
 		(on_board yes)
 		(dnp yes)
@@
 			)
 		)
-		(property "Description" "Capacitor, MLCC, X7R, 50V, 5%, 100nF, 0603"
+		(property "Description" "Capacitor, MLCC, X7R, 50V, 5%, 100nF, 0402"
 			(at 80.01 166.37 0)
 			(effects
@@
 		(unit 1)
 		(exclude_from_sim no)
-		(in_bom yes)
+		(in_bom no)
 		(on_board yes)
 		(dnp yes)
@@
 			)
 		)
-		(property "Mouser Part Number" ""
+		(property "Mouser Part Number" "873-AS183-92LF"
+			(at 224.79 72.39 0)
+			(effects
+				(font
+					(size 1.27 1.27)
+				)
+				(hide yes)
+			)
+		)
+		(property "MFG" "SKYWORKS"
 			(at 224.79 72.39 0)
 			(effects
@@
 		(unit 1)
 		(exclude_from_sim no)
-		(in_bom yes)
+		(in_bom no)
 		(on_board yes)
 		(dnp yes)
@@
 		(unit 1)
 		(exclude_from_sim no)
-		(in_bom yes)
+		(in_bom no)
 		(on_board yes)
 		(dnp yes)
@@
 			)
 		)
-		(property "Description" "capacitor, US symbol"
+		(property "Description" "Capacitor, MLCC, NP0, 25V, 5%, 150pF, 0402"
 			(at 201.93 115.57 0)
 			(effects
@@
 			)
 		)
-		(property "Mouser Part Number" "581-04023A151J"
+		(property "Mouser Part Number" "C0402C151J3GACTU"
 			(at 201.93 115.57 90)
 			(effects
@@
 			)
 		)
-		(property "MPN" "04023A151JAT2A"
+		(property "MPN" "C0402C151J3GACTU"
 			(at 201.93 115.57 90)
 			(effects
@@
 			)
 		)
-		(property "MFG" "Kyocera"
+		(property "MFG" "KEMET"
 			(at 201.93 115.57 0)
 			(effects
@@
 			)
 		)
-		(property "Description" "capacitor, US symbol"
+		(property "Description" "Capacitor, MLCC, NP0, 25V, 5%, 1uF, 0402"
 			(at 78.74 97.79 0)
 			(effects
@@
 			)
 		)
-		(property "Description" "capacitor, US symbol"
+		(property "Description" "Capacitor, MLCC, NP0, 25V, 5%, 910pF, 0603"
 			(at 176.53 58.42 0)
 			(effects
@@
 			)
 		)
-		(property "Description" "capacitor, US symbol"
+		(property "Description" "Capacitor, MLCC, NP0, 25V, 5%, 910pF, 0603"
 			(at 201.93 58.42 0)
 			(effects
@@
 			)
 		)
-		(property "Description" "capacitor, US symbol"
+		(property "Description" "Capacitor, MLCC, NP0, 25V, 5%, 300pF, 0402"
 			(at 189.23 115.57 0)
 			(effects
@@
 			)
 		)
-		(property "Description" "capacitor, US symbol"
+		(property "Description" "Capacitor, MLCC, NP0, 25V, 5%, 300pF, 0402"
 			(at 201.93 85.09 0)
 			(effects
@@
 			)
 		)
-		(property "Mouser Part Number" ""
+		(property "Mouser Part Number" "873-AS183-92LF"
+			(at 107.95 95.25 0)
+			(effects
+				(font
+					(size 1.27 1.27)
+				)
+				(hide yes)
+			)
+		)
+		(property "MFG" "SKYWORKS"
 			(at 107.95 95.25 0)
 			(effects
@@
 		(unit 1)
 		(exclude_from_sim no)
-		(in_bom yes)
+		(in_bom no)
 		(on_board yes)
 		(dnp no)
@@
 			)
 		)
-		(property "Description" "capacitor, US symbol"
+		(property "Description" "Capacitor, MLCC, NP0, 25V, 5%, 150pF, 0402"
 			(at 189.23 58.42 0)
 			(effects
@@
 			)
 		)
-		(property "Mouser Part Number" ""
+		(property "Mouser Part Number" "873-AS183-92LF"
+			(at 224.79 124.46 0)
+			(effects
+				(font
+					(size 1.27 1.27)
+				)
+				(hide yes)
+			)
+		)
+		(property "MFG" "SKYWORKS"
 			(at 224.79 124.46 0)
 			(effects
@@
 			)
 		)
-		(property "Description" "capacitor, US symbol"
+		(property "Description" "Capacitor, MLCC, NP0, 25V, 5%, 75pF, 0402"
 			(at 176.53 142.24 0)
 			(effects
@@
 		(unit 1)
 		(exclude_from_sim no)
-		(in_bom yes)
+		(in_bom no)
 		(on_board yes)
 		(dnp no)
@@
 		(unit 1)
 		(exclude_from_sim no)
-		(in_bom yes)
+		(in_bom no)
 		(on_board yes)
 		(dnp yes)
@@
 			)
 		)
-		(property "Value" "SN74LVC2G14DCK3"
+		(property "Value" "SN74LVC2G14DCKRE4"
 			(at 53.34 154.94 0)
 			(effects
@@
 			)
 		)
-		(property "Description" ""
+		(property "Description" "Inverters Dual Schmitt-Trigger"
+			(at 53.34 161.29 0)
+			(effects
+				(font
+					(size 1.27 1.27)
+				)
+				(hide yes)
+			)
+		)
+		(property "MFG" "TI"
+			(at 53.34 161.29 0)
+			(effects
+				(font
+					(size 1.27 1.27)
+				)
+				(hide yes)
+			)
+		)
+		(property "MPN" "SN74LVC2G14DCKRE4"
+			(at 53.34 161.29 0)
+			(effects
+				(font
+					(size 1.27 1.27)
+				)
+				(hide yes)
+			)
+		)
+		(property "Mouser Part Number" "595-SN74LVC2G14DCKRE4"
 			(at 53.34 161.29 0)
 			(effects
@@
 			)
 		)
-		(property "Description" "capacitor, US symbol"
+		(property "Description" "Capacitor, MLCC, NP0, 25V, 5%, 2.2uF, 0402"
 			(at 92.71 97.79 0)
 			(effects
@@
 			)
 		)
-		(property "Description" "capacitor, US symbol"
+		(property "Description" "Capacitor, MLCC, NP0, 25V, 5%, 150pF, 0402"
 			(at 176.53 115.57 0)
 			(effects
@@
 			)
 		)
-		(property "Mouser Part Number" "581-04023A151J"
+		(property "Mouser Part Number" "C0402C151J3GACTU"
 			(at 176.53 115.57 90)
 			(effects
@@
 			)
 		)
-		(property "MPN" "04023A151JAT2A"
+		(property "MPN" "C0402C151J3GACTU"
 			(at 176.53 115.57 90)
 			(effects
@@
 			)
 		)
-		(property "MFG" "Kyocera"
+		(property "MFG" "KEMET"
 			(at 176.53 115.57 0)
 			(effects
@@
 		(unit 1)
 		(exclude_from_sim no)
-		(in_bom yes)
+		(in_bom no)
 		(on_board yes)
 		(dnp yes)
@@
 		(unit 1)
 		(exclude_from_sim no)
-		(in_bom yes)
+		(in_bom no)
 		(on_board yes)
 		(dnp yes)
@@
 		(unit 1)
 		(exclude_from_sim no)
-		(in_bom yes)
+		(in_bom no)
 		(on_board yes)
 		(dnp no)
@@
 			)
 		)
-		(property "Description" "capacitor, US symbol"
+		(property "Description" "Capacitor, MLCC, NP0, 25V, 5%, 75pF, 0402"
 			(at 201.93 142.24 0)
 			(effects
@@
 			)
 		)
-		(property "Mouser Part Number" ""
+		(property "Mouser Part Number" "873-AS183-92LF"
+			(at 158.75 71.12 0)
+			(effects
+				(font
+					(size 1.27 1.27)
+				)
+				(hide yes)
+			)
+		)
+		(property "MFG" "SKYWORKS"
 			(at 158.75 71.12 0)
 			(effects
@@
 			)
 		)
-		(property "Description" "capacitor, US symbol"
+		(property "Description" "Capacitor, MLCC, NP0, 25V, 5%, 2.2uF, 0402"
 			(at 49.53 97.79 0)
 			(effects

Commit message: Fix inductors so they show up in BOM even though I have stock in hand
Parts:
- L301, L302: MFG (none) -> Coilcraft; MPN 1812CS-332XJR -> 1812CS-272XJR; Mouser Part Number (none) -> 994-1812CS-272XJRC; now fitted; now in the parts list
- L303, L304: MFG (none) -> Coilcraft; Mouser Part Number (none) -> 994-1812CS-122XJRC; now fitted; now in the parts list
- L305, L307: MFG (none) -> Coilcraft; Mouser Part Number (none) -> 994-1812CS-332XJRC; now in the parts list
- L306: MFG (none) -> Coilcraft; Mouser Part Number (none) -> 994-1812CS-272XJRC; now in the parts list
- L308, L309: MFG (none) -> Coilcraft; Mouser Part Number (none) -> 994-1008CS-561XJRC; now fitted; now in the parts list
- L310, L311: MFG (none) -> Coilcraft; Mouser Part Number (none) -> 994-1008CS-331XJRC; now fitted; now in the parts list
Changed lines of the file:
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@@
 		(unit 1)
 		(exclude_from_sim no)
-		(in_bom no)
+		(in_bom yes)
 		(on_board yes)
-		(dnp yes)
+		(dnp no)
 		(property "Reference" "L301"
 			(at 181.61 51.054 90)
@@
 			)
 		)
-		(property "Description" "Inductor with ferrite core, small symbol"
+		(property "Description" "SMD RF chip inductor, 2.7uH, 1812"
 			(at 181.61 53.34 0)
 			(effects
@@
 			)
 		)
-		(property "Mouser Part Number" ""
+		(property "Mouser Part Number" "994-1812CS-272XJRC"
 			(at 181.61 53.34 90)
 			(effects
@@
 			)
 		)
-		(property "MPN" "1812CS-332XJR"
+		(property "MPN" "1812CS-272XJR"
 			(at 181.61 53.34 90)
 			(effects
@@
 			)
 		)
+		(property "MFG" "Coilcraft"
+			(at 181.61 53.34 90)
+			(effects
+				(font
+					(size 1.27 1.27)
+				)
+				(hide yes)
+			)
+		)
 		(pin "2"
 		)
@@
 		(unit 1)
 		(exclude_from_sim no)
-		(in_bom no)
+		(in_bom yes)
 		(on_board yes)
-		(dnp yes)
+		(dnp no)
 		(property "Reference" "L303"
 			(at 181.61 77.724 90)
@@
 			)
 		)
-		(property "Description" "Inductor with ferrite core, small symbol"
+		(property "Description" "SMD RF chip inductor, 1.2uH, 1812"
 			(at 181.61 80.01 0)
 			(effects
@@
 			)
 		)
-		(property "Mouser Part Number" ""
+		(property "Mouser Part Number" "994-1812CS-122XJRC"
 			(at 181.61 80.01 90)
 			(effects
@@
 			)
 		)
+		(property "MFG" "Coilcraft"
+			(at 181.61 80.01 90)
+			(effects
+				(font
+					(size 1.27 1.27)
+				)
+				(hide yes)
+			)
+		)
 		(pin "2"
 		)
@@
 		(unit 1)
 		(exclude_from_sim no)
-		(in_bom no)
+		(in_bom yes)
 		(on_board yes)
-		(dnp yes)
+		(dnp no)
 		(property "Reference" "L302"
 			(at 195.58 51.054 90)
@@
 			)
 		)
-		(property "Description" "Inductor with ferrite core, small symbol"
+		(property "Description" "SMD RF chip inductor, 2.7uH, 1812"
 			(at 195.58 53.34 0)
 			(effects
@@
 			)
 		)
-		(property "Mouser Part Number" ""
+		(property "Mouser Part Number" "994-1812CS-272XJRC"
 			(at 195.58 53.34 90)
 			(effects
@@
 			)
 		)
-		(property "MPN" "1812CS-332XJR"
+		(property "MPN" "1812CS-272XJR"
 			(at 195.58 53.34 90)
 			(effects
@@
 			)
 		)
+		(property "MFG" "Coilcraft"
+			(at 195.58 53.34 90)
+			(effects
+				(font
+					(size 1.27 1.27)
+				)
+				(hide yes)
+			)
+		)
 		(pin "2"
 		)
@@
 		(unit 1)
 		(exclude_from_sim no)
-		(in_bom no)
+		(in_bom yes)
 		(on_board yes)
-		(dnp yes)
+		(dnp no)
 		(property "Reference" "L308"
 			(at 181.61 108.204 90)
@@
 			)
 		)
-		(property "Description" "Inductor with ferrite core, small symbol"
+		(property "Description" "SMD RF chip inductor, 560nH, 1008"
 			(at 181.61 110.49 0)
 			(effects
@@
 			)
 		)
-		(property "Mouser Part Number" ""
+		(property "Mouser Part Number" "994-1008CS-561XJRC"
 			(at 181.61 110.49 90)
 			(effects
@@
 			)
 		)
+		(property "MFG" "Coilcraft"
+			(at 181.61 110.49 90)
+			(effects
+				(font
+					(size 1.27 1.27)
+				)
+				(hide yes)
+			)
+		)
 		(pin "2"
 		)
@@
 		(unit 1)
 		(exclude_from_sim no)
-		(in_bom no)
+		(in_bom yes)
 		(on_board yes)
-		(dnp yes)
+		(dnp no)
 		(property "Reference" "L309"
 			(at 195.58 108.204 90)
@@
 			)
 		)
-		(property "Description" "Inductor with ferrite core, small symbol"
+		(property "Description" "SMD RF chip inductor, 560nH, 1008"
 			(at 195.58 110.49 0)
 			(effects
@@
 			)
 		)
-		(property "Mouser Part Number" ""
+		(property "Mouser Part Number" "994-1008CS-561XJRC"
 			(at 195.58 110.49 90)
 			(effects
@@
 			)
 		)
+		(property "MFG" "Coilcraft"
+			(at 195.58 110.49 90)
+			(effects
+				(font
+					(size 1.27 1.27)
+				)
+				(hide yes)
+			)
+		)
 		(pin "2"
 		)
@@
 		(unit 1)
 		(exclude_from_sim no)
-		(in_bom no)
+		(in_bom yes)
 		(on_board yes)
 		(dnp no)
@@
 			)
 		)
-		(property "Description" "Inductor with ferrite core, small symbol"
+		(property "Description" "SMD RF chip inductor, 2.7uH, 1812"
 			(at 69.85 104.14 0)
 			(effects
@@
 			)
 		)
-		(property "Mouser Part Number" ""
+		(property "Mouser Part Number" "994-1812CS-272XJRC"
 			(at 69.85 104.14 0)
 			(effects
@@
 			)
 		)
+		(property "MFG" "Coilcraft"
+			(at 69.85 104.14 0)
+			(effects
+				(font
+					(size 1.27 1.27)
+				)
+				(hide yes)
+			)
+		)
 		(pin "2"
 		)
@@
 		(unit 1)
 		(exclude_from_sim no)
-		(in_bom no)
+		(in_bom yes)
 		(on_board yes)
 		(dnp no)
@@
 			)
 		)
-		(property "Description" "Inductor with ferrite core, small symbol"
+		(property "Description" "SMD RF chip inductor, 3.3uH, 1812"
 			(at 83.82 104.14 0)
 			(effects
@@
 			)
 		)
-		(property "Mouser Part Number" ""
+		(property "Mouser Part Number" "994-1812CS-332XJRC"
 			(at 83.82 104.14 0)
 			(effects
@@
 			)
 		)
+		(property "MFG" "Coilcraft"
+			(at 83.82 104.14 0)
+			(effects
+				(font
+					(size 1.27 1.27)
+				)
+				(hide yes)
+			)
+		)
 		(pin "2"
 		)
@@
 		(unit 1)
 		(exclude_from_sim no)
-		(in_bom no)
+		(in_bom yes)
 		(on_board yes)
-		(dnp yes)
+		(dnp no)
 		(property "Reference" "L311"
 			(at 195.58 134.874 90)
@@
 			)
 		)
-		(property "Description" "Inductor with ferrite core, small symbol"
+		(property "Description" "SMD RF chip inductor, 330nH, 1008"
 			(at 195.58 137.16 0)
 			(effects
@@
 			)
 		)
-		(property "Mouser Part Number" ""
+		(property "Mouser Part Number" "994-1008CS-331XJRC"
 			(at 195.58 137.16 90)
 			(effects
@@
 			)
 		)
+		(property "MFG" "Coilcraft"
+			(at 195.58 137.16 90)
+			(effects
+				(font
+					(size 1.27 1.27)
+				)
+				(hide yes)
+			)
+		)
 		(pin "2"
 		)
@@
 		(unit 1)
 		(exclude_from_sim no)
-		(in_bom no)
+		(in_bom yes)
 		(on_board yes)
-		(dnp yes)
+		(dnp no)
 		(property "Reference" "L310"
 			(at 181.61 134.874 90)
@@
 			)
 		)
-		(property "Description" "Inductor with ferrite core, small symbol"
+		(property "Description" "SMD RF chip inductor, 330nH, 1008"
 			(at 181.61 137.16 0)
 			(effects
@@
 			)
 		)
-		(property "Mouser Part Number" ""
+		(property "Mouser Part Number" "994-1008CS-331XJRC"
 			(at 181.61 137.16 90)
 			(effects
@@
 			)
 		)
+		(property "MFG" "Coilcraft"
+			(at 181.61 137.16 90)
+			(effects
+				(font
+					(size 1.27 1.27)
+				)
+				(hide yes)
+			)
+		)
 		(pin "2"
 		)
@@
 		(unit 1)
 		(exclude_from_sim no)
-		(in_bom no)
+		(in_bom yes)
 		(on_board yes)
-		(dnp yes)
+		(dnp no)
 		(property "Reference" "L304"
 			(at 195.58 77.724 90)
@@
 			)
 		)
-		(property "Description" "Inductor with ferrite core, small symbol"
+		(property "Description" "SMD RF chip inductor, 1.2uH, 1812"
 			(at 195.58 80.01 0)
 			(effects
@@
 			)
 		)
-		(property "Mouser Part Number" ""
+		(property "Mouser Part Number" "994-1812CS-122XJRC"
 			(at 195.58 80.01 90)
 			(effects
@@
 			)
 		)
+		(property "MFG" "Coilcraft"
+			(at 195.58 80.01 90)
+			(effects
+				(font
+					(size 1.27 1.27)
+				)
+				(hide yes)
+			)
+		)
 		(pin "2"
 		)
@@
 		(unit 1)
 		(exclude_from_sim no)
-		(in_bom no)
+		(in_bom yes)
 		(on_board yes)
 		(dnp no)
@@
 			)
 		)
-		(property "Description" "Inductor with ferrite core, small symbol"
+		(property "Description" "SMD RF chip inductor, 3.3uH, 1812"
 			(at 54.61 104.14 0)
 			(effects
@@
 			)
 		)
-		(property "Mouser Part Number" ""
+		(property "Mouser Part Number" "994-1812CS-332XJRC"
 			(at 54.61 104.14 0)
 			(effects
@@
 			(at 54.61 104.14 0)
 			(effects
+				(font
+					(size 1.27 1.27)
+				)
+				(hide yes)
+			)
+		)
+		(property "MFG" "Coilcraft"
+			(at 54.61 104.14 0)
+			(effects
