File: hw/filter-tester/filter-tester-filters.kicad_sch (KiCad schematic)
At the start: 59 parts, among them U201 AS183-92LF, U202 AS183-92LF, U203 AS183-92LF, U204 AS183-92LF, U205 AS183-92LF, U206 AS183-92LF, U207 AS183-92LF, U208 AS183-92LF, U209 AS183-92LF, U210 AS183-92LF

Commit message: DVT4 uses higher Q inductors, some layout tweaks, series R on SWDCLK and SWDIO.
Parts:
- L209: value 470nH -> 500nH; footprint Library:L_1206_3216Metric-keepout -> Inductor_SMD:L_Coilcraft_2929SQ-501; symbol Device:L_Ferrite_Small -> Device:L_Small; MPN AISC-1206-R47G-T -> 2929SQ-501JEC; Manufacturer Abracon -> Coilcraft; Mouser_PN 994-1206CS-471XJRC -> 994-2929SQ-501JEC; now in the parts list
- L212: footprint Library:L_1206_3216Metric-keepout -> Inductor_SMD:L_Coilcraft_2222SQ-161; symbol Device:L_Ferrite_Small -> Device:L_Small; MPN AISC-1206-R15G-T -> 2222SQ-161JEC; Manufacturer Abracon -> Coilcraft; Mouser_PN 994-1206CS-151XJRC -> 994-2222SQ-161JEC; now in the parts list
- L215: footprint Library:L_1206_3216Metric-keepout -> Inductor_SMD:L_Coilcraft_1515SQ-82N; symbol Device:L_Ferrite_Small -> Device:L_Small; MPN AISC-1206-82NK-T -> 1515SQ-82NJEC; Manufacturer Abracon -> Coilcraft; Mouser_PN 994-1206CS-820XJRC -> 994-1515SQ-82NJEC; now in the parts list
Other:
- note removed: "needs custom footprint?"
Changed lines of the file:
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@@
 		(company "WB7NAB")
 	)
-	(text "needs custom footprint?"
-		(exclude_from_sim no)
-		(at 158.496 119.888 0)
-		(effects
-			(font
-				(size 1.27 1.27)
-			)
-		)
-	)
 	(text "AM reject HPF 1.75MHz"
 		(exclude_from_sim no)
@@
 		)
 	)
-	(text "needs custom footprint?"
-		(exclude_from_sim no)
-		(at 157.226 150.368 0)
-		(effects
-			(font
-				(size 1.27 1.27)
-			)
-		)
-	)
-	(text "needs custom footprint?"
-		(exclude_from_sim no)
-		(at 154.94 94.742 0)
-		(effects
-			(font
-				(size 1.27 1.27)
-			)
-		)
-	)
 	(junction
 		(at 128.27 143.51)
@@
 	)
 	(symbol
-		(lib_id "Device:L_Ferrite_Small")
+		(lib_id "Device:L_Small")
 		(at 139.7 118.11 180)
 		(unit 1)
 		(exclude_from_sim no)
-		(in_bom no)
+		(in_bom yes)
 		(on_board yes)
 		(dnp no)
@@
 			)
 		)
-		(property "Footprint" "Library:L_1206_3216Metric-keepout"
+		(property "Footprint" "Inductor_SMD:L_Coilcraft_2222SQ-161"
 			(at 139.7 118.11 0)
 			(effects
@@
 			)
 		)
-		(property "Datasheet" "https://abracon.com/Magnetics/new/AISC-1206.pdf"
+		(property "Datasheet" "~"
 			(at 139.7 118.11 0)
 			(effects
@@
 			)
 		)
-		(property "Description" "Inductor with ferrite core, small symbol"
+		(property "Description" "Inductor, small symbol"
 			(at 139.7 118.11 0)
 			(effects
@@
 			)
 		)
-		(property "Manufacturer" "Abracon"
+		(property "Manufacturer" "Coilcraft"
 			(at 139.7 118.11 0)
 			(effects
@@
 			)
 		)
-		(property "MPN" "AISC-1206-R15G-T"
+		(property "MPN" "2222SQ-161JEC"
 			(at 139.7 118.11 0)
 			(effects
@@
 			)
 		)
-		(property "Mouser_PN" "994-1206CS-151XJRC"
+		(property "Mouser_PN" "994-2222SQ-161JEC"
 			(at 139.7 118.11 0)
 			(effects
@@
 	)
 	(symbol
-		(lib_id "Device:L_Ferrite_Small")
+		(lib_id "Device:L_Small")
 		(at 138.43 148.59 180)
 		(unit 1)
 		(exclude_from_sim no)
-		(in_bom no)
+		(in_bom yes)
 		(on_board yes)
 		(dnp no)
@@
 			)
 		)
-		(property "Footprint" "Library:L_1206_3216Metric-keepout"
+		(property "Footprint" "Inductor_SMD:L_Coilcraft_1515SQ-82N"
 			(at 138.43 148.59 0)
 			(effects
@@
 			)
 		)
-		(property "Description" "Inductor with ferrite core, small symbol"
+		(property "Description" "Inductor, small symbol"
 			(at 138.43 148.59 0)
 			(effects
@@
 			)
 		)
-		(property "Manufacturer" "Abracon"
+		(property "Manufacturer" "Coilcraft"
 			(at 138.43 148.59 0)
 			(effects
@@
 			)
 		)
-		(property "MPN" "AISC-1206-82NK-T"
+		(property "MPN" "1515SQ-82NJEC"
 			(at 138.43 148.59 0)
 			(effects
@@
 			)
 		)
-		(property "Mouser_PN" "994-1206CS-820XJRC"
+		(property "Mouser_PN" "994-1515SQ-82NJEC"
 			(at 138.43 148.59 0)
 			(effects
@@
 	)
 	(symbol
-		(lib_id "Device:L_Ferrite_Small")
+		(lib_id "Device:L_Small")
 		(at 139.7 91.44 180)
 		(unit 1)
 		(exclude_from_sim no)
-		(in_bom no)
+		(in_bom yes)
 		(on_board yes)
 		(dnp no)
@@
 			)
 		)
-		(property "Value" "470nH"
+		(property "Value" "500nH"
 			(at 142.748 92.71 0)
 			(effects
@@
 			)
 		)
-		(property "Footprint" "Library:L_1206_3216Metric-keepout"
+		(property "Footprint" "Inductor_SMD:L_Coilcraft_2929SQ-501"
 			(at 139.7 91.44 0)
 			(effects
@@
 			)
 		)
-		(property "Description" "Inductor with ferrite core, small symbol"
+		(property "Description" "Inductor, small symbol"
 			(at 139.7 91.44 0)
 			(effects
@@
 			)
 		)
-		(property "Manufacturer" "Abracon"
+		(property "Manufacturer" "Coilcraft"
 			(at 139.7 91.44 0)
 			(effects
@@
 			)
 		)
-		(property "MPN" "AISC-1206-R47G-T"
+		(property "MPN" "2929SQ-501JEC"
 			(at 139.7 91.44 0)
 			(effects
@@
 			)
 		)
-		(property "Mouser_PN" "994-1206CS-471XJRC"
+		(property "Mouser_PN" "994-2929SQ-501JEC"
 			(at 139.7 91.44 0)
 			(effects
